File: pcb/mainboard_lite/dp_in.kicad_sch (KiCad schematic)
At the start: 17 parts, among them J402 HDMI_A, Q401 BSS138, Q402 BSS138, Q403 BSS138

Commit message: Lite version r0p1
Parts:
- removed Q401, Q402, Q403: BSS138, Package_TO_SOT_SMD:SOT-23, symbol Transistor_FET:BSS138
- added Q6 (x3): AO3400A, Package_TO_SOT_SMD:SOT-23, symbol Device:Q_NMOS_GSD
- added R60: 120K/1%, Resistor_SMD:R_0402_1005Metric, symbol Device:R
- added R61: 240K/1%, Resistor_SMD:R_0402_1005Metric, symbol Device:R
- renumbered D405 to D10, D404 to D9, J402 to J4, R412 to R48, R413 to R52, R414 to R55
Connections:
- net +3V3: now also Q6.1 (G), Q6.1 (G), Q6.1 (G)
- net DDC_SCL: now also Q6.2 (S)
- net DDC_SDA: now also Q6.2 (S)
- net FPGA_DONE: now also Q6.2 (S)
- net GND: now also R61.2
- net HPD_5V: now also Q6.3 (D)
- net SCL_5V: now also Q6.3 (D)
- net SDA_5V: now also Q6.3 (D)
- net at J4.18 (+5V): now also R60.1
- new net HDMI_DET: R60.2, R61.1
- no-connect marks 3 -> 2
