File: pcb/mainboard_lite/fpga.kicad_sch (KiCad schematic)
At the start: 20 parts, among them J201 Conn_02x05_Odd_Even, U200 XC6SLX16-FTG256, U406 W25Q16JVP, Y201 33MHz

Commit message: Lite version r0p1
Parts:
- removed C443: 220nF, Capacitor_SMD:C_0402_1005Metric, symbol Device:C
- removed R424: 10K/1%, Resistor_SMD:R_0402_1005Metric, symbol Device:R
- removed R425, R426: 4.7K, Resistor_SMD:R_0402_1005Metric, symbol Device:R
- removed U406: W25Q16JVP, Package_SON:WSON-8-1EP_6x5mm_P1.27mm_EP3.4x4.3mm, symbol Memory_Flash:W25Q32JVZP
- renumbered C201 to C26, C203 to C27, C204 to C28, C202 to C29, C209 to C30, J201 to J2, R310 to R10, R201 to R11, R202 to R12, R306 to R13, R309 to R14, R428 to R15, R209 to R16, U200 to U5, Y201 to Y1
Connections:
- net DDC_SCL: no longer names the net of U5.A12 (IO_L62N_VREF_0)
- net DDC_SDA: no longer names the net of U5.A13 (IO_L63N_SCP6_0)
- net EPD_POWEREN: no longer names the net of U5.B15 (IO_L29P_A23_M1A13_1)
