File: pcb/mainboard_lite/fpga_ddr.kicad_sch (KiCad schematic)
At the start: 37 parts, among them U200 XC6SLX16-FTG256, U502 MT41K64M16TW

Commit message: Lite version r0p1
Parts:
- renumbered C503 to C64, C501 to C65, C504 to C66, C502 to C67, C529 to C68, C508 to C69, C510 to C70, C511 to C71, C509 to C72, C513 to C73, C514 to C74, C512 to C75, C515 to C76, C516 to C77, C517 to C78, C518 to C79, C519 to C80, C520 to C81, C521 to C82, C522 to C83, C523 to C84, C524 to C85, C525 to C86, C526 to C87, C527 to C88, R509 to R35, R510 to R36, R505 to R37, R506 to R38, R501 to R39, R507 to R40, R502 to R41, R508 to R42, R503 to R43, R504 to R44, U502 to U12, U200 to U5
Connections:
- net +3V3: now also R36.1
- net GND: no longer R36.1
- net FPGA_CS: now reaches U5.L10 (IO_L16P_2)
- net EPD_VCOM_PWM: no longer names the net of U5.T4 (IO_L63N_2)
- net FPGA_FCCLK renamed FPGA_SCLK
- net FPGA_FCS: no longer names the net of U5.T3 (IO_L65N_CSO_B_2)
- net FPGA_FMISO renamed FPGA_MOSI
- net FPGA_FMOSI renamed FPGA_MISO
