File: pcb/mainboard_lite/power.kicad_sch (KiCad schematic)
At the start: 46 parts, among them J403 USB_C_Receptacle_USB2.0, J404 Power Switch, U200 XC6SLX16-FTG256, U401 SY8120, U404 SY8120, U405 SY8120

Commit message: Lite version r0p1
Parts:
- removed C442: 10uF/10V, Capacitor_SMD:C_0805_2012Metric, symbol Device:C
- removed J403: USB_C_Receptacle_USB2.0, Connector_USB:USB_C_Receptacle_HRO_TYPE-C-31-M-12, symbol Connector:USB_C_Receptacle_USB2.0
- removed J404: Power Switch, Connector_PinHeader_2.54mm:PinHeader_1x02_P2.54mm_Vertical, symbol Connector_Generic:Conn_01x02
- removed R417, R418: 5.1K/1%, Resistor_SMD:R_0402_1005Metric, symbol Device:R
- added C103: 47uF/10V, Capacitor_SMD:C_1206_3216Metric, symbol Device:C
- added C211, C214, C219: 220nF, Capacitor_SMD:C_0402_1005Metric, symbol Device:C
- added R9: 10K/1%, Resistor_SMD:R_0402_1005Metric, symbol Device:R
- added U4: MT9700, Package_TO_SOT_SMD:SOT-23-5, symbol symbols:MT9700
- renumbered C409 to C1, C420 to C10, C421 to C11, C433 to C12, C434 to C13, C435 to C14, C437 to C15, C438 to C16, C411 to C2, C412 to C3, C413 to C4, C415 to C5, C416 to C6, C417 to C8, C419 to C9, L404 to L1, L406 to L2, L407 to L3, R415 to R3, R416 to R4, R419 to R5, R420 to R6, R421 to R7, R422 to R8, U401 to U1, U404 to U2, U405 to U3, U200 to U5
Connections:
- net +1V0: now also C219.1
- net +3V3: now also C211.1, C214.1
- net +5V: now also C103.2, U4.1 (VOUT)
- net GND: now also C103.1, C211.2, C214.2, C219.2, R9.1, U4.2 (GND)
- net VBUS: now also U4.4 (EN), U4.5 (VIN)
- new net: R9.2, U4.3 (SET)
- no-connect marks 6 -> 0
Other:
- note added: "Ilim = 0.68A"
- moved on the sheet: C210, C211, C213, C214, C215, C217, C219, C220, C618, H1, H2, H3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
