File: pcb/mainboard_lite/eink.kicad_sch (KiCad schematic)
At the start: 78 parts, among them J401 FH12-40S-0.5SH, Q404 BSS84, Q406 S8050W, U402 MT3608, U403 MT9700, U404 LGS5148, U408 MT3608, U411 LM321

Commit message: Lite version r0p1
Parts:
- removed C302, C303, C304: 220nF, Capacitor_SMD:C_0402_1005Metric, symbol Device:C
- removed C414: 47uF/10V, Capacitor_SMD:C_1206_3216Metric, symbol Device:C
- removed Q404: BSS84, Package_TO_SOT_SMD:SOT-23, symbol Transistor_FET:BSS84
- removed U402, U408: MT3608, Package_TO_SOT_SMD:TSOT-23-5, symbol symbols:LT1615
- added C1: 10uF/10V, Capacitor_SMD:C_0805_2012Metric, symbol Device:C
- added Q1, Q7, Q8: AO3401A, Package_TO_SOT_SMD:SOT-23, symbol Device:Q_PMOS_GSD
- added Q6: AO3400A, Package_TO_SOT_SMD:SOT-23, symbol Device:Q_NMOS_GSD
- added R420 (x2): 51R, Resistor_SMD:R_0402_1005Metric, symbol Device:R
- added R420: 120K/1%, Resistor_SMD:R_0402_1005Metric, symbol Device:R
- added R420: 10K/1%, Resistor_SMD:R_0402_1005Metric, symbol Device:R
- added R420: 20K/1%, Resistor_SMD:R_0402_1005Metric, symbol Device:R
- added U7, U8: MT3608(SOT23-6), Package_TO_SOT_SMD:SOT-23-6, symbol symbols:MT3608(SOT23-6)
- C437: value 10uF/10V -> 1uF; footprint Capacitor_SMD:C_0805_2012Metric -> Capacitor_SMD:C_0402_1005Metric
- D5: value 4148WT -> 4148WS; footprint Diode_SMD:D_SOD-523 -> Diode_SMD:D_SOD-323
- Q2: renamed from Q406; value S8050W -> S8050; footprint Package_TO_SOT_SMD:SOT-323_SC-70 -> Package_TO_SOT_SMD:SOT-23
- RN1: renamed from RN401; value 33R -> 33R / 4D02WGF330JTCE
- RN2: renamed from RN402; value 33R -> 33R / 4D02WGF330JTCE
- RN3: renamed from RN403; value 33R -> 33R / 4D02WGF330JTCE
- RN4: renamed from RN404; value 33R -> 33R / 4D02WGF330JTCE
- RN5: renamed from RN405; value 33R -> 33R / 4D02WGF330JTCE
- RN6: renamed from RN406; value 33R -> 33R / 4D02WGF330JTCE
- renumbered C305 to C60, C306 to C61, C307 to C62, C308 to C63, D401 to D1, D402 to D2, D406 to D3, D403 to D4, D408 to D6, J401 to J3, U411 to U11
Connections:
- net +3V3: now also Q7.2 (S), R420.1
- net +5V: now also Q1.2 (S); no longer U403.5 (VIN)
- net +5V_EPD: now also U7.4 (~{SHDN}), U7.5 (VIN), U7.6 (NC), U8.4 (~{SHDN}), U8.5 (VIN), U8.6 (NC)
- net GND: now also C1.1, U7.2 (GND), U8.2 (GND)
- net VCOM: now also Q6.3 (D), R420.2; no longer U11.3 (-), U11.4
- net VNEG: now also R420.2
- net at D1.2 (A), L404.2: now also U7.1 (SW)
- net at C421.1, R415.1, R416.2: now also U7.3 (NFB)
- net at Q2.3 (C), R419.1: now also Q1.1 (G)
- net at D5.2 (A), D5.2 (A): now also Q1.3 (D)
- net at C421.1, R415.1, R416.2: now also U8.3 (NFB)
- net at D2.2 (A), L404.2: now also U8.1 (SW)
- net EPD_POWEREN renamed EPD_PWR_EN
- new net: Q7.1 (G), R420.2
- new net: Q6.1 (G), Q7.3 (D), R420.1
- new net: Q8.1 (G), R420.1
- new net: Q6.2 (S), U11.3 (-), U11.4
- new net: Q8.3 (D), R420.1
- new net VBUS: C1.2, U403.5 (VIN)
- new net VCOM_EN: R420.1
- new net VCOM_MEA: Q8.2 (S), R420.2
- new net VCOM_MEA_EN: R420.2
Other:
- moved on the sheet: C3, C415, C437, C60, C61, C62, C63, D5, J3, R1, R2, RN1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
