File: pcb/mainboard/pcb.kicad_pcb (KiCad board)
At the start: 4 copper layers, 60 x 60 mm, 267 parts, among them J1 USB_C_Receptacle, J2 DNP, J3 FH12-40S-0.5SH, J4 DVI, J5 SM03B-SRSS-TB, Q1 AO3401A, Q2 S8050, Q6 AO3400A, Q7 AO3401A, Q8 AO3401A, SW1 SW, SW2 SW, U1 SY8120, U10 LGS5148, U11 LM321, U12 MT41K64M16TW, U13 W25Q32JV, U14 RP2040, U15 ADV7611, U16 USBLC6-2P6, U17 FUSB302BMPX, U18 CBTL02043A, U19 PTN3460, U2 SY8120, U3 SY8120, U4 MT9700, U5 XC6SLX16-FTG256, U6 MT9700, U7 MT3608(SOT23-6), U8 MT3608(SOT23-6), U9 LGS5148, Y1 33MHz, Y2 12MHz, Y3 28.63636MHz

Commit message: r0p7 layout done
Parts:
- removed J2: DNP, Connector_PinHeader_1.27mm:PinHeader_2x05_P1.27mm_Vertical_SMD
- removed R16: 4.7K, Resistor_SMD:R_0402_1005Metric
- removed R56: 1K, Resistor_SMD:R_0402_1005Metric
- added C140: 470nF, Capacitor_SMD:C_0402_1005Metric, B.Cu at (120.0, 66.0)
- added C141: 470nF, Capacitor_SMD:C_0402_1005Metric, B.Cu at (120.3, 69.9)
- added C142: 47uF/6.3V, Capacitor_SMD:C_0603_1608Metric, B.Cu at (138.9, 75.2)
- added C143: 47uF/6.3V, Capacitor_SMD:C_0603_1608Metric, F.Cu at (129.6, 82.5)
- added C144: 4.7uF, Capacitor_SMD:C_0402_1005Metric, B.Cu at (117.8, 70.3)
- added C145: 47uF/6.3V, Capacitor_SMD:C_0603_1608Metric, F.Cu at (114.3, 56.7)
- added C146: 470nF, Capacitor_SMD:C_0402_1005Metric, B.Cu at (117.2, 77.0)
- added C147: 47uF/6.3V, Capacitor_SMD:C_0603_1608Metric, F.Cu at (114.3, 58.3)
- added C148: 4.7uF, Capacitor_SMD:C_0402_1005Metric, B.Cu at (128.0, 69.9)
- added C149: 470nF, Capacitor_SMD:C_0402_1005Metric, B.Cu at (135.0, 67.5)
- added C150: 470nF, Capacitor_SMD:C_0402_1005Metric, B.Cu at (126.0, 69.9)
- added C151: 10uF/10V, Capacitor_SMD:C_0805_2012Metric, F.Cu at (128.2, 98.5)
- added C152: 100nF, Capacitor_SMD:C_0402_1005Metric, F.Cu at (128.7, 97.0)
- added C153: 100nF, Capacitor_SMD:C_0402_1005Metric, F.Cu at (130.6, 94.0)
- added C154: 47pF, Capacitor_SMD:C_0402_1005Metric, F.Cu at (125.8, 91.2)
- added C155: 10uF/10V, Capacitor_SMD:C_0805_2012Metric, F.Cu at (131.8, 98.5)
- added FID1: Fiducial, Fiducial:Fiducial_1mm_Mask2mm, F.Cu at (153.5, 82.5)
- added FID2: Fiducial, Fiducial:Fiducial_1mm_Mask2mm, F.Cu at (136.0, 45.0)
- added FID3: Fiducial, Fiducial:Fiducial_1mm_Mask2mm, F.Cu at (96.5, 79.5)
- added FID4: Fiducial, Fiducial:Fiducial_1mm_Mask2mm, B.Cu at (99.0, 93.0)
- added FID5: Fiducial, Fiducial:Fiducial_1mm_Mask2mm, B.Cu at (99.5, 46.5)
- added FID6: Fiducial, Fiducial:Fiducial_1mm_Mask2mm, B.Cu at (147.5, 84.5)
- added L8: FTC201610S4R7MBCA, Inductor_SMD:L_Murata_DFE201610P, F.Cu at (131.4, 96.2)
- added R10: 20K/1%, Resistor_SMD:R_0402_1005Metric, F.Cu at (125.8, 90.2)
- added R48: 10K/1%, Resistor_SMD:R_0402_1005Metric, F.Cu at (127.8, 91.7)
- added U20: SY8120, Package_TO_SOT_SMD:TSOT-23-6, F.Cu at (128.2, 94.3)
- C116, C126, C129, C130, C138, R14, R15: moved to B.Cu
- C18, C19, C24, C25, C26, C27, C64: value 220nF -> 47uF/6.3V; footprint Capacitor_SMD:C_0402_1005Metric -> Capacitor_SMD:C_0603_1608Metric
- C20, C22, C28, C57, C59, C66: value 220nF -> 4.7uF
- C21, C29, C58, C67: value 220nF -> 470nF
- C23: value 22uF -> 4.7uF; footprint Capacitor_SMD:C_0603_1608Metric -> Capacitor_SMD:C_0402_1005Metric
- C65: value 220nF -> 47uF/6.3V; footprint Capacitor_SMD:C_0402_1005Metric -> Capacitor_SMD:C_0603_1608Metric; moved to F.Cu
- C86: value 10uF/10V -> 22uF; footprint Capacitor_SMD:C_0805_2012Metric -> Capacitor_SMD:C_0603_1608Metric
- J4: footprint Connector_HDMI:HDMI_Micro-D_Molex_46765-1x01 -> footprints:HDMI_Micro-D_Molex_46765-1x01_MOD
- R46: moved to F.Cu
- R7: value 16K/1% -> 20K/1%
- R8: value 27K/1% -> 20K/1%
- moved C56 46.1 mm to (119.0, 90.4)
- moved R64 42.1 mm to (118.8, 86.6)
- moved C49 33.7 mm to (100.2, 86.5), turned to 180 degrees
- moved R26 30.5 mm to (121.7, 81.3), turned to 0 degrees
- moved C64 30.2 mm to (114.3, 52.7)
- moved C65 22.1 mm to (114.3, 51.1), turned to 180 degrees
- moved C84 19.3 mm to (118.3, 44.9)
- moved C60 18.1 mm to (103.5, 90.3)
- moved R14 16.2 mm to (120.5, 76.5), turned to 0 degrees
- moved R42 14.5 mm to (131.0, 66.5), turned to 180 degrees
- moved C29 12.2 mm to (128.1, 68.9), turned to 0 degrees
- moved C26 11.6 mm to (118.0, 66.5), turned to -90 degrees
- moved C66 11.4 mm to (131.2, 63.9), turned to 0 degrees
- moved D5 10.5 mm to (109.8, 60.1)
- moved R27 10.4 mm to (106.4, 60.5), turned to 0 degrees
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Connections:
- net +1V0 renamed +1V2
- net DDC_SDA renamed /mcu/GPIO0
- net Net-(RN10-R1.1) renamed /tmds_in/ADV_P23
- net Net-(RN10-R2.1) renamed /tmds_in/ADV_P22
- net Net-(RN10-R3.1) renamed /tmds_in/ADV_P21
- net Net-(RN10-R4.1) renamed /tmds_in/ADV_P20
- net Net-(RN11-R1.1) renamed /tmds_in/ADV_P19
- net Net-(RN11-R2.1) renamed /tmds_in/ADV_P18
- net Net-(RN11-R3.1) renamed /tmds_in/ADV_P17
- net Net-(RN11-R4.1) renamed /tmds_in/ADV_P16
- net Net-(RN12-R1.1) renamed /tmds_in/ADV_P7
- net Net-(RN12-R2.1) renamed /tmds_in/ADV_P6
- net Net-(RN12-R3.1) renamed /tmds_in/ADV_P5
- net Net-(RN12-R4.1) renamed /tmds_in/ADV_P4
- net Net-(RN13-R1.1) renamed /tmds_in/ADV_P3
- net Net-(RN13-R2.1) renamed /tmds_in/ADV_P2
- net Net-(RN13-R3.1) renamed /tmds_in/ADV_P1
- net Net-(RN13-R4.1) renamed /tmds_in/ADV_P0
- net Net-(RN7-R1.1) renamed /tmds_in/ADV_DE
- net Net-(RN7-R2.1) renamed /tmds_in/ADV_HS
- net Net-(RN7-R3.1) renamed /tmds_in/ADV_VS
- net Net-(RN8-R1.1) renamed /tmds_in/ADV_P11
- net Net-(RN8-R2.1) renamed /tmds_in/ADV_P10
- net Net-(RN8-R3.1) renamed /tmds_in/ADV_P9
- net Net-(RN8-R4.1) renamed /tmds_in/ADV_P8
- net Net-(RN9-R1.1) renamed /tmds_in/ADV_P15
- net Net-(RN9-R2.1) renamed /tmds_in/ADV_P14
- net Net-(RN9-R3.1) renamed /tmds_in/ADV_P13
- net Net-(RN9-R4.1) renamed /tmds_in/ADV_P12
- net Net-(U15-LLC) renamed /tmds_in/ADV_CK
- C116 pad 1: Net-(U19-VDD18REG) -> +1V8
- C119 pad 1: Net-(U19-VDD18REG) -> +1V8
- C122 pad 1: Net-(U19-VDD18REG) -> +1V8
- C64 pad 1: +3V3 -> +1V35
- C65 pad 1: +3V3 -> +1V35
- D13 pad 2: /dp_in/CC1 -> /dp_in/SBU2
- D13 pad 4: /dp_in/SBU2 -> /dp_in/CC1
- D13 pad 7: /dp_in/SBU2 -> /dp_in/CC1
- D13 pad 9: /dp_in/CC1 -> /dp_in/SBU2
- Q1 pad 2: +5V -> +5V_EPD
- R28 pad 2: +5V -> +5V_EPD
- SW1 pad 1: Net-(R56-Pad2) -> KEY2
- U14 pad 3: DDC_SCL -> ADV_INT
- U14 pad 37: /mcu/GPIO25 -> DEC_RST
- U14 pad 4: TCPC_SDA -> I2C_SDA
- U14 pad 5: TCPC_SCL -> I2C_SCL
- U14 pad 7: KEY -> KEY2
- U14 pad 8: /mcu/GPIO6 -> KEY
- U18 pad 11: Net-(U18-GND-Pad11) -> GND
- U18 pad 2: TYPEC_ORI -> GND
- U18 pad 20: Net-(U18-GND-Pad11) -> GND
- U18 pad 21: Net-(U18-GND-Pad11) -> GND
- U18 pad 5: Net-(U18-GND-Pad11) -> GND
- U18 pad 9: GND -> TYPEC_ORI
- U19 pad 19: Net-(U19-VDD18REG) -> unconnected-(U19-VDD18REG-Pad19)
- U19 pad 45: Net-(U19-VDD18REG) -> +1V8
- U19 pad 56: unconnected-(U19-EPS_N-Pad56) -> GND
- U19 pad 6: Net-(U19-VDD18REG) -> +1V8
- U5 pad A10: LVDS_ODD_CKN -> LVDS_ODD_CKP
- U5 pad A13: LVDS_EVEN_CN -> LVDS_EVEN_BP
- U5 pad A14: VIN_HPD -> LVDS_EVEN_CN
- U5 pad A8: LVDS_ODD_CN -> LVDS_ODD_BP
- U5 pad B10: LVDS_ODD_CKP -> LVDS_ODD_CKN
- U5 pad B14: unconnected-(U5A-IO_L65P_SCP3_0-PadB14) -> LVDS_EVEN_CP
- U5 pad B8: LVDS_ODD_CP -> LVDS_ODD_BN
- U5 pad C13: LVDS_EVEN_CP -> LVDS_EVEN_BN
- U5 pad C5: LVDS_ODD_AN -> unconnected-(U5A-IO_L3N_0-PadC5)
- U5 pad D11: unconnected-(U5A-IO_L66P_SCP1_0-PadD11) -> LVDS_EVEN_AN
- U5 pad D12: unconnected-(U5A-IO_L66N_SCP0_0-PadD12) -> LVDS_EVEN_AP
- U5 pad D5: LVDS_ODD_AP -> unconnected-(U5A-IO_L3P_0-PadD5)
- U5 pad D9: LVDS_EVEN_BN -> LVDS_ODD_CN
- U5 pad E6: LVDS_ODD_BN -> unconnected-(U5A-IO_L5N_0-PadE6)
- U5 pad E7: LVDS_EVEN_AP -> LVDS_ODD_AN
- U5 pad E8: LVDS_EVEN_AN -> LVDS_ODD_AP
- U5 pad F7: LVDS_ODD_BP -> unconnected-(U5A-IO_L5P_0-PadF7)
- U5 pad F9: LVDS_EVEN_BP -> LVDS_ODD_CP
Routing:
- net GND: track 59.8 -> 312.6 mm, vias 66 -> 211
- net +1V8: track 0.00 -> 114.4 mm, vias 0 -> 8
- net +5V: track 0.00 -> 109.2 mm, vias 0 -> 5
- net I2C_SCL: track 0.00 -> 105.4 mm, vias 0 -> 4
- net I2C_SDA: track 0.00 -> 104.9 mm, vias 0 -> 4
- net VBUS: track 0.00 -> 104.5 mm, vias 0 -> 6
- net DEC_RST: track 0.00 -> 101.1 mm, vias 0 -> 3
- net ADV_INT: track 0.00 -> 97.7 mm, vias 0 -> 2
- net +3V3: track 30.6 -> 128.3 mm, vias 14 -> 53
- net USB_DP: track 1.14 -> 97.1 mm, vias 1 -> 3
- net USB_DN: track 1.16 -> 95.6 mm, vias 1 -> 2
- net TCPC_INT: track 0.00 -> 91.8 mm, vias 0 -> 2
- net TYPEC_ORI: track 0.00 -> 79.2 mm, vias 0 -> 6
- net DP_PDN: track 0.00 -> 77.5 mm, vias 0 -> 4
- net KEY2: track 0.00 -> 73.7 mm, vias 0 -> 2
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- added copper zone on F.Cu, net +1V2
- added copper zone on In1.Cu, net +1V2
- added copper zone on F.Cu, net +1V35
- added copper zone on In1.Cu, net +1V35
- added copper zone on F.Cu, net +3V3
- added copper zone on In1.Cu, net +3V3
- added copper zone on F.Cu, net +5V
- added copper zone on In1.Cu, net +5V_EPD
- added copper zone on In2.Cu, net GND
- added copper zone on F.Cu, net VBUS
- added copper zone on F.Cu, net VNEG
Other:
- board text added: "R0.7 Modos"
- board text removed: "FPGA JTAG"
- board text removed: "R0.8 Modos"
