File: pcb/mainboard/pcb.kicad_pcb (KiCad board)
At the start: 4 copper layers, 60 x 60 mm, 290 parts, among them J1 USB_C_Receptacle, J3 FH12-40S-0.5SH, J4 DVI, J5 SM03B-SRSS-TB, Q1 AO3401A, Q2 S8050, Q6 AO3400A, Q7 AO3401A, Q8 AO3401A, SW1 SW, SW2 SW, U1 SY8120, U10 LGS5148, U11 LM321, U12 MT41K64M16TW, U13 W25Q32JV, U14 RP2040, U15 ADV7611, U16 USBLC6-2P6, U17 FUSB302BMPX, U18 CBTL02043A, U19 PTN3460, U2 SY8120, U20 SY8120, U3 SY8120, U4 MT9700, U5 XC6SLX16-FTG256, U6 MT9700, U7 MT3608(SOT23-6), U8 MT3608(SOT23-6), U9 LGS5148, Y1 33MHz, Y2 12MHz, Y3 28.63636MHz

Commit message: PCB r0p8
Parts:
- added C156: 100nF, Capacitor_SMD:C_0402_1005Metric, F.Cu at (97.4, 46.0)
- added J2: XUNPU HDMI-101S, footprints:HDMI_Micro-D_Molex_46765-1x01_MOD, F.Cu at (153.2, 89.0)
- added R16: 10K, Resistor_SMD:R_0402_1005Metric, B.Cu at (139.0, 93.8)
- added R49: 10K, Resistor_SMD:R_0402_1005Metric, B.Cu at (140.0, 93.8)
- added R50: 1M, Resistor_SMD:R_0402_1005Metric, F.Cu at (99.4, 46.0)
- added R51: 1M, Resistor_SMD:R_0402_1005Metric, F.Cu at (97.4, 47.2)
- J1: value USB_C_Receptacle -> XUNPU TYPEC-324G-ACP24; footprint footprints:AMPHENOL_10137065-00021LF -> footprints:XUNPU_TypeC-324G-ACP24
- J4: value DVI -> SM03B-SRSS-TB; footprint footprints:HDMI_Micro-D_Molex_46765-1x01_MOD -> Connector_JST:JST_SH_SM03B-SRSS-TB_1x03-1MP_P1.00mm_Horizontal
- moved J4 54.8 mm to (98.4, 88.4), turned to -90 degrees
- moved C49 11.6 mm to (96.4, 75.6), turned to -90 degrees
- moved FID5 2.42 mm to (101.0, 48.4)
- moved U7 0.85 mm to (102.2, 75.4)
- moved C51 0.80 mm to (98.8, 75.6)
- moved C40 0.70 mm to (102.7, 72.6)
- moved R23 0.70 mm to (100.5, 72.6)
- moved R22 0.70 mm to (101.6, 72.6)
- moved J5 0.66 mm to (98.4, 58.5)
- moved C53 0.36 mm to (100.2, 83.8)
- moved C31 0.36 mm to (96.5, 82.6)
- moved L4 0.36 mm to (100.2, 80.2)
- moved J1 0.25 mm to (152.9, 74.9)
- moved R57 0.25 mm to (100.4, 51.9)
Connections:
- net HDMI_DET renamed /mcu/GPIO8
- J4 pad 1: /tmds_in/TMDS_D2P -> VBUS
- J4 pad 3: /tmds_in/TMDS_D2N -> FL_PWM
- U14 pad 27: /mcu/GPIO16 -> FL_PWM
- U14 pad 41: /mcu/GPIO29_ADC3 -> VBUS_MEA
- U15 pad 53: I2C_SDA -> I2C_SCL
- U15 pad 54: I2C_SCL -> I2C_SDA
Routing:
- net VBUS: track 104.5 -> 163.3 mm, vias 6 -> 8
- net FL_PWM: track 0.00 -> 36.9 mm, vias 0 -> 2
- net VBUS_MEA: track 0.00 -> 20.6 mm, vias 0 -> 2
- net /tmds_in/HDMI_HPD: track 10.8 -> 20.7 mm
- net /tmds_in/HDMI_5V: track 12.6 -> 18.8 mm
- net GND: track 312.6 -> 316.4 mm, vias 211 -> 214
- net /dp_in/TX1N: track 7.70 -> 9.96 mm
- net /dp_in/TX1P: track 7.81 -> 9.94 mm
- net /tmds_in/HDMI_SCL: track 11.8 -> 13.5 mm
- net FPGA_CS: track 37.0 -> 38.7 mm
- net Net-(D1-A): track 6.32 -> 7.93 mm
- net /tmds_in/HDMI_SDA: track 13.6 -> 15.0 mm
- net VPOS: track 41.2 -> 40.1 mm
- net USB_DN: track 95.6 -> 94.7 mm
- net +5V_EPD: track 42.3 -> 41.5 mm
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- removed copper zone on B.Cu, net GND
Other:
- board text added: "R0.8 WZ"
- board text removed: "R0.7 Modos"

Commit message: BOM adjustments
Parts:
- C38, C39, C40, C41: value 22pF -> 18pF
- C84, C85, C86: value 22uF -> 47uF/6.3V
- D1, D2, D3, D4, D6: value 1N5819WS -> B0530WS
- D5, D7, D8: value 4148WS -> B0530WS
- FB1, FB2: value 120 -> 120R
- R1, R12, R13, R14, R2, R38, R40, R42: value 4.7K -> 5.1K
- R21, R29: value 5.1K/1% -> 5.1K
- R46: value 33 -> 27R
- Y2, Y3: footprint Oscillator:Oscillator_SMD_Abracon_ASE-4Pin_3.2x2.5mm -> Crystal:Crystal_SMD_3225-4Pin_3.2x2.5mm
