File: pcb/mainboard/eink.kicad_sch (KiCad schematic)
At the start: 48 parts, among them J401 FH12-40S-0.5SH, U401 MAX17135

Commit message: pcb: r0p4
Parts:
- L303, L401: footprint footprints:L_1212 -> footprints:L_FXL0420; LCSC C340379 -> C167208
Connections:
- net EPD_PWR_SCL renamed I2C_SCL
- net EPD_PWR_SDA renamed I2C_SDA
Other:
- company: Copyright 2021 Modos / Engineer: Wenting Zhang -> Copyright 2022 Modos / Engineer: Wenting Zhang
- moved on the sheet: C302, C303, C304, C305, C306, C307, C308, C310, C312, C313, C317, C319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

Commit message: pcb: r0p5
Parts:
- removed C310, C313: 100nF, Capacitor_SMD:C_0402_1005Metric, symbol Device:C
- removed C312: 10uF, Capacitor_SMD:C_0603_1608Metric, symbol Device:C
- removed C317: 1uF/25V, Capacitor_SMD:C_0805_2012Metric, symbol Device:C
- removed C319: 2.2nF, Capacitor_SMD:C_0402_1005Metric, symbol Device:C
- removed C320: 4.7uF/25V, Capacitor_SMD:C_0805_2012Metric, symbol Device:C
- removed C321: 1uF, Capacitor_SMD:C_0402_1005Metric, symbol Device:C
- removed D301, D302, D303, D304, D305: B0530WS, Diode_SMD:D_SOD-323, symbol Device:D_Schottky
- removed L303: 4.7uH, footprints:L_FXL0420, symbol Device:L
- removed R307: 562K/1%, Resistor_SMD:R_0402_1005Metric, symbol Device:R
- removed R308: 27K/1%, Resistor_SMD:R_0402_1005Metric, symbol Device:R
- removed R401: 806K/1%, Resistor_SMD:R_0402_1005Metric, symbol Device:R
- removed U401: MAX17135, Package_DFN_QFN:QFN-32-1EP_5x5mm_P0.5mm_EP3.1x3.1mm_ThermalVias, symbol symbols:MAX17135
- added C413, C414, C415, C417, C419: 4.7uF, Capacitor_SMD:C_0603_1608Metric, symbol Device:C
- added C416, C418, C421: 4.7uF/25V, Capacitor_SMD:C_0805_2012Metric, symbol Device:C
- added C420: 100nF, Capacitor_SMD:C_0402_1005Metric, symbol Device:C
- added D402, D403, D404, D405, D406: B0530WS, Diode_SMD:D_SOD-323, symbol Device:D_Schottky
- added L402: FXL0420-4R7-M, footprints:L_FXL0420, symbol Device:L
- added R410: 510K/1%, Resistor_SMD:R_0402_1005Metric, symbol Device:R
- added R411: 24K/1%, Resistor_SMD:R_0402_1005Metric, symbol Device:R
- added TH401: 10K, Resistor_SMD:R_0402_1005Metric, symbol Device:Thermistor_NTC
- added U401: TPS65185, footprints:QFN-48-1EP_7x7mm_P0.5mm_EP4.1x4.1mm_ThermalVias, symbol symbols:TPS65185
- C401, C403: value 1uF/25V -> 4.7uF/25V; LCSC C111769 -> (none); Ref.Price 0.0174 -> (none)
- C402: value 1uF/25V -> 100nF; footprint Capacitor_SMD:C_0805_2012Metric -> Capacitor_SMD:C_0402_1005Metric; LCSC C111769 -> (none); Ref.Price 0.0174 -> (none)
- C404: value 100nF -> 4.7uF; footprint Capacitor_SMD:C_0402_1005Metric -> Capacitor_SMD:C_0603_1608Metric; LCSC C56392 -> (none); Ref.Price 0.0023 -> (none)
- C405, C410: value 4.7uF/25V -> 10uF; footprint Capacitor_SMD:C_0805_2012Metric -> Capacitor_SMD:C_0603_1608Metric; LCSC C105489 -> (none); Ref.Price 0.0271 -> (none)
- C406, C408, C412: LCSC C105489 -> (none); Ref.Price 0.0271 -> (none)
- C407: value 10uF -> 10nF; footprint Capacitor_SMD:C_0603_1608Metric -> Capacitor_SMD:C_0402_1005Metric; LCSC C105490 -> (none); Ref.Price 0.0165 -> (none)
- C409: value 4.7uF/25V -> 4.7uF; footprint Capacitor_SMD:C_0805_2012Metric -> Capacitor_SMD:C_0603_1608Metric; LCSC C105489 -> (none); Ref.Price 0.0271 -> (none)
- C411: value 4.7uF/25V -> 10nF; footprint Capacitor_SMD:C_0805_2012Metric -> Capacitor_SMD:C_0402_1005Metric; LCSC C105489 -> (none); Ref.Price 0.0271 -> (none)
- D401: LCSC C475612 -> (none); Ref.Price 0.0209 -> (none)
- L401: value 4.7uH -> FXL0420-2R2-M; LCSC C167208 -> (none); Ref.Price 0.0643 -> (none)
- R402: value 49.9K/1% -> 470K/1%; LCSC C137969 -> (none); Ref.Price 0.001 -> (none)
- R403: value 10R -> 18K/1%; LCSC C137925 -> (none); Ref.Price 0.0006 -> (none)
- R404: value 0.5R -> 43K; footprint Resistor_SMD:R_0603_1608Metric -> Resistor_SMD:R_0402_1005Metric; LCSC C45312 -> (none); Ref.Price 0.004 -> (none)
Connections:
- net +3V3: now also C419.1, U401.12 (VCOM_CTRL), U401.45 (VIN3P3)
- net +3V3_LCD: now also C417.1, U401.46 (V3P3)
- net +5V: now also C405.2, C410.1, L401.1, U401.24 (VINP); no longer C407.2, R403.2
- net GND: now also C401.1, C402.1, C403.1, C404.1, C405.1, C406.1, C408.1, C409.1, C410.2, C412.2, R403.2, R404.1, C413.2, C414.2, C415.2, C416.2, C417.2, C418.1, C419.2, C420.2, C421.1, L402.2, R411.2, TH401.1, U401.14 (VCOM_DIS), U401.32 (PGND2), U401.41 (PGND1), U401.48 (AGND2), U401.6 (DGND), U401.8 (AGND1)
- net I2C_SCL: now also U401.17 (SCL)
- net I2C_SDA: now also U401.18 (SDA)
- net VCOM: now also C404.2, U401.15 (VCOM)
- net VGH: now also C403.2, D401.1 (K), R402.1, U401.35 (VDDH_DIS); no longer C402.2
- net VGL: now also C421.2, D406.2 (A), R410.1, U401.29 (VEE_DIS); no longer C401.2
- net VNEG: now also C418.2, U401.3 (VNEG), U401.9 (VNEG_DIS); no longer C406.2, C409.2
- net VPOS: now also C401.2, U401.19 (VPOS_DIS), U401.44 (VPOS); no longer C405.2, C408.2
- net at R402.2: now also R403.1, U401.33 (VDDH_FB)
- net at R404.2: now also TH401.2, U401.47 (TS); no longer C410.2
- removed net GNDPWR: C401.1, C402.1, C403.1, C405.1, C406.1, C407.1, C408.1, C409.1, C410.1, C411.1, C412.1, L401.2
- new net: C412.1, C415.1, C416.1, D404.1 (K), U401.16 (VCOM_PWR), U401.22 (PBKG), U401.26 (VN), U401.27 (VEE_IN), U401.4 (VNEG_IN), U401.49 (EP)
- new net: D404.2 (A), L402.1, U401.25 (VN_SW)
- new net: C407.1, D401.2 (A), D402.1 (K)
- new net: C402.2, D402.2 (A), U401.34 (VDDH_D)
- new net: C406.2, C408.2, D403.1 (K), U401.37 (VDDH_IN), U401.42 (VB), U401.43 (VPOS_IN)
- new net: D403.2 (A), L401.2, U401.40 (VB_SW)
- new net: C411.1, U401.28 (VEE_DRV)
- new net: C411.2, D405.2 (A), D406.1 (K)
- new net: C414.1, U401.1 (VREF)
- new net: C420.1, D405.1 (K), U401.30 (VEE_D)
- new net: R410.2, R411.1, U401.31 (VEE_FB)
- new net: C407.2, U401.36 (VDDH_DRV)
- new net: C413.1, U401.7 (INT_LDO)
- new net EPD_PWROK: U401.23 (PWR_GOOD)
- new net EPD_PWR_EN: U401.21 (PWRUP), U401.5 (WAKEUP)
- new net IPSOUT: C409.2, U401.10 (VIN)
- no-connect marks 10 -> 7
Other:
- note removed: "Split Ground plane, connect only via Pin 31 and EP"
- moved on the sheet: C302, C303, C304, C305, C306, C307, C308, J401, RN401, RN402, RN403, RN404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

Commit message: pcb: r0p6
Parts:
- removed C401, C403, C406, C408, C412, C416, C418, C421: 4.7uF/25V, Capacitor_SMD:C_0805_2012Metric, symbol Device:C
- removed C402, C420: 100nF, Capacitor_SMD:C_0402_1005Metric, symbol Device:C
- removed C404, C409, C413, C414, C415, C417, C419: 4.7uF, Capacitor_SMD:C_0603_1608Metric, symbol Device:C
- removed C405, C410: 10uF, Capacitor_SMD:C_0603_1608Metric, symbol Device:C
- removed C407, C411: 10nF, Capacitor_SMD:C_0402_1005Metric, symbol Device:C
- removed D401, D402, D403, D404, D405, D406: B0530WS, Diode_SMD:D_SOD-323, symbol Device:D_Schottky
- removed L401: FXL0420-2R2-M, footprints:L_FXL0420, symbol Device:L
- removed L402: FXL0420-4R7-M, footprints:L_FXL0420, symbol Device:L
- removed R402: 470K/1%, Resistor_SMD:R_0402_1005Metric, symbol Device:R
- removed R403: 18K/1%, Resistor_SMD:R_0402_1005Metric, symbol Device:R
- removed R404: 43K, Resistor_SMD:R_0402_1005Metric, symbol Device:R
- removed R410: 510K/1%, Resistor_SMD:R_0402_1005Metric, symbol Device:R
- removed R411: 24K/1%, Resistor_SMD:R_0402_1005Metric, symbol Device:R
- removed TH401: 10K, Resistor_SMD:R_0402_1005Metric, symbol Device:Thermistor_NTC
- removed U401: TPS65185, footprints:QFN-48-1EP_7x7mm_P0.5mm_EP4.1x4.1mm_ThermalVias, symbol symbols:TPS65185
- added C1: 100nF, Capacitor_SMD:C_0402_1005Metric, symbol Device:C
- added C10, C11, C3 (x5), C8, C9: 1uF/50V, Capacitor_SMD:C_0603_1608Metric, symbol Device:C
- added C2: 10uF, Capacitor_SMD:C_0603_1608Metric, symbol Device:C
- added C3, C4: 10nF, Capacitor_SMD:C_0402_1005Metric, symbol Device:C
- added C5: 22pF, Capacitor_SMD:C_0402_1005Metric, symbol Device:C
- added C7 (x4): 10uF/25V, Capacitor_SMD:C_0603_1608Metric, symbol Device:C
- added D1 (x2), D3: B0530WS, Diode_SMD:D_SOD-323, symbol Device:D
- added D2, D3, D4, D5 (x2): 4148WT, Diode_SMD:D_SOD-523, symbol Device:D
- added D6: EDZVT2R22B, Diode_SMD:D_SOD-323, symbol Device:D
- added D7: EDZVT2R20B, Diode_SMD:D_SOD-323, symbol Device:D
- added L1: WPN4020H2R2MT, Inductor_SMD:L_Changjiang_FNR4020S, symbol Device:L
- added L1 (x2): WPN4020H100MT, Inductor_SMD:L_Changjiang_FNR4020S, symbol Device:L
- added R1: 18K/1%, Resistor_SMD:R_0402_1005Metric, symbol Device:R
- added R1, R212 (x3): 120K/1%, Resistor_SMD:R_0402_1005Metric, symbol Device:R
- added R2 (x2): 5.1K/1%, Resistor_SMD:R_0402_1005Metric, symbol Device:R
- added R3, R4 (x2): 2K, Resistor_SMD:R_0402_1005Metric, symbol Device:R
- added R4: 0, Resistor_SMD:R_0402_1005Metric, symbol Device:R
- added U1: SX1308, Package_TO_SOT_SMD:SOT-23-6, symbol Regulator_Switching:MT3608
Connections:
- net +3V3_LCD is gone; now on net +3V3: C306.1, J401.11 (Pin_11), J401.5 (Pin_5)
- net +5V: now also C1.1, C2.1, L1.1, U1.5 (IN)
- net EPD_PWR_EN: now also U1.4 (EN)
- net GND: now also C1.2, C10.1, C11.2, C2.2, C3.1, C3.1, C3.2, C7.2, C7.2, C7.2, C7.2, C8.2, C9.1, D1.1 (K), D5.2 (A), D6.2 (A), D7.1 (K), L1.1, R2.2, R212.1, R212.1, R212.2, U1.2 (GND)
- net VCOM: now also C3.2, R1.2, R2.1
- net VGH: now also C11.1, D6.1 (K), R212.2, R3.2
- net VGL: now also C10.2, D3.2 (A), D7.2 (A), R212.1, R4.2
- net VNEG: now also C7.1, C7.1, D3.1 (K), L1.2, R1.1, R212.2, R4.1
- net VPOS: now also C5.2, C7.1, C7.1, D1.1 (K), R1.1, R4.1
- new net: C4.2, D4.1 (K), D5.2 (A)
- new net: C3.2, D4.2 (A), R4.2
- new net: C8.1, D5.1 (K), R3.1
- new net: C3.1, D2.1 (K), D3.2 (A)
- new net: C3.2, C3.2, C4.1, D1.2 (A), L1.2
- new net: C9.2, D2.2 (A), R4.1
- new net: C5.1, R1.2, R2.1, U1.3 (FB)
- new net: C3.1, D3.1 (K), R4.2
- new net: C3.1, C3.1, L1.2, U1.1 (SW)
- new net: C3.2, D1.2 (A), L1.1
- new net EPD_VCOM_PWM: D5.1 (K), R2.2
- no-connect marks 7 -> 6
Other:
- moved on the sheet: C302, C303, C304, C305, C306, C307, C308, J401, RN401, RN402, RN403, RN404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

Commit message: r0p7 wip, check in before switch to kicad 8
Parts:
- removed C10, C11, C3 (x5), C8, C9: 1uF/50V, Capacitor_SMD:C_0603_1608Metric, symbol Device:C
- removed C2: 10uF, Capacitor_SMD:C_0603_1608Metric, symbol Device:C
- removed C3, C4: 10nF, Capacitor_SMD:C_0402_1005Metric, symbol Device:C
- removed C302, C303, C304: 220nF, Capacitor_SMD:C_0402_1005Metric, symbol Device:C
- removed C5: 22pF, Capacitor_SMD:C_0402_1005Metric, symbol Device:C
- removed C7 (x4): 10uF/25V, Capacitor_SMD:C_0603_1608Metric, symbol Device:C
- removed D1 (x2), D3: B0530WS, Diode_SMD:D_SOD-323, symbol Device:D
- removed D2, D3, D4, D5 (x2): 4148WT, Diode_SMD:D_SOD-523, symbol Device:D
- removed D6: EDZVT2R22B, Diode_SMD:D_SOD-323, symbol Device:D
- removed D7: EDZVT2R20B, Diode_SMD:D_SOD-323, symbol Device:D
- removed L1: WPN4020H2R2MT, Inductor_SMD:L_Changjiang_FNR4020S, symbol Device:L
- removed L1 (x2): WPN4020H100MT, Inductor_SMD:L_Changjiang_FNR4020S, symbol Device:L
- removed R1: 18K/1%, Resistor_SMD:R_0402_1005Metric, symbol Device:R
- removed R1, R212 (x3): 120K/1%, Resistor_SMD:R_0402_1005Metric, symbol Device:R
- removed R2 (x2): 5.1K/1%, Resistor_SMD:R_0402_1005Metric, symbol Device:R
- removed R3, R4 (x2): 2K, Resistor_SMD:R_0402_1005Metric, symbol Device:R
- removed R4: 0, Resistor_SMD:R_0402_1005Metric, symbol Device:R
- removed U1: SX1308, Package_TO_SOT_SMD:SOT-23-6, symbol Regulator_Switching:MT3608
- added C3: 220nF, Capacitor_SMD:C_0402_1005Metric, symbol Device:C
- added C411 (x2), C437 (x2): 4.7uF/50V, Capacitor_SMD:C_0805_2012Metric, symbol Device:C
- added C415, C419 (x2): 100nF, Capacitor_SMD:C_0402_1005Metric, symbol Device:C
- added C418, C429, C436, C439, C440, C441: 47uF/10V, Capacitor_SMD:C_1206_3216Metric, symbol Device:C
- added C421 (x2), C433 (x2): 22pF, Capacitor_SMD:C_0402_1005Metric, symbol Device:C
- added C437 (x4): 10uF/50V, Capacitor_SMD:C_1206_3216Metric, symbol Device:C
- added C437 (x2): 10uF/10V, Capacitor_SMD:C_0805_2012Metric, symbol Device:C
- added C437: 1uF, Capacitor_SMD:C_0402_1005Metric, symbol Device:C
- added D1, D2, D3, D4, D6: 1N5819WS, Diode_SMD:D_SOD-323, symbol Diode:1N5819WS
- added D5 (x3): 4148WS, Diode_SMD:D_SOD-323, symbol Device:D
- added L404, L406: WPN4020H4R7MT, Inductor_SMD:L_Changjiang_FNR4020S, symbol Device:L
- added L404, L406: FTC201610S4R7MBCA, Inductor_SMD:L_Murata_DFE201610P, symbol Device:L
- added Q1, Q7, Q8: AO3401A, Package_TO_SOT_SMD:SOT-23, symbol Device:Q_PMOS_GSD
- added Q2: S8050, Package_TO_SOT_SMD:SOT-23, symbol Device:Q_NPN_BEC
- added Q6: AO3400A, Package_TO_SOT_SMD:SOT-23, symbol Device:Q_NMOS_GSD
- added R1, R419: 91K/1%, Resistor_SMD:R_0402_1005Metric, symbol Device:R
- added R2, R420: 27K/1%, Resistor_SMD:R_0402_1005Metric, symbol Device:R
- added R415: 360K/1%, Resistor_SMD:R_0402_1005Metric, symbol Device:R
- added R415, R419: 240K/1%, Resistor_SMD:R_0402_1005Metric, symbol Device:R
- added R416 (x2), R420 (x2), R423: 10K/1%, Resistor_SMD:R_0402_1005Metric, symbol Device:R
- added R419, R420 (x5): 120K/1%, Resistor_SMD:R_0402_1005Metric, symbol Device:R
- added R420 (x2): 51R, Resistor_SMD:R_0402_1005Metric, symbol Device:R
- added R420 (x2): 5.1K/1%, Resistor_SMD:R_0402_1005Metric, symbol Device:R
- added R420: 20K/1%, Resistor_SMD:R_0402_1005Metric, symbol Device:R
- added U11: LM321, Package_TO_SOT_SMD:SOT-23-5, symbol Amplifier_Operational:LM321
- added U403: MT9700, Package_TO_SOT_SMD:SOT-23-5, symbol symbols:MT9700
- added U404 (x2): LGS5148, Package_TO_SOT_SMD:TSOT-23-6, symbol symbols:SY8120
- added U7, U8: MT3608(SOT23-6), Package_TO_SOT_SMD:SOT-23-6, symbol symbols:MT3608(SOT23-6)
- C1: value 100nF -> 10uF/10V; footprint Capacitor_SMD:C_0402_1005Metric -> Capacitor_SMD:C_0805_2012Metric
- RN1: renamed from RN401; value 33 -> 33R / 4D02WGF330JTCE
- RN2: renamed from RN402; value 33 -> 33R / 4D02WGF330JTCE
- RN3: renamed from RN403; value 33 -> 33R / 4D02WGF330JTCE
- RN4: renamed from RN404; value 33 -> 33R / 4D02WGF330JTCE
- RN5: renamed from RN405; value 33 -> 33R / 4D02WGF330JTCE
- RN6: renamed from RN406; value 33 -> 33R / 4D02WGF330JTCE
- renumbered C305 to C60, C306 to C61, C307 to C62, C308 to C63, J401 to J3
Connections:
- net +3V3: now also Q7.2 (S), R420.1
- net +5V: now also Q1.2 (S), R419.2; no longer C1.1
- net EPD_PWR_EN: now also U403.4 (EN)
- net EPD_VCOM_PWM: now also D5.1 (K), R2.2
- net GND: now also C1.1, C3.1, C415.1, C418.1, C429.1, C433.2, C433.2, C436.1, C437.1, C437.1, C437.1, C437.1, C437.1, C437.1, C437.2, C437.2, C437.2, C439.1, C440.1, C441.1, D3.1 (K), D4.1 (K), D5.2 (A), L406.2, L406.2, Q2.2 (E), R416.1, R416.1, R419.2, R419.2, R420.1, R423.1, U11.5 (V+), U403.2 (GND), U7.2 (GND), U8.2 (GND); no longer C1.2
- net VCOM: now also C437.2, Q6.3 (D), R420.2
- net VGH: now also C421.2, C437.2, D2.1 (K), R415.2
- net VGL: now also C411.1, C437.1, D3.2 (A), D6.2 (A), R420.1, R420.1, U404.2 (GND)
- net VNEG: now also C411.1, C415.2, C437.1, C437.1, D4.2 (A), D6.1 (K), R1.1, R420.1, R420.1, R420.2, U11.2 (V-), U404.2 (GND)
- net VPOS: now also C421.2, C437.2, C437.2, D1.1 (K), R415.2
- new net: C419.1, L406.1, U404.6 (SW) (x2)
- new net: C419.2, U404.1 (BS) (x2)
- new net: Q7.1 (G), R420.2
- new net: Q2.1 (B), R420.2, R420.2
- new net: Q6.1 (G), Q7.3 (D), R420.1
- new net: C433.1, R419.1, R420.2, U404.3 (FB) (x2)
- new net: D1.2 (A), L404.2, U7.1 (SW)
- new net: D5.1 (K), R420.2 (x2)
- new net: Q1.1 (G), Q2.3 (C), R419.1
- new net: Q8.1 (G), R420.1
- new net: D5.2 (A), D5.2 (A), Q1.3 (D)
- new net: D2.2 (A), L404.2, U8.1 (SW)
- new net: C421.1, R415.1, R416.2, U8.3 (NFB)
- new net: C3.2, R1.2, R2.1, U11.1 (+)
- new net: Q6.2 (S), U11.3 (-), U11.4
- new net: Q8.3 (D), R420.1
- new net: C421.1, R415.1, R416.2, U7.3 (NFB)
- new net: R423.2, U403.3 (SET)
- new net +5V_EPD: C411.2, C411.2, C418.2, C429.2, C436.2, C437.2, C437.2, C439.2, C440.2, C441.2, L404.1, L404.1, R420.1, U403.1 (VOUT), U404.5 (IN), U404.5 (IN), U7.4 (~{SHDN}), U7.5 (VIN), U7.6 (NC), U8.4 (~{SHDN}), U8.5 (VIN), U8.6 (NC)
- new net EN_VGL: R420.1, R420.2, U404.4 (~{SHDN})
- new net EN_VNEG: R420.1, R420.2, U404.4 (~{SHDN})
- new net VBUS: C1.2, U403.5 (VIN)
- new net VCOM_EN: R420.1
- new net VCOM_MEA: Q8.2 (S), R420.2
- new net VCOM_MEA_EN: R420.2
Other:
- note added: "Ilim = 0.68A"
- note added: "Range: -0.89V ~ -3.43V"
- moved on the sheet: C60, C61, C62, C63, J3, RN1, RN2, RN3, RN4, RN5, RN6

Commit message: r0p7 wip
Parts:
- renumbered C1 to C104, C437 to C31, C437 to C32, C411 to C33, C411 to C34, C419 to C35, C419 to C36, C441 to C37, C433 to C38, C433 to C39, C421 to C40, C421 to C41, C440 to C42, C437 to C43, C437 to C44, C439 to C45, C437 to C46, C437 to C47, C437 to C48, C436 to C49, C437 to C50, C429 to C51, C418 to C53, C415 to C54, C437 to C56, L404 to L4, L404 to L5, L406 to L6, L406 to L7, R423 to R17, R419 to R18, R420 to R19, R419 to R20, R420 to R21, R415 to R22, R416 to R23, R415 to R24, R416 to R25, R419 to R28, R420 to R29, R420 to R30, R420 to R31, R420 to R32, R420 to R33, R420 to R34, R420 to R62, R420 to R63, R420 to R64, R420 to R65, R420 to R66, U404 to U10, U403 to U6, U404 to U9

Commit message: r0p7 layout done
Connections:
- net +5V is gone; now on net +5V_EPD: Q1.2 (S), R28.2
Changed lines of the file:
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@@
 	)
 	(symbol
-		(lib_id "power:+5V")
-		(at 129.54 127 0)
-		(unit 1)
-		(exclude_from_sim no)
-		(in_bom yes)
-		(on_board yes)
-		(dnp no)
-		(fields_autoplaced yes)
-		(property "Reference" "#PWR074"
-			(at 129.54 130.81 0)
-			(effects
-				(font
-					(size 1.27 1.27)
-				)
-				(hide yes)
-			)
-		)
-		(property "Value" "+5V"
-			(at 129.54 121.92 0)
-			(effects
-				(font
-					(size 1.27 1.27)
-				)
-			)
-		)
-		(property "Footprint" ""
-			(at 129.54 127 0)
-			(effects
-				(font
-					(size 1.27 1.27)
-				)
-				(hide yes)
-			)
-		)
-		(property "Datasheet" ""
-			(at 129.54 127 0)
-			(effects
-				(font
-					(size 1.27 1.27)
-				)
-				(hide yes)
-			)
-		)
-		(property "Description" ""
-			(at 129.54 127 0)
-			(effects
-				(font
-					(size 1.27 1.27)
-				)
-				(hide yes)
-			)
-		)
-		(pin "1"
-		)
-		(instances
-			(project "pcb"
-				(path "/4654897e-3e2f-4522-96c3-20b19803c088/b1d5941d-0481-47a2-a434-0b8e587a166a"
-					(reference "#PWR074")
-					(unit 1)
-				)
-			)
-		)
-	)
-	(symbol
 		(lib_id "Device:C")
 		(at 251.46 143.51 0)
@@
 					(unit 1)
 				)
+			)
+		)
+	)
+	(symbol
+		(lib_id "symbols:+5V_EPD")
+		(at 129.54 127 0)
+		(unit 1)
+		(exclude_from_sim no)
+		(in_bom yes)
+		(on_board yes)
+		(dnp no)
+		(fields_autoplaced yes)
+		(property "Reference" "#PWR048"
+			(at 129.54 130.81 0)
+			(effects
+				(font
+					(size 1.27 1.27)
+				)
+				(hide yes)
+			)
+		)
+		(property "Value" "+5V_EPD"
+			(at 129.54 121.92 0)
+			(effects
+				(font
+					(size 1.27 1.27)
+				)
+			)
+		)
+		(property "Footprint" ""
+			(at 129.54 127 0)
+			(effects
+				(font
+					(size 1.27 1.27)
+				)
+				(hide yes)
+			)
+		)
+		(property "Datasheet" ""
+			(at 129.54 127 0)
+			(effects
+				(font
+					(size 1.27 1.27)
+				)
+				(hide yes)
+			)
+		)
+		(property "Description" ""
+			(at 129.54 127 0)
+			(effects
+				(font
+					(size 1.27 1.27)
+				)
+				(hide yes)
+			)
+		)
+		(pin "1"
+		)
+		(instances
+			(project "pcb"
+				(path "/4654897e-3e2f-4522-96c3-20b19803c088/b1d5941d-0481-47a2-a434-0b8e587a166a"
+					(reference "#PWR048")
+					(unit 1)
+				)

Commit message: Bug fixes and changes for r0p8
Parts:
- added J4: SM03B-SRSS-TB, Connector_JST:JST_SH_SM03B-SRSS-TB_1x03-1MP_P1.00mm_Horizontal, symbol Connector_Generic_MountingPin:Conn_01x03_MountingPin
Connections:
- net GND: now also J4.2 (Pin_2), J4.MP (MountPin)
- net VBUS: now also J4.1 (Pin_1)
- new net FL_PWM: J4.3 (Pin_3)
Other:
- company: Copyright 2022 Modos / Engineer: Wenting Zhang -> Copyright 2024 Wenting Zhang
- title: Caster EPDC -> Glider
