File: pcb/mainboard/eink.kicad_sch (KiCad schematic)
At the start: 84 parts, among them J3 FH12-40S-0.5SH, J4 SM03B-SRSS-TB, Q1 AO3401A, Q2 S8050, Q6 AO3400A, Q7 AO3401A, Q8 AO3401A, U10 LGS5148, U11 LM321, U6 MT9700, U7 MT3608(SOT23-6), U8 MT3608(SOT23-6), U9 LGS5148

Commit message: BOM adjustments
Parts:
- C37, C42, C45, C49, C51, C53: LCSC C105490 -> (none)
- C38, C39, C40, C41: value 22pF -> 18pF
- C60, C61, C62, C63: LCSC C880414 -> (none)
- D1, D2, D3, D4, D6: value 1N5819WS -> B0530WS
- D5: value 4148WS -> B0530WS
- R21, R29: value 5.1K/1% -> 5.1K
Changed lines of the file:
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@@
 			)
 		)
-		(property "Value" "5.1K/1%"
+		(property "Value" "5.1K"
 			(at 157.48 149.86 0)
 			(effects
@@
 			)
 		)
-		(property "LCSC" "C105490"
+		(property "LCSC" ""
 			(at 149.86 41.91 0)
 			(effects
@@
 			)
 		)
-		(property "LCSC" "C880414"
+		(property "LCSC" ""
 			(at 259.08 143.51 0)
 			(effects
@@
 			)
 		)
-		(property "LCSC" "C105490"
+		(property "LCSC" ""
 			(at 73.66 41.91 0)
 			(effects
@@
 			)
 		)
-		(property "LCSC" "C880414"
+		(property "LCSC" ""
 			(at 251.46 143.51 0)
 			(effects
@@
 			)
 		)
-		(property "Value" "1N5819WS"
+		(property "Value" "B0530WS"
 			(at 96.52 177.8 90)
 			(effects
@@
 			)
 		)
-		(property "Datasheet" "https://datasheet.lcsc.com/lcsc/2204281430_Guangdong-Hottech-1N5819WS_C191023.pdf"
+		(property "Datasheet" ""
 			(at 93.98 176.53 0)
 			(effects
@@
 			)
 		)
-		(property "Value" "4148WS"
+		(property "Value" "B0530WS"
 			(at 157.48 121.92 0)
 			(effects
@@
 			)
 		)
-		(property "Datasheet" "~"
+		(property "Datasheet" ""
 			(at 156.21 124.46 0)
 			(effects
@@
 			)
 		)
-		(property "Value" "4148WS"
+		(property "Value" "B0530WS"
 			(at 157.48 132.08 0)
 			(effects
@@
 			)
 		)
-		(property "Datasheet" "~"
+		(property "Datasheet" ""
 			(at 156.21 134.62 0)
 			(effects
@@
 			)
 		)
-		(property "Value" "1N5819WS"
+		(property "Value" "B0530WS"
 			(at 70.1675 67.31 0)
 			(effects
@@
 			)
 		)
-		(property "Datasheet" "https://datasheet.lcsc.com/lcsc/2204281430_Guangdong-Hottech-1N5819WS_C191023.pdf"
+		(property "Datasheet" ""
 			(at 69.85 71.12 0)
 			(effects
@@
 			)
 		)
-		(property "Value" "22pF"
+		(property "Value" "18pF"
 			(at 91.44 111.76 0)
 			(effects
@@
 			)
 		)
-		(property "LCSC" "C105490"
+		(property "LCSC" ""
 			(at 134.62 41.91 0)
 			(effects
@@
 			)
 		)
-		(property "Value" "22pF"
+		(property "Value" "18pF"
 			(at 88.9 142.24 0)
 			(effects
@@
 			)
 		)
-		(property "Value" "1N5819WS"
+		(property "Value" "B0530WS"
 			(at 70.1675 100.33 0)
 			(effects
@@
 			)
 		)
-		(property "Datasheet" "https://datasheet.lcsc.com/lcsc/2204281430_Guangdong-Hottech-1N5819WS_C191023.pdf"
+		(property "Datasheet" ""
 			(at 69.85 104.14 0)
 			(effects
@@
 			)
 		)
-		(property "Value" "1N5819WS"
+		(property "Value" "B0530WS"
 			(at 144.78 173.6725 90)
 			(effects
@@
 			)
 		)
-		(property "Datasheet" "https://datasheet.lcsc.com/lcsc/2204281430_Guangdong-Hottech-1N5819WS_C191023.pdf"
+		(property "Datasheet" ""
 			(at 142.24 172.72 0)
 			(effects
@@
 			)
 		)
-		(property "Value" "4148WS"
+		(property "Value" "B0530WS"
 			(at 127 109.855 90)
 			(effects
@@
 			)
 		)
-		(property "Datasheet" "~"
+		(property "Datasheet" ""
 			(at 124.46 107.95 0)
 			(effects
@@
 			)
 		)
-		(property "LCSC" "C105490"
+		(property "LCSC" ""
 			(at 119.38 41.91 0)
 			(effects
@@
 			)
 		)
-		(property "Value" "22pF"
+		(property "Value" "18pF"
 			(at 88.9 170.18 0)
 			(effects
@@
 			)
 		)
-		(property "LCSC" "C880414"
+		(property "LCSC" ""
 			(at 256.54 143.51 0)
 			(effects
@@
 			)
 		)
-		(property "Value" "1N5819WS"
+		(property "Value" "B0530WS"
 			(at 96.52 149.5425 90)
 			(effects
@@
 			)
 		)
-		(property "Datasheet" "https://datasheet.lcsc.com/lcsc/2204281430_Guangdong-Hottech-1N5819WS_C191023.pdf"
+		(property "Datasheet" ""
 			(at 93.98 148.59 0)
 			(effects
@@
 			)
 		)
-		(property "LCSC" "C105490"
+		(property "LCSC" ""
 			(at 104.14 41.91 0)
 			(effects
@@
 			)
 		)
-		(property "LCSC" "C105490"
+		(property "LCSC" ""
 			(at 88.9 41.91 0)
 			(effects
@@
 			)
 		)
-		(property "Value" "22pF"
+		(property "Value" "18pF"
 			(at 91.44 78.74 0)
 			(effects
@@
 			)
 		)
-		(property "Value" "5.1K/1%"
+		(property "Value" "5.1K"
 			(at 78.74 177.8 0)
 			(effects
@@
 			)
 		)
-		(property "LCSC" "C880414"
+		(property "LCSC" ""
 			(at 254 143.51 0)
 			(effects
