File: pcb/mainboard/fpga.kicad_sch (KiCad schematic)
At the start: 29 parts, among them J201 Conn_02x05_Odd_Even, U200 XC6SLX16-FTG256, U202 W25X16JVP, Y201 24MHz

Commit message: pcb: r0p4
Parts:
- removed C212: 220nF, Capacitor_SMD:C_0402_1005Metric, symbol Device:C
- removed D306: LED, LED_SMD:LED_0603_1608Metric, symbol Device:LED
- removed R203: 49.9K/1%, Resistor_SMD:R_0402_1005Metric, symbol Device:R
- removed R303: 1K, Resistor_SMD:R_0402_1005Metric, symbol Device:R
- removed R304, R305: 4.7K, Resistor_SMD:R_0402_1005Metric, symbol Device:R
- removed U202: W25X16JVP, Package_SON:WSON-8-1EP_6x5mm_P1.27mm_EP3.4x4.3mm, symbol Memory_Flash:W25Q32JVZP
- U200: footprint Package_BGA:Xilinx_FTG256 -> footprints:Xilinx_FTG256
Connections:
- net GCLK: no longer U200.E8 (IO_L36N_GCLK14_0)
- net LVDS_ODD_CKN: now also U200.A9 (IO_L34N_GCLK18_0); no longer U200.A8 (IO_L33N_0)
- net LVDS_ODD_CKP: now also U200.C9 (IO_L34P_GCLK19_0); no longer U200.B8 (IO_L33P_0)
- net DDC_SCL: no longer names the net of U200.D11 (IO_L66P_SCP1_0)
- net DDC_SDA: no longer names the net of U200.D12 (IO_L66N_SCP0_0)
- net LVDS_EVEN_CKN: no longer names the net of U200.A13 (IO_L63N_SCP6_0)
- net LVDS_EVEN_CKP: no longer names the net of U200.C13 (IO_L63P_SCP7_0)
- net LVDS_EVEN_DN: no longer names the net of U200.D9 (IO_L40N_0)
- net LVDS_EVEN_DP: no longer names the net of U200.F9 (IO_L40P_0)
- net LVDS_ODD_DN: no longer names the net of U200.C8 (IO_L38N_VREF_0)
- net LVDS_ODD_DP: no longer names the net of U200.D8 (IO_L38P_0)
Other:
- company: Copyright 2021 Modos / Engineer: Wenting Zhang -> Copyright 2022 Modos / Engineer: Wenting Zhang
- moved on the sheet: C210, C213, C215, C217, C219, C220, R306

Commit message: pcb: r0p5
Parts:
- R201: value 22R -> 27
- Y201: value 24MHz -> 33MHz
Changed lines of the file:
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@@
       (effects (font (size 1.27 1.27)) (justify left))
     )
-    (property "Value" "24MHz" (id 1) (at 243.84 31.75 0)
+    (property "Value" "33MHz" (id 1) (at 243.84 31.75 0)
       (effects (font (size 1.27 1.27)) (justify left))
     )
@@
     (in_bom yes) (on_board yes)
     (property "Reference" "R201" (id 0) (at 224.79 36.83 90))
-    (property "Value" "22R" (id 1) (at 234.95 36.83 90))
+    (property "Value" "27" (id 1) (at 234.95 36.83 90))
     (property "Footprint" "Resistor_SMD:R_0402_1005Metric" (id 2) (at 229.87 39.878 90)
       (effects (font (size 1.27 1.27)) hide)

Commit message: pcb: r0p6
Parts:
- removed C210, C211, C213, C214, C215, C217, C219: 220nF, Capacitor_SMD:C_0402_1005Metric, symbol Device:C
- removed C220: 22uF, Capacitor_SMD:C_0603_1608Metric, symbol Device:C

Commit message: r0p7 wip, check in before switch to kicad 8
Parts:
- added R15: 1K/1%, Resistor_SMD:R_0402_1005Metric, symbol Device:R
- J2: renamed from J201; value Conn_02x05_Odd_Even -> DNP
- R11: renamed from R201; value 27 -> 27R
- renumbered C201 to C26, C203 to C27, C204 to C28, C202 to C29, C209 to C30, R310 to R10, R202 to R12, R306 to R13, R309 to R14, R209 to R16, U200 to U5, Y201 to Y1
Connections:
- net +3V3: now also R15.1
- net FPGA_DONE: now also R15.2
- net LVDS_EVEN_AN: no longer U5.A10 (IO_L35N_GCLK16_0)
- net LVDS_EVEN_AP: no longer U5.B10 (IO_L35P_GCLK17_0)
- net LVDS_EVEN_BN: no longer U5.A11 (IO_L39N_0)
- net LVDS_EVEN_BP: no longer U5.C11 (IO_L39P_0)
- net LVDS_EVEN_CN: no longer U5.A12 (IO_L62N_VREF_0)
- net LVDS_EVEN_CP: no longer U5.B12 (IO_L62P_0)
- net LVDS_ODD_AN: no longer U5.A5 (IO_L2N_0)
- net LVDS_ODD_AP: no longer U5.B5 (IO_L2P_0)
- net LVDS_ODD_BN: no longer U5.A6 (IO_L4N_0)
- net LVDS_ODD_BP: no longer U5.B6 (IO_L4P_0)
- net LVDS_ODD_CKN: no longer U5.A9 (IO_L34N_GCLK18_0)
- net LVDS_ODD_CKP: no longer U5.C9 (IO_L34P_GCLK19_0)
- net LVDS_ODD_CN: no longer U5.C6 (IO_L7N_0)
- net LVDS_ODD_CP: no longer U5.D6 (IO_L7P_0)
- net VIN_HPD: now reaches U5.A14 (IO_L65N_SCP2_0)
- net TMDS_CKP: now reaches U5.C10 (IO_L37N_GCLK12_0)
- net TMDS_CKN: now reaches U5.E10 (IO_L37P_GCLK13_0)
- new net TMDS_D0N: U5.C9 (IO_L34P_GCLK19_0)
- new net TMDS_D0P: U5.A9 (IO_L34N_GCLK18_0)
- new net TMDS_D1N: U5.D6 (IO_L7P_0)
- new net TMDS_D1P: U5.C6 (IO_L7N_0)
- new net TMDS_D2N: U5.B6 (IO_L4P_0)
- new net TMDS_D2P: U5.A6 (IO_L4N_0)

Commit message: r0p7 wip
Parts:
- removed R10: 4.7K, Resistor_SMD:R_0402_1005Metric, symbol Device:R
Connections:
- net EPDC_D10: now also U5.K14 (IO_L41N_GCLK8_M1CASN_1); no longer U5.J14 (IO_L43P_GCLK5_M1DQ4_1)
- net LVDS_EVEN_AN: now also U5.E8 (IO_L36N_GCLK14_0)
- net LVDS_EVEN_AP: now also U5.E7 (IO_L36P_GCLK15_0)
- net LVDS_EVEN_BN: now also U5.D9 (IO_L40N_0)
- net LVDS_EVEN_BP: now also U5.F9 (IO_L40P_0)
- net LVDS_EVEN_CN: now also U5.A13 (IO_L63N_SCP6_0)
- net LVDS_EVEN_CP: now also U5.C13 (IO_L63P_SCP7_0)
- net LVDS_ODD_AN: now also U5.C5 (IO_L3N_0)
- net LVDS_ODD_AP: now also U5.D5 (IO_L3P_0)
- net LVDS_ODD_BN: now also U5.E6 (IO_L5N_0)
- net LVDS_ODD_BP: now also U5.F7 (IO_L5P_0)
- net LVDS_ODD_CKN: now also U5.A10 (IO_L35N_GCLK16_0)
- net LVDS_ODD_CKP: now also U5.B10 (IO_L35P_GCLK17_0)
- net LVDS_ODD_CN: now also U5.A8 (IO_L33N_0)
- net LVDS_ODD_CP: now also U5.B8 (IO_L33P_0)
- net DPI_R5: now reaches U5.B15 (IO_L29P_A23_M1A13_1)
- net DPI_R4: now reaches U5.B16 (IO_L29N_A22_M1A14_1)
- net DPI_R3: now reaches U5.C15 (IO_L33P_A15_M1A10_1)
- net DPI_R2: now reaches U5.C16 (IO_L33N_A14_M1A4_1)
- net DPI_R6: now reaches U5.D14 (IO_L31P_A19_M1CKE_1)
- net DPI_G3: now reaches U5.D16 (IO_L31N_A18_M1A12_1)
- net DPI_R7: now reaches U5.E12 (IO_L1N_A24_VREF_1)
- net DPI_R1: now reaches U5.E13 (IO_L1P_A25_1)
- net DPI_G2: now reaches U5.E15 (IO_L34P_A13_M1WE_1)
- net DPI_G1: now reaches U5.E16 (IO_L34N_A12_M1BA2_1)
- net DPI_G6: now reaches U5.F12 (IO_L30P_A21_M1RESET_1)
- net DPI_R0: now reaches U5.F13 (IO_L32P_A17_M1A8_1)
- net DPI_G7: now reaches U5.F14 (IO_L32N_A16_M1A9_1)
- net DPI_G0: now reaches U5.F15 (IO_L35P_A11_M1A7_1)
- net DPI_B7: now reaches U5.F16 (IO_L35N_A10_M1A2_1)
- net DPI_B6: now reaches U5.G11 (IO_L30N_A20_M1A11_1)
- net DPI_G4: now reaches U5.G12 (IO_L38P_A5_M1CLK_1)
- net DPI_G5: now reaches U5.G14 (IO_L36P_A9_M1BA0_1)
- net DPI_B2: now reaches U5.H11 (IO_L38N_A4_M1CLKN_1)
- net DPI_B3: now reaches U5.H13 (IO_L39P_M1A3_1)
- net DPI_B5: now reaches U5.H14 (IO_L39N_M1ODT_1)
- net DPI_B4: now reaches U5.H15 (IO_L37P_A7_M1A0_1)
- net DPI_HS: now reaches U5.J11 (IO_L40P_GCLK11_M1A5_1)
- net DPI_DE: now reaches U5.J12 (IO_L40N_GCLK10_M1A6_1)
- net DPI_B0: now reaches U5.J13 (IO_L41P_GCLK9_IRDY1_M1RASN_1)
- net DPI_PCLK: now reaches U5.K11 (IO_L42N_GCLK6_TRDY1_M1LDM_1)
- net DPI_VS: now reaches U5.K12 (IO_L42P_GCLK7_M1UDM_1)
- net TMDS_CKN: no longer names the net of U5.E10 (IO_L37P_GCLK13_0)
- net TMDS_CKP: no longer names the net of U5.C10 (IO_L37N_GCLK12_0)
- net TMDS_D0N: no longer names the net of U5.C9 (IO_L34P_GCLK19_0)
- net TMDS_D0P: no longer names the net of U5.A9 (IO_L34N_GCLK18_0)
- net TMDS_D1N: no longer names the net of U5.D6 (IO_L7P_0)
- net TMDS_D1P: no longer names the net of U5.C6 (IO_L7N_0)
- net TMDS_D2N: no longer names the net of U5.B6 (IO_L4P_0)
- net TMDS_D2P: no longer names the net of U5.A6 (IO_L4N_0)
- new net DPI_B1: U5.J14 (IO_L43P_GCLK5_M1DQ4_1)

Commit message: r0p7 layout done
Parts:
- removed J2: DNP, Connector_PinHeader_1.27mm:PinHeader_2x05_P1.27mm_Vertical_SMD, symbol Connector_Generic:Conn_02x05_Odd_Even
- removed R16: 4.7K, Resistor_SMD:R_0402_1005Metric, symbol Device:R
- added C140, C141, C146, C149, C67: 470nF, Capacitor_SMD:C_0402_1005Metric, symbol Device:C
- added C142, C143, C145, C147, C64, C65: 47uF/6.3V, Capacitor_SMD:C_0603_1608Metric, symbol Device:C
- added C144, C148, C66: 4.7uF, Capacitor_SMD:C_0402_1005Metric, symbol Device:C
- C26, C27: value 220nF -> 47uF/6.3V; footprint Capacitor_SMD:C_0402_1005Metric -> Capacitor_SMD:C_0603_1608Metric
- C28: value 220nF -> 4.7uF
- C29: value 220nF -> 470nF
Connections:
- net VIN_HPD is gone; now on net LVDS_EVEN_CN: U5.A14 (IO_L65N_SCP2_0)
- net +3V3: now also C141.1, C142.1, C143.1, C144.1, C145.1, C146.1, C147.1, C148.1, C149.1
- net GND: now also C140.2, C141.2, C142.2, C143.2, C144.2, C145.2, C146.2, C147.2, C148.2, C149.2, C64.2, C65.2, C66.2, C67.2
- net LVDS_EVEN_AN: now also U5.D11 (IO_L66P_SCP1_0); no longer U5.E8 (IO_L36N_GCLK14_0)
- net LVDS_EVEN_AP: now also U5.D12 (IO_L66N_SCP0_0); no longer U5.E7 (IO_L36P_GCLK15_0)
- net LVDS_EVEN_BN: now also U5.C13 (IO_L63P_SCP7_0); no longer U5.D9 (IO_L40N_0)
- net LVDS_EVEN_BP: now also U5.A13 (IO_L63N_SCP6_0); no longer U5.F9 (IO_L40P_0)
- net LVDS_EVEN_CN: no longer U5.A13 (IO_L63N_SCP6_0)
- net LVDS_EVEN_CP: now also U5.B14 (IO_L65P_SCP3_0); no longer U5.C13 (IO_L63P_SCP7_0)
- net LVDS_ODD_AN: now also U5.E7 (IO_L36P_GCLK15_0); no longer U5.C5 (IO_L3N_0)
- net LVDS_ODD_AP: now also U5.E8 (IO_L36N_GCLK14_0); no longer U5.D5 (IO_L3P_0)
- net LVDS_ODD_BN: now also U5.B8 (IO_L33P_0); no longer U5.E6 (IO_L5N_0)
- net LVDS_ODD_BP: now also U5.A8 (IO_L33N_0); no longer U5.F7 (IO_L5P_0)
- net LVDS_ODD_CKN: now also U5.B10 (IO_L35P_GCLK17_0); no longer U5.A10 (IO_L35N_GCLK16_0)
- net LVDS_ODD_CKP: now also U5.A10 (IO_L35N_GCLK16_0); no longer U5.B10 (IO_L35P_GCLK17_0)
- net LVDS_ODD_CN: now also U5.D9 (IO_L40N_0); no longer U5.A8 (IO_L33N_0)
- net LVDS_ODD_CP: now also U5.F9 (IO_L40P_0); no longer U5.B8 (IO_L33P_0)
- new net +1V35: C140.1, C64.1, C65.1, C66.1, C67.1
- no-connect marks 3 -> 11
Other:
- note added: "VCCO0"
- note added: "VCCO1"
- note added: "VCCO2"
- note added: "VCCO3"
- moved on the sheet: R13, R14, R15, U5C

Commit message: Bug fixes and changes for r0p8
Other:
- company: Copyright 2022 Modos / Engineer: Wenting Zhang -> Copyright 2024 Wenting Zhang
- title: Caster EPDC -> Glider
Changed lines of the file:
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@@
 	(paper "A4")
 	(title_block
-		(title "Caster EPDC")
-		(date "2022-07-03")
-		(rev "R0.4")
-		(company "Copyright 2022 Modos / Engineer: Wenting Zhang")
+		(title "Glider")
+		(date "2024-05-09")
+		(rev "R0.8")
+		(company "Copyright 2024 Wenting Zhang")
 	)
 	(junction
