File: pcb/mainboard/fpga.kicad_sch (KiCad schematic)
At the start: 26 parts, among them U5 XC6SLX16-FTG256, Y1 33MHz

Commit message: BOM adjustments
Parts:
- C140, C141, C142, C143, C144, C145, C146, C147, C148, C149, C26, C27, C28, C29, C30, C64, C65, C66, C67: LCSC C880414 -> (none)
- R11: LCSC C93929 -> (none)
- R12, R13, R14: value 4.7K -> 5.1K; LCSC C105870 -> (none)
- R15: LCSC C105870 -> (none)
- U5: LCSC C39313 -> (none)
- Y1: LCSC C252339 -> (none)
Changed lines of the file:
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@@
 			)
 		)
-		(property "LCSC" "C880414"
+		(property "LCSC" ""
 			(at 264.16 34.29 0)
 			(effects
@@
 			)
 		)
-		(property "Value" "4.7K"
+		(property "Value" "5.1K"
 			(at 260.35 68.58 0)
 			(effects
@@
 			)
 		)
-		(property "LCSC" "C105870"
+		(property "LCSC" ""
 			(at 256.54 67.31 0)
 			(effects
@@
 			)
 		)
-		(property "LCSC" "C880414"
+		(property "LCSC" ""
 			(at 220.98 102.87 0)
 			(effects
@@
 			)
 		)
-		(property "LCSC" "C880414"
+		(property "LCSC" ""
 			(at 170.18 118.11 0)
 			(effects
@@
 			)
 		)
-		(property "LCSC" "C880414"
+		(property "LCSC" ""
 			(at 195.58 102.87 0)
 			(effects
@@
 			)
 		)
-		(property "Value" "4.7K"
+		(property "Value" "5.1K"
 			(at 260.35 86.36 0)
 			(effects
@@
 			)
 		)
-		(property "LCSC" "C105870"
+		(property "LCSC" ""
 			(at 256.54 85.09 0)
 			(effects
@@
 			)
 		)
-		(property "LCSC" "C880414"
+		(property "LCSC" ""
 			(at 195.58 118.11 0)
 			(effects
@@
 			)
 		)
-		(property "LCSC" "C880414"
+		(property "LCSC" ""
 			(at 182.88 118.11 0)
 			(effects
@@
 			)
 		)
-		(property "LCSC" "C880414"
+		(property "LCSC" ""
 			(at 220.98 133.35 0)
 			(effects
@@
 			)
 		)
-		(property "LCSC" "C880414"
+		(property "LCSC" ""
 			(at 170.18 133.35 0)
 			(effects
@@
 			)
 		)
-		(property "LCSC" "C880414"
+		(property "LCSC" ""
 			(at 208.28 102.87 0)
 			(effects
@@
 			)
 		)
-		(property "LCSC" "C880414"
+		(property "LCSC" ""
 			(at 208.28 133.35 0)
 			(effects
@@
 			)
 		)
-		(property "LCSC" "C880414"
+		(property "LCSC" ""
 			(at 208.28 118.11 0)
 			(effects
@@
 			)
 		)
-		(property "LCSC" "C39313"
+		(property "LCSC" ""
 			(at 91.44 104.14 0)
 			(effects
@@
 			)
 		)
-		(property "LCSC" "C880414"
+		(property "LCSC" ""
 			(at 208.28 148.59 0)
 			(effects
@@
 			)
 		)
-		(property "LCSC" "C39313"
+		(property "LCSC" ""
 			(at 201.93 73.66 0)
 			(effects
@@
 			)
 		)
-		(property "LCSC" "C880414"
+		(property "LCSC" ""
 			(at 182.88 102.87 0)
 			(effects
@@
 			)
 		)
-		(property "LCSC" "C880414"
+		(property "LCSC" ""
 			(at 170.18 102.87 0)
 			(effects
@@
 			)
 		)
-		(property "LCSC" "C880414"
+		(property "LCSC" ""
 			(at 195.58 133.35 0)
 			(effects
@@
 			)
 		)
-		(property "LCSC" "C880414"
+		(property "LCSC" ""
 			(at 195.58 148.59 0)
 			(effects
@@
 			)
 		)
-		(property "LCSC" "C880414"
+		(property "LCSC" ""
 			(at 182.88 148.59 0)
 			(effects
@@
 			)
 		)
-		(property "LCSC" "C105870"
+		(property "LCSC" ""
 			(at 264.16 67.31 0)
 			(effects
@@
 			)
 		)
-		(property "Value" "4.7K"
+		(property "Value" "5.1K"
 			(at 257.81 35.56 0)
 			(effects
@@
 			)
 		)
-		(property "LCSC" "C105870"
+		(property "LCSC" ""
 			(at 254 34.29 0)
 			(effects
@@
 			)
 		)
-		(property "LCSC" "C252339"
+		(property "LCSC" ""
 			(at 246.38 38.1 0)
 			(effects
@@
 			)
 		)
-		(property "LCSC" "C880414"
+		(property "LCSC" ""
 			(at 182.88 133.35 0)
 			(effects
@@
 			)
 		)
-		(property "LCSC" "C880414"
+		(property "LCSC" ""
 			(at 170.18 148.59 0)
 			(effects
@@
 			)
 		)
-		(property "LCSC" "C93929"
+		(property "LCSC" ""
 			(at 229.87 38.1 0)
 			(effects

Commit message: R0P9 PCB WIP
Connections:
- no-connect marks 11 -> 1
Other:
- moved on the sheet: C30, R11, R12, R13, R15, Y1

Commit message: PCB r0p9
Parts:
- removed U5: XC6SLX16-FTG256, footprints:Xilinx_FTG256, symbol FPGA_Xilinx_Spartan6:XC6SLX16-FTG256
