File: pcb/mainboard/fpga_ddr.kicad_sch (KiCad schematic)
At the start: 39 parts, among them U200 XC6SLX16-FTG256, U502 MT41K64M16TW

Commit message: pcb: r0p4
Parts:
- removed R511: 4.7K, Resistor_SMD:R_0402_1005Metric, symbol Device:R
- R509, R510: value 4.7K -> 0
- U200: footprint Package_BGA:Xilinx_FTG256 -> footprints:Xilinx_FTG256
Connections:
- net GND: no longer U200.N11 (IO_L13P_M1_2)
- net FPGA_CS: now reaches U200.L10 (IO_L16P_2)
- net GCLK: now reaches U200.N8 (IO_L29N_GCLK2_2)
- net EPD_PWR_SCL: no longer names the net of U200.R9 (IO_L23P_2)
- net EPD_PWR_SDA: no longer names the net of R510.2
- net EPD_PWR_SDA: now also U200.N11 (IO_L13P_M1_2); no longer U200.T9 (IO_L23N_2)
- net FPGA_FCCLK renamed FPGA_SCLK
- net FPGA_FCS: no longer names the net of U200.T3 (IO_L65N_CSO_B_2)
- net FPGA_FMISO renamed FPGA_MOSI
- net FPGA_FMOSI renamed FPGA_MISO
Other:
- company: Copyright 2021 Modos / Engineer: Wenting Zhang -> Copyright 2022 Modos / Engineer: Wenting Zhang
- moved on the sheet: C509, C512, R501, R502, R506, R507, R508, U502

Commit message: pcb: r0p5
Parts:
- removed TP501: TestPoint, TestPoint:TestPoint_Pad_D1.0mm, symbol Connector:TestPoint
Connections:
- no-connect marks 2 -> 3
Changed lines of the file:
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@@
   (no_connect (at 208.28 40.64))
   (no_connect (at 137.16 50.8))
+  (no_connect (at 26.67 137.16))
   (wire (pts (xy 219.71 134.62) (xy 209.55 134.62))
     (stroke (width 0) (type solid) (color 0 0 0 0))
@@
     (pin "2")
   )
-  (symbol (lib_id "Connector:TestPoint") (at 26.67 137.16 90) (unit 1)
-    (in_bom yes) (on_board yes) (fields_autoplaced)
-    (property "Reference" "TP501" (id 0) (at 24.638 130.81 90))
-    (property "Value" "TestPoint" (id 1) (at 24.638 133.35 90))
-    (property "Footprint" "TestPoint:TestPoint_Pad_D1.0mm" (id 2) (at 26.67 132.08 0)
-      (effects (font (size 1.27 1.27)) hide)
-    )
-    (property "Datasheet" "~" (id 3) (at 26.67 132.08 0)
-      (effects (font (size 1.27 1.27)) hide)
-    )
-    (property "LCSC" "-" (id 4) (at 26.67 137.16 0)
-      (effects (font (size 1.27 1.27)) hide)
-    )
-    (property "Ref.Price" "0" (id 5) (at 26.67 137.16 0)
-      (effects (font (size 1.27 1.27)) hide)
-    )
-    (pin "1")
-  )
   (symbol (lib_id "Device:C") (at 245.11 146.05 0) (unit 1)

Commit message: r0p7 wip, check in before switch to kicad 8
Parts:
- C86: renamed from C525; value 10uF -> 10uF/10V; footprint Capacitor_SMD:C_0603_1608Metric -> Capacitor_SMD:C_0805_2012Metric
- R35: renamed from R509; value 0 -> 0R
- R36: renamed from R510; value 0 -> 0R
- R37: renamed from R505; value 100R 1% -> 100R/1%
- R39: renamed from R501; value 470R -> 100R/1%
- R43: renamed from R503; value 1.5K/0.5% -> 1K/1%
- R44: renamed from R504; value 1.5K/0.5% -> 1K/1%
- renumbered C503 to C64, C501 to C65, C504 to C66, C502 to C67, C529 to C68, C508 to C69, C510 to C70, C511 to C71, C509 to C72, C513 to C73, C514 to C74, C512 to C75, C515 to C76, C516 to C77, C517 to C78, C518 to C79, C519 to C80, C520 to C81, C521 to C82, C522 to C83, C523 to C84, C524 to C85, C526 to C87, C527 to C88, R506 to R38, R507 to R40, R502 to R41, R508 to R42, U502 to U12, U200 to U5

Commit message: r0p7 layout done
Parts:
- removed C64, C65, C66, C67: 220nF, Capacitor_SMD:C_0402_1005Metric, symbol Device:C
- C86: value 10uF/10V -> 22uF; footprint Capacitor_SMD:C_0805_2012Metric -> Capacitor_SMD:C_0603_1608Metric

Commit message: Bug fixes and changes for r0p8
Other:
- company: Copyright 2022 Modos / Engineer: Wenting Zhang -> Copyright 2024 Wenting Zhang
- title: Caster EPDC -> Glider
Changed lines of the file:
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@@
 	(paper "A4")
 	(title_block
-		(title "Caster EPDC")
-		(date "2022-07-03")
-		(rev "R0.4")
-		(company "Copyright 2022 Modos / Engineer: Wenting Zhang")
+		(title "Glider")
+		(date "2024-05-09")
+		(rev "R0.8")
+		(company "Copyright 2024 Wenting Zhang")
 	)
 	(junction
