File: pcb/mainboard/fpga_ddr.kicad_sch (KiCad schematic)
At the start: 31 parts, among them U12 MT41K64M16TW, U5 XC6SLX-FTG256

Commit message: PCB r0p10
Parts:
- U1: renamed from U5; footprint (none) -> footprints:Xilinx_FTG256
Changed lines of the file:
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@@
 			)
 		)
-		(property "LCSC" ""
+		(property "Ref.Price" "0.001"
 			(at 184.15 93.98 0)
 			(effects
@@
 			)
 		)
-		(property "Ref.Price" "0.001"
+		(property "desc" ""
 			(at 184.15 93.98 0)
 			(effects
@@
 			)
 		)
-		(property "LCSC" ""
+		(property "Ref.Price" "0.0025"
 			(at 248.92 140.97 0)
 			(effects
@@
 			)
 		)
-		(property "Ref.Price" "0.0025"
+		(property "desc" ""
 			(at 248.92 140.97 0)
 			(effects
@@
 			)
 		)
-		(property "LCSC" ""
+		(property "Ref.Price" "0.0009"
 			(at 238.76 118.11 0)
 			(effects
@@
 			)
 		)
-		(property "Ref.Price" "0.0009"
+		(property "desc" ""
 			(at 238.76 118.11 0)
 			(effects
@@
 			)
 		)
-		(property "LCSC" ""
+		(property "Ref.Price" "0.0036"
 			(at 190.5 158.75 0)
 			(effects
@@
 			)
 		)
-		(property "Ref.Price" "0.0036"
+		(property "desc" ""
 			(at 190.5 158.75 0)
 			(effects
@@
 			)
 		)
-		(property "LCSC" ""
+		(property "Ref.Price" "0.0036"
 			(at 175.26 36.83 0)
 			(effects
@@
 			)
 		)
-		(property "Ref.Price" "0.0036"
+		(property "desc" ""
 			(at 175.26 36.83 0)
 			(effects
@@
 			)
 		)
-		(property "LCSC" ""
+		(property "Ref.Price" "0.0006"
 			(at 177.8 118.11 0)
 			(effects
@@
 			)
 		)
-		(property "Ref.Price" "0.0006"
+		(property "desc" ""
 			(at 177.8 118.11 0)
 			(effects
@@
 			)
 		)
-		(property "LCSC" ""
+		(property "Ref.Price" "0.0023"
 			(at 264.16 153.67 0)
 			(effects
@@
 			)
 		)
-		(property "Ref.Price" "0.0023"
+		(property "desc" ""
 			(at 264.16 153.67 0)
 			(effects
@@
 			)
 		)
-		(property "LCSC" ""
+		(property "Ref.Price" "0.0036"
 			(at 160.02 138.43 0)
 			(effects
@@
 			)
 		)
-		(property "Ref.Price" "0.0036"
+		(property "desc" ""
 			(at 160.02 138.43 0)
 			(effects
@@
 			)
 		)
-		(property "LCSC" ""
+		(property "Ref.Price" "0.0036"
 			(at 170.18 138.43 0)
 			(effects
@@
 			)
 		)
-		(property "Ref.Price" "0.0036"
+		(property "desc" ""
 			(at 170.18 138.43 0)
 			(effects
@@
 			)
 		)
-		(property "LCSC" ""
+		(property "Ref.Price" "0.0006"
 			(at 187.96 118.11 0)
 			(effects
@@
 			)
 		)
-		(property "Ref.Price" "0.0006"
+		(property "desc" ""
 			(at 187.96 118.11 0)
 			(effects
@@
 			)
 		)
-		(property "LCSC" ""
+		(property "Ref.Price" "0.0036"
 			(at 180.34 138.43 0)
 			(effects
@@
 			)
 		)
-		(property "Ref.Price" "0.0036"
+		(property "desc" ""
 			(at 180.34 138.43 0)
 			(effects
@@
 			)
 		)
-		(property "LCSC" ""
+		(property "Ref.Price" "0.0036"
 			(at 111.76 49.53 0)
 			(effects
@@
 			)
 		)
-		(property "Ref.Price" "0.0036"
+		(property "desc" ""
 			(at 111.76 49.53 0)
 			(effects
@@
 			)
 		)
-		(property "LCSC" ""
+		(property "Ref.Price" "0.0301"
 			(at 220.98 158.75 0)
 			(effects
@@
 			)
 		)
-		(property "Ref.Price" "0.0301"
+		(property "desc" ""
 			(at 220.98 158.75 0)
 			(effects
@@
 			)
 		)
-		(property "LCSC" ""
+		(property "Ref.Price" "0.0007"
 			(at 97.79 43.18 0)
 			(effects
@@
 			)
 		)
-		(property "Ref.Price" "0.0007"
+		(property "desc" ""
 			(at 97.79 43.18 0)
 			(effects
@@
 			)
 		)
-		(property "LCSC" ""
+		(property "Ref.Price" "0.0036"
 			(at 111.76 181.61 0)
 			(effects
@@
 			)
 		)
-		(property "Ref.Price" "0.0036"
+		(property "desc" ""
 			(at 111.76 181.61 0)
 			(effects
@@
 			)
 		)
-		(property "LCSC" ""
+		(property "Ref.Price" "0.0036"
 			(at 210.82 138.43 0)
 			(effects
@@
 			)
 		)
-		(property "Ref.Price" "0.0036"
+		(property "desc" ""
 			(at 210.82 138.43 0)
 			(effects
@@
 			)
 		)
-		(property "LCSC" ""
+		(property "Ref.Price" "3.2405"
 			(at 220.98 22.86 0)
 			(effects
@@
 			)
 		)
-		(property "Ref.Price" "3.2405"
+		(property "desc" ""
 			(at 220.98 22.86 0)
 			(effects
@@
 			)
 		)
-		(property "LCSC" ""
+		(property "Ref.Price" "0.0006"
 			(at 251.46 118.11 0)
 			(effects
@@
 			)
 		)
-		(property "Ref.Price" "0.0006"
+		(property "desc" ""
 			(at 251.46 118.11 0)
 			(effects
@@
 			)
 		)
-		(property "LCSC" ""
+		(property "Ref.Price" "0.0301"
 			(at 220.98 138.43 0)
 			(effects
@@
 			)
 		)
-		(property "Ref.Price" "0.0301"
+		(property "desc" ""
 			(at 220.98 138.43 0)
 			(effects
@@
 			)
 		)
-		(property "LCSC" ""
+		(property "Ref.Price" "0.0025"
 			(at 248.92 153.67 0)
 			(effects
@@
 			)
 		)
-		(property "Ref.Price" "0.0025"
+		(property "desc" ""
 			(at 248.92 153.67 0)
 			(effects
@@
 			)
 		)
-		(property "LCSC" ""
+		(property "Ref.Price" "0.0036"
 			(at 210.82 158.75 0)
 			(effects
@@
 			)
 		)
-		(property "Ref.Price" "0.0036"
+		(property "desc" ""
 			(at 210.82 158.75 0)
 			(effects
@@
 			)
 		)
-		(property "LCSC" ""
+		(property "Ref.Price" "0.0036"
 			(at 200.66 158.75 0)
 			(effects
@@
 			)
 		)
-		(property "Ref.Price" "0.0036"
+		(property "desc" ""
 			(at 200.66 158.75 0)
 			(effects
@@
 			)
 		)
-		(property "LCSC" ""
+		(property "Ref.Price" "0.0036"
 			(at 200.66 138.43 0)
 			(effects
@@
 			)
 		)
-		(property "Ref.Price" "0.0036"
+		(property "desc" ""
 			(at 200.66 138.43 0)
 			(effects
@@
 		(dnp no)
 		(fields_autoplaced yes)
-		(property "Reference" "U5"
+		(property "Reference" "U1"
 			(at 44.45 104.1399 0)
 			(effects
@@
 			)
 		)
-		(property "Footprint" ""
+		(property "Footprint" "footprints:Xilinx_FTG256"
 			(at 68.58 111.76 0)
 			(effects
@@
 			)
 		)
+		(property "desc" ""
+			(at 63.5 104.14 0)
+			(effects
+				(font
+					(size 1.27 1.27)
+				)
+				(hide yes)
+			)
+		)
 		(pin "A8"
 		)
@@
 			(project "pcb"
 				(path "/4654897e-3e2f-4522-96c3-20b19803c088/866a5b4a-453a-413a-94a2-5e610f40d8dd"
-					(reference "U5")
+					(reference "U1")
 					(unit 4)
 				)
@@
 			)
 		)
-		(property "LCSC" ""
+		(property "Ref.Price" "0.0036"
 			(at 185.42 36.83 0)
 			(effects
@@
 			)
 		)
-		(property "Ref.Price" "0.0036"
+		(property "desc" ""
 			(at 185.42 36.83 0)
 			(effects
@@
 			)
 		)
-		(property "LCSC" ""
+		(property "Ref.Price" "0.0036"
 			(at 180.34 158.75 0)
 			(effects
@@
 			)
 		)
-		(property "Ref.Price" "0.0036"
+		(property "desc" ""
 			(at 180.34 158.75 0)
 			(effects
@@
 			)
 		)
-		(property "LCSC" ""
+		(property "Ref.Price" "0.0036"
 			(at 190.5 138.43 0)
 			(effects
@@
 			)
 		)
-		(property "Ref.Price" "0.0036"
+		(property "desc" ""
 			(at 190.5 138.43 0)
 			(effects
@@
 			)
 		)
-		(property "LCSC" ""
+		(property "Ref.Price" "0.0023"
 			(at 264.16 140.97 0)
 			(effects
@@
 			)
 		)
-		(property "Ref.Price" "0.0023"
+		(property "desc" ""
 			(at 264.16 140.97 0)
 			(effects
@@
 			)
 		)
-		(property "LCSC" ""
+		(property "Ref.Price" "0.0036"
 			(at 170.18 158.75 0)
 			(effects
@@
 			)
 		)
-		(property "Ref.Price" "0.0036"
+		(property "desc" ""
 			(at 170.18 158.75 0)
 			(effects
@@
 			)
 		)
-		(property "LCSC" ""
+		(property "Ref.Price" "0.0165"
 			(at 238.76 146.05 0)
 			(effects
@@
 			)
 		)
-		(property "Ref.Price" "0.0165"
+		(property "desc" ""
 			(at 238.76 146.05 0)
 			(effects
@@
 			)
 		)
-		(property "LCSC" ""
+		(property "Ref.Price" "0.0036"
 			(at 160.02 158.75 0)
 			(effects
@@
 			)
 		)
-		(property "Ref.Price" "0.0036"
+		(property "desc" ""
 			(at 160.02 158.75 0)
 			(effects

Commit message: PCB r0p13
Parts:
- C144, C88: value 100nF -> 100nF/50V
- C69, C70, C73, C79, C80, C81, C82, C83, C84: value 220nF -> 470nF/25V
- C71, C72, C74, C75, C76, C77, C78: value 220nF -> 100nF/50V
- C85, C86, C87: value 47uF/6.3V -> 22uF/6.3V
- R101, R103, R44: value 5.1K -> 5.1K/1%
Other:
- company: Copyright 2024 Wenting Zhang -> Copyright 2025 Wenting Zhang
Changed lines of the file:
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@@
 	(title_block
 		(title "Glider")
-		(date "2024-05-09")
-		(rev "R0.8")
-		(company "Copyright 2024 Wenting Zhang")
+		(date "2025-04-18")
+		(rev "R0.13")
+		(company "Copyright 2025 Wenting Zhang")
 	)
 	(junction
@@
 			)
 		)
-		(property "Value" "220nF"
+		(property "Value" "470nF/25V"
 			(at 193.421 159.893 0)
 			(effects
@@
 			)
 		)
-		(property "Value" "220nF"
+		(property "Value" "470nF/25V"
 			(at 178.181 37.973 0)
 			(effects
@@
 			)
 		)
-		(property "Value" "5.1K"
+		(property "Value" "5.1K/1%"
 			(at 179.578 119.253 0)
 			(effects
@@
 			)
 		)
-		(property "Value" "100nF"
+		(property "Value" "100nF/50V"
 			(at 267.081 154.813 0)
 			(effects
@@
 			)
 		)
-		(property "Value" "220nF"
+		(property "Value" "100nF/50V"
 			(at 162.941 139.573 0)
 			(effects
@@
 			)
 		)
-		(property "Value" "220nF"
+		(property "Value" "100nF/50V"
 			(at 173.101 139.573 0)
 			(effects
@@
 			)
 		)
-		(property "Value" "5.1K"
+		(property "Value" "5.1K/1%"
 			(at 189.738 119.253 0)
 			(effects
@@
 			)
 		)
-		(property "Value" "220nF"
+		(property "Value" "100nF/50V"
 			(at 183.261 139.573 0)
 			(effects
@@
 			)
 		)
-		(property "Value" "220nF"
+		(property "Value" "470nF/25V"
 			(at 114.681 50.673 0)
 			(effects
@@
 			)
 		)
-		(property "Value" "47uF/6.3V"
+		(property "Value" "22uF/6.3V"
 			(at 223.901 159.893 0)
 			(effects
@@
 			)
 		)
-		(property "Value" "220nF"
+		(property "Value" "470nF/25V"
 			(at 114.681 182.753 0)
 			(effects
@@
 			)
 		)
-		(property "Value" "220nF"
+		(property "Value" "470nF/25V"
 			(at 213.741 139.573 0)
 			(effects
@@
 			)
 		)
-		(property "Value" "5.1K"
+		(property "Value" "5.1K/1%"
 			(at 253.238 119.253 0)
 			(effects
@@
 			)
 		)
-		(property "Value" "47uF/6.3V"
+		(property "Value" "22uF/6.3V"
 			(at 223.901 139.573 0)
 			(effects
@@
 			)
 		)
-		(property "Value" "220nF"
+		(property "Value" "470nF/25V"
 			(at 213.741 159.893 0)
 			(effects
@@
 			)
 		)
-		(property "Value" "220nF"
+		(property "Value" "470nF/25V"
 			(at 203.581 159.893 0)
 			(effects
@@
 			)
 		)
-		(property "Value" "220nF"
+		(property "Value" "470nF/25V"
 			(at 203.581 139.573 0)
 			(effects
@@
 			)
 		)
-		(property "Value" "220nF"
+		(property "Value" "100nF/50V"
 			(at 188.341 37.973 0)
 			(effects
@@
 			)
 		)
-		(property "Value" "220nF"
+		(property "Value" "100nF/50V"
 			(at 183.261 159.893 0)
 			(effects
@@
 			)
 		)
-		(property "Value" "220nF"
+		(property "Value" "470nF/25V"
 			(at 193.421 139.573 0)
 			(effects
@@
 			)
 		)
-		(property "Value" "100nF"
+		(property "Value" "100nF/50V"
 			(at 267.081 142.113 0)
 			(effects
@@
 			)
 		)
-		(property "Value" "220nF"
+		(property "Value" "100nF/50V"
 			(at 173.101 159.893 0)
 			(effects
@@
 			)
 		)
-		(property "Value" "47uF/6.3V"
+		(property "Value" "22uF/6.3V"
 			(at 241.681 147.193 0)
 			(effects
@@
 			)
 		)
-		(property "Value" "220nF"
+		(property "Value" "100nF/50V"
 			(at 162.941 159.893 0)
 			(effects

Commit message: PCB r1.1
Parts:
- C144, C71, C72, C74, C75, C76, C77, C78, C88: LCSC (none) -> C131394
- C69, C70, C73, C79, C80, C81, C82, C83, C84: LCSC (none) -> C6119801
- C85, C86, C87: LCSC (none) -> C59461
- R100, R40: LCSC (none) -> C25076
- R101, R103, R44: LCSC (none) -> C25905
- R102: LCSC (none) -> C25094
- R104, R105: LCSC (none) -> C11702
- U1: LCSC (none) -> C39313
- U12: LCSC (none) -> C524855
Other:
- company: Copyright 2025 Wenting Zhang -> Copyright 2025 Modos Tech Inc
