File: pcb/mainboard/mcu.kicad_sch (KiCad schematic)
At the start: 24 parts, among them SW701 EVQPUJ02K, U701 W25X16JVP, U702 RP2040, Y701 12MHz

Commit message: pcb: r0p5
Parts:
- U701: value W25X16JVP -> W25Q32JV
Connections:
- net GPIO21 renamed EPD_PWR_EN
Other:
- note removed: "Make sure C10 is close to pin 44 of RP2040"
- note removed: "Make sure C8 is close to pin 45 of RP2040"
- note removed: "Make sure R3 and R4 are close to RP2040"
Changed lines of the file:
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@@
     (stroke (width 0) (type solid) (color 0 0 0 0))
   )
-  (text "Make sure R3 and R4\nare close to RP2040" (at 220.98 48.26 0)
-    (effects (font (size 1.27 1.27)) (justify left bottom))
-  )
-  (text "Make sure C10 is close to pin 44 of RP2040" (at 207.01 36.83 0)
-    (effects (font (size 1.27 1.27)) (justify left bottom))
-  )
-  (text "Make sure C8 is close to pin 45 of RP2040" (at 109.22 36.83 0)
-    (effects (font (size 1.27 1.27)) (justify left bottom))
-  )
   (label "XIN" (at 106.68 109.22 180)
     (effects (font (size 1.27 1.27)) (justify right bottom))
@@
     (property "Intersheet References" "${INTERSHEET_REFS}" (id 0) (at 232.5371 71.0406 0)
       (effects (font (size 1.27 1.27)) (justify left) hide)
+    )
+  )
+  (global_label "EPD_PWR_EN" (shape output) (at 220.98 124.46 0)
+    (effects (font (size 1.27 1.27)) (justify left))
+    (property "Intersheet References" "${INTERSHEET_REFS}" (id 0) (at 325.12 238.76 0)
+      (effects (font (size 1.27 1.27)) hide)
     )
   )
@@
     (in_bom yes) (on_board yes)
     (property "Reference" "U701" (id 0) (at 88.9 68.809 0))
-    (property "Value" "W25X16JVP" (id 1) (at 88.9 71.12 0))
+    (property "Value" "W25Q32JV" (id 1) (at 88.9 71.12 0))
     (property "Footprint" "Package_SON:WSON-8-1EP_6x5mm_P1.27mm_EP3.4x4.3mm" (id 2) (at 81.28 83.82 0)
       (effects (font (size 1.27 1.27)) hide)

Commit message: pcb: r0p6
Connections:
- net GPIO22 renamed EPD_VCOM_PWM

Commit message: r0p7 wip, check in before switch to kicad 8
Parts:
- removed R703, R704: 4.7K, Resistor_SMD:R_0402_1005Metric, symbol Device:R
- removed U702: RP2040, footprints:RP2040-QFN-56, symbol MCU_RaspberryPi_RP2040:RP2040
- added J5: SM03B-SRSS-TB, Connector_JST:JST_SH_SM03B-SRSS-TB_1x03-1MP_P1.00mm_Horizontal, symbol Connector_Generic_MountingPin:Conn_01x03_MountingPin
- added SW401: SW, Button_Switch_SMD:Panasonic_EVQPUL_EVQPUC, symbol Switch:SW_Push
- added U14: RP2040, footprints:RP2040-QFN-56, symbol MCU_RaspberryPi:RP2040
- R58: renamed from R705; value 27 -> 27R
- R59: renamed from R706; value 27 -> 27R
- SW1: renamed from SW701; value EVQPUJ02K -> SW; footprint Button_Switch_SMD:SW_SPST_CK_KXT3 -> Button_Switch_SMD:Panasonic_EVQPUL_EVQPUC
- renumbered C711 to C100, C713 to C101, C714 to C102, C701 to C89, C702 to C90, C703 to C91, C704 to C92, C705 to C93, C706 to C94, C707 to C95, C708 to C96, C709 to C97, C710 to C98, C712 to C99, R701 to R56, R702 to R57, U701 to U13, Y701 to Y2
Connections:
- net +3V3: now also U14.1 (IOVDD), U14.10 (IOVDD), U14.22 (IOVDD), U14.33 (IOVDD), U14.42 (IOVDD), U14.43 (ADC_AVDD), U14.44 (VREG_IN), U14.48 (USB_VDD), U14.49 (IOVDD)
- net DP_HPD: now also U14.9 (GPIO7)
- net DP_PDN: now also U14.12 (GPIO9)
- net DP_VALID: now also U14.6 (GPIO4)
- net EPD_PWR_EN: now also U14.32 (GPIO21)
- net EPD_VCOM_PWM: now also U14.34 (GPIO22)
- net FPGA_CS: now also U14.16 (GPIO13)
- net FPGA_DONE: now also U14.29 (GPIO18)
- net FPGA_MISO: now also U14.15 (GPIO12)
- net FPGA_MOSI: now also U14.18 (GPIO15)
- net FPGA_PROG: now also U14.28 (GPIO17)
- net FPGA_SCLK: now also U14.17 (GPIO14)
- net FPGA_SUSP: now also U14.30 (GPIO19)
- net GND: now also J5.2 (Pin_2), J5.MP (MountPin), SW401.2, U14.19 (TESTEN), U14.57 (GND)
- net GPIO16: now also U14.27 (GPIO16)
- net GPIO20: now also U14.31 (GPIO20)
- net GPIO23: now also U14.35 (GPIO23)
- net GPIO24: now also U14.36 (GPIO24)
- net GPIO25: now also U14.37 (GPIO25)
- net GPIO29_ADC3: now also U14.41 (GPIO29_ADC3)
- net GPIO6: now also U14.8 (GPIO6)
- net MCU_1V1: now also U14.23 (DVDD), U14.45 (VREG_VOUT), U14.50 (DVDD)
- net QSPI_SCLK: now also U14.52 (QSPI_SCLK)
- net QSPI_SD0: now also U14.53 (QSPI_SD0)
- net QSPI_SD1: now also U14.55 (QSPI_SD1)
- net QSPI_SD2: now also U14.54 (QSPI_SD2)
- net QSPI_SD3: now also U14.51 (QSPI_SD3)
- net QSPI_SS: now also U14.56 (QSPI_SS)
- net RUN: now also U14.26 (RUN)
- net SWCLK: now also J5.1 (Pin_1), U14.24 (SWCLK)
- net SWD: now also J5.3 (Pin_3), U14.25 (SWD)
- net TCPC_INT: now also U14.14 (GPIO11)
- net TYPEC_ORI: now also U14.13 (GPIO10)
- net XIN: now also U14.20 (XIN)
- net XOUT: now also U14.21 (XOUT)
- net at R59.2: now also U14.46 (USB_DM)
- net at R58.2: now also U14.47 (USB_DP)
- new net DDC_SCL: U14.3 (GPIO1)
- new net DDC_SDA: U14.2 (GPIO0)
- new net HDMI_DET: U14.11 (GPIO8)
- new net KEY: SW401.1, U14.7 (GPIO5)
- new net TCPC_SCL: U14.5 (GPIO3)
- new net TCPC_SDA: U14.4 (GPIO2)
- new net VCOM_EN: U14.40 (GPIO28_ADC2)
- new net VCOM_MEA: U14.39 (GPIO27_ADC1)
- new net VCOM_MEA_EN: U14.38 (GPIO26_ADC0)
Other:
- moved on the sheet: C100, C101, C102, C89, C90, C91, C92, C93, C94, C95, C96, C97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

Commit message: r0p7 wip
Parts:
- renumbered SW401 to SW2

Commit message: r0p7 layout done
Parts:
- removed R56: 1K, Resistor_SMD:R_0402_1005Metric, symbol Device:R
Connections:
- net GPIO6 is gone; now on net KEY: U14.8 (GPIO6)
- net KEY: no longer U14.7 (GPIO5)
- net KEY2: now reaches SW1.1
- net KEY2: now also U14.7 (GPIO5)
- net DDC_SCL renamed ADV_INT
- net DDC_SDA renamed GPIO0
- net GPIO25 renamed DEC_RST
- net TCPC_SCL renamed I2C_SCL
- net TCPC_SDA renamed I2C_SDA
Other:
- moved on the sheet: C89, C90, C91, C92, C93, C94, C95, C96, C97, C98, C99, R57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

Commit message: Bug fixes and changes for r0p8
Parts:
- added C156: 100nF, Capacitor_SMD:C_0402_1005Metric, symbol Device:C
- added R50, R51: 1M, Resistor_SMD:R_0402_1005Metric, symbol Device:R
Connections:
- net GND: now also C156.2, R51.2
- net GPIO24 renamed FL_PWM
- net GPIO29_ADC3 renamed VBUS_MEA
- net VBUS_MEA: now also C156.1, R50.2, R51.1
- net HDMI_DET renamed GPIO8
- new net VBUS: R50.1
Other:
- company: Copyright 2022 Modos / Engineer: Wenting Zhang -> Copyright 2024 Wenting Zhang
- title: Caster EPDC -> Glider
- moved on the sheet: C92, C93, C97, R57, SW1, SW2, U13, Y2

Commit message: PCB r0p8
Connections:
- net GPIO16 is gone; now on net FL_PWM: U14.27 (GPIO16)
- net FL_PWM: no longer U14.36 (GPIO24)
- new net GPIO24: U14.36 (GPIO24)
Changed lines of the file:
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@@
 	(global_label "FL_PWM"
 		(shape output)
-		(at 233.68 124.46 0)
+		(at 233.68 104.14 0)
 		(effects
 			(font
@@
 		)
 		(property "Intersheetrefs" "${INTERSHEET_REFS}"
-			(at 337.82 238.76 0)
+			(at 337.82 218.44 0)
 			(effects
 				(font

Commit message: BOM adjustments
Parts:
- U13: LCSC C571260 -> (none)
- Y2: footprint Oscillator:Oscillator_SMD_Abracon_ASE-4Pin_3.2x2.5mm -> Crystal:Crystal_SMD_3225-4Pin_3.2x2.5mm
Changed lines of the file:
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@@
 			)
 		)
-		(property "LCSC" "C571260"
+		(property "LCSC" ""
 			(at 86.36 58.42 0)
 			(effects
@@
 			)
 		)
-		(property "Footprint" "Oscillator:Oscillator_SMD_Abracon_ASE-4Pin_3.2x2.5mm"
+		(property "Footprint" "Crystal:Crystal_SMD_3225-4Pin_3.2x2.5mm"
 			(at 91.44 92.71 0)
 			(effects
