File: pcb/mainboard/power.kicad_sch (KiCad schematic)
At the start: 31 parts, among them J1 USB_B_Micro, U200 XC6SLX16-FTG256, U204 SY8008, U205 SY8008, U206 SY8008

Commit message: pcb: r0p4
Parts:
- removed C1: 10uF, Capacitor_SMD:C_0603_1608Metric, symbol Device:C
- removed H3: MountingHole, MountingHole:MountingHole_2.2mm_M2_DIN965, symbol Mechanical:MountingHole
- removed J1: USB_B_Micro, Connector_USB:USB_Micro-B_Amphenol_10103594-0001LF_Horizontal, symbol Connector:USB_B_Micro
- added C205, C206: 100uF/6.3V, Capacitor_SMD:C_1206_3216Metric, symbol Device:C
- U200: footprint Package_BGA:Xilinx_FTG256 -> footprints:Xilinx_FTG256
Connections:
- net +5V: now also C205.2, C206.2
- net GND: now also C205.1, C206.1
- no-connect marks 3 -> 0
Other:
- company: Copyright 2021 Modos / Engineer: Wenting Zhang -> Copyright 2022 Modos / Engineer: Wenting Zhang
- moved on the sheet: C223, C224, C225, C226, C227, C228, C230, C231, C232, C233, C234, C235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

Commit message: pcb: r0p6
Parts:
- added C210, C211, C213, C214, C215, C217, C219: 220nF, Capacitor_SMD:C_0402_1005Metric, symbol Device:C
- added C220: 22uF, Capacitor_SMD:C_0603_1608Metric, symbol Device:C
- C205, C206: value 100uF/6.3V -> 100uF/6.3V
- R212: value 121K/1% -> 120K/1%
- R214: value 22.6K/1% -> 20K/1%
- R215: value 27K/1% -> 24K/1%
- R216: value 34.8K/1% -> 24K/1%
- R217: value 27K/1% -> 20K/1%
Connections:
- net +1V1: now also C210.1, C213.1, C215.1, C217.1, C219.1, C220.1
- net +3V3: now also C211.1, C214.1
- net GND: now also C210.2, C211.2, C213.2, C214.2, C215.2, C217.2, C219.2, C220.2
Other:
- moved on the sheet: U200D

Commit message: r0p7 wip, check in before switch to kicad 8
Parts:
- removed C205, C206: 100uF/6.3V, Capacitor_SMD:C_1206_3216Metric, symbol Device:C
- removed C223, C224, C225, C233, C234, C235: 10uF, Capacitor_SMD:C_0603_1608Metric, symbol Device:C
- removed C226, C227, C228: 100nF, Capacitor_SMD:C_0402_1005Metric, symbol Device:C
- removed C230, C231, C232: 220nF, Capacitor_SMD:C_0402_1005Metric, symbol Device:C
- removed L201, L202, L203: 4.7uH, footprints:L_1212, symbol Device:L
- removed R212: 120K/1%, Resistor_SMD:R_0402_1005Metric, symbol Device:R
- removed R213: 27K/1%, Resistor_SMD:R_0402_1005Metric, symbol Device:R
- removed R214, R217: 20K/1%, Resistor_SMD:R_0402_1005Metric, symbol Device:R
- removed R215, R216: 24K/1%, Resistor_SMD:R_0402_1005Metric, symbol Device:R
- removed U204, U205, U206: SY8008, Package_TO_SOT_SMD:TSOT-23-5, symbol symbols:SY8008
- added C1, C14, C15, C16, C2, C3, C618: 10uF/10V, Capacitor_SMD:C_0805_2012Metric, symbol Device:C
- added C10, C4, C5, C6, C8, C9: 100nF, Capacitor_SMD:C_0402_1005Metric, symbol Device:C
- added C103: 47uF/10V, Capacitor_SMD:C_1206_3216Metric, symbol Device:C
- added C11, C12, C13: 47pF, Capacitor_SMD:C_0402_1005Metric, symbol Device:C
- added C211, C214, C219: 220nF, Capacitor_SMD:C_0402_1005Metric, symbol Device:C
- added H3: MountingHole, MountingHole:MountingHole_2.2mm_M2_DIN965, symbol Mechanical:MountingHole
- added L1, L2, L3: FTC201610S4R7MBCA, Inductor_SMD:L_Murata_DFE201610P, symbol Device:L
- added R3: 91K/1%, Resistor_SMD:R_0402_1005Metric, symbol Device:R
- added R4, R5: 20K/1%, Resistor_SMD:R_0402_1005Metric, symbol Device:R
- added R6, R7: 16K/1%, Resistor_SMD:R_0402_1005Metric, symbol Device:R
- added R8: 27K/1%, Resistor_SMD:R_0402_1005Metric, symbol Device:R
- added R9: 10K/1%, Resistor_SMD:R_0402_1005Metric, symbol Device:R
- added U1, U2, U3: SY8120, Package_TO_SOT_SMD:TSOT-23-6, symbol symbols:SY8120
- added U4: MT9700, Package_TO_SOT_SMD:SOT-23-5, symbol symbols:MT9700
- renumbered U200 to U5
Connections:
- net +1V35: now also C12.2, C15.2, L2.2, R5.2
- net +3V3: now also C11.2, C14.2, C211.1, C214.1, L1.2, R3.2
- net +5V: now also C1.2, C103.2, C2.2, C3.2, C4.2, C5.2, C6.2, C618.2, U1.4 (~{SHDN}), U1.5 (IN), U2.4 (~{SHDN}), U2.5 (IN), U3.4 (~{SHDN}), U3.5 (IN), U4.1 (VOUT)
- net GND: now also C1.1, C103.1, C14.1, C15.1, C16.1, C2.1, C211.2, C214.2, C219.2, C3.1, C4.1, C5.1, C6.1, C618.1, R4.1, R6.1, R8.1, R9.1, U1.2 (GND), U2.2 (GND), U3.2 (GND), U4.2 (GND)
- net +1V1 renamed +1V0
- net +1V0: now also C13.2, C16.2, C219.1, L3.2, R7.2
- new net: C13.1, R7.1, R8.2, U3.3 (FB)
- new net: C11.1, R3.1, R4.2, U1.3 (FB)
- new net: C8.1, L1.1, U1.6 (SW)
- new net: C9.1, L2.1, U2.6 (SW)
- new net: C12.1, R5.1, R6.2, U2.3 (FB)
- new net: C10.2, U3.1 (BS)
- new net: C10.1, L3.1, U3.6 (SW)
- new net: R9.2, U4.3 (SET)
- new net: C8.2, U1.1 (BS)
- new net: C9.2, U2.1 (BS)
- new net VBUS: U4.4 (EN), U4.5 (VIN)
Other:
- note added: "Ilim = 0.68A"
- note added: "Vout = 0.956V"
- note added: "Vout = 1.350V"
- note added: "Vout = 3.330V"
- moved on the sheet: C210, C211, C213, C214, C215, C217, C219, C220, H1, H2, H4, U5D

Commit message: r0p7 wip
Parts:
- renumbered C618 to C17, C210 to C18, C213 to C19, C215 to C20, C217 to C21, C219 to C22, C220 to C23, C211 to C24, C214 to C25, C211 to C57, C214 to C58, C219 to C59

Commit message: r0p7 layout done
Parts:
- added C150: 470nF, Capacitor_SMD:C_0402_1005Metric, symbol Device:C
- added C151, C155: 10uF/10V, Capacitor_SMD:C_0805_2012Metric, symbol Device:C
- added C152, C153: 100nF, Capacitor_SMD:C_0402_1005Metric, symbol Device:C
- added C154: 47pF, Capacitor_SMD:C_0402_1005Metric, symbol Device:C
- added FID1, FID2, FID3, FID4, FID5, FID6: Fiducial, Fiducial:Fiducial_1mm_Mask2mm, symbol Mechanical:Fiducial
- added L8: FTC201610S4R7MBCA, Inductor_SMD:L_Murata_DFE201610P, symbol Device:L
- added R10: 20K/1%, Resistor_SMD:R_0402_1005Metric, symbol Device:R
- added R48: 10K/1%, Resistor_SMD:R_0402_1005Metric, symbol Device:R
- added U20: SY8120, Package_TO_SOT_SMD:TSOT-23-6, symbol symbols:SY8120
- C18, C19, C24, C25: value 220nF -> 47uF/6.3V; footprint Capacitor_SMD:C_0402_1005Metric -> Capacitor_SMD:C_0603_1608Metric
- C20, C22, C57, C59: value 220nF -> 4.7uF
- C21, C58: value 220nF -> 470nF
- C23: value 22uF -> 4.7uF; footprint Capacitor_SMD:C_0603_1608Metric -> Capacitor_SMD:C_0402_1005Metric; LCSC C94018 -> C880414; Ref.Price 0.0301 -> 0.0036
- R7: value 16K/1% -> 20K/1%
- R8: value 27K/1% -> 20K/1%
Connections:
- net +3V3: now also C150.1
- net +5V: now also C151.2, C152.2, U20.4 (~{SHDN}), U20.5 (IN)
- net GND: now also C150.2, C151.1, C152.1, C155.1, R48.1, U20.2 (GND)
- net +1V0 renamed +1V2
- new net: C153.1, L8.1, U20.6 (SW)
- new net: C153.2, U20.1 (BS)
- new net: C154.1, R10.1, R48.2, U20.3 (FB)
- new net +1V8: C154.2, C155.2, L8.2, R10.2
Other:
- note added: "VCCAUX"
- note added: "VCCINT"
- note added: "Vout = 1.200V"
- note removed: "Vout = 0.956V"
- moved on the sheet: C1, C103, C11, C14, C17, C4, C8, H1, H2, H3, H4, L1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

Commit message: Bug fixes and changes for r0p8
Other:
- company: Copyright 2022 Modos / Engineer: Wenting Zhang -> Copyright 2024 Wenting Zhang
- title: Caster EPDC -> Glider
Changed lines of the file:
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@@
 	(paper "A4")
 	(title_block
-		(title "Caster EPDC")
-		(date "2022-07-03")
-		(rev "R0.4")
-		(company "Copyright 2022 Modos / Engineer: Wenting Zhang")
+		(title "Glider")
+		(date "2024-05-09")
+		(rev "R0.8")
+		(company "Copyright 2024 Wenting Zhang")
 	)
 	(junction

Commit message: BOM adjustments
Parts:
- C103, C17: LCSC C105490 -> (none)
- C150, C18, C19, C20, C21, C22, C23, C24, C25, C57, C58, C59: LCSC C880414 -> (none)
- U5: LCSC C39313 -> (none)
Changed lines of the file:
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@@
 			)
 		)
-		(property "LCSC" "C880414"
+		(property "LCSC" ""
 			(at 228.6 148.59 0)
 			(effects
@@
 			)
 		)
-		(property "LCSC" "C880414"
+		(property "LCSC" ""
 			(at 190.5 130.81 0)
 			(effects
@@
 			)
 		)
-		(property "LCSC" "C880414"
+		(property "LCSC" ""
 			(at 190.5 148.59 0)
 			(effects
@@
 			)
 		)
-		(property "LCSC" "C880414"
+		(property "LCSC" ""
 			(at 215.9 130.81 0)
 			(effects
@@
 			)
 		)
-		(property "LCSC" "C880414"
+		(property "LCSC" ""
 			(at 215.9 148.59 0)
 			(effects
@@
 			)
 		)
-		(property "LCSC" "C880414"
+		(property "LCSC" ""
 			(at 241.3 130.81 0)
 			(effects
@@
 			)
 		)
-		(property "LCSC" "C880414"
+		(property "LCSC" ""
 			(at 203.2 148.59 0)
 			(effects
@@
 			)
 		)
-		(property "LCSC" "C880414"
+		(property "LCSC" ""
 			(at 228.6 130.81 0)
 			(effects
@@
 			)
 		)
-		(property "LCSC" "C105490"
+		(property "LCSC" ""
 			(at 121.92 44.45 0)
 			(effects
@@
 			)
 		)
-		(property "LCSC" "C105490"
+		(property "LCSC" ""
 			(at 106.68 44.45 0)
 			(effects
@@
 			)
 		)
-		(property "LCSC" "C880414"
+		(property "LCSC" ""
 			(at 254 130.81 0)
 			(effects
@@
 			)
 		)
-		(property "LCSC" "C880414"
+		(property "LCSC" ""
 			(at 177.8 148.59 0)
 			(effects
@@
 			)
 		)
-		(property "LCSC" "C39313"
+		(property "LCSC" ""
 			(at 220.98 81.28 0)
 			(effects
@@
 			)
 		)
-		(property "LCSC" "C880414"
+		(property "LCSC" ""
 			(at 203.2 130.81 0)
 			(effects
@@
 			)
 		)
-		(property "LCSC" "C880414"
+		(property "LCSC" ""
 			(at 177.8 130.81 0)
 			(effects
