File: pcb/mainboard/power.kicad_sch (KiCad schematic)
At the start: 63 parts, among them U1 SY8120, U2 SY8120, U20 SY8120, U3 SY8120, U4 MT9700, U5 XC6SLX16-FTG256

Commit message: R0P9 PCB WIP
Parts:
- added R60, R61: 50mR, Resistor_SMD:R_0805_2012Metric, symbol Device:R
Connections:
- net +1V2: now also R61.2; no longer C13.2, C16.2, L3.2, R7.2
- net +1V35: now also R60.2; no longer C12.2, C15.2, L2.2, R5.2
- new net S5N: C12.2, C15.2, L2.2, R5.2, R60.1
- new net S6N: C13.2, C16.2, L3.2, R61.1, R7.2
Other:
- note added: "Vout = 1.800V"

Commit message: PCB r0p9
Parts:
- removed C10, C6: 100nF, Capacitor_SMD:C_0402_1005Metric, symbol Device:C
- removed C13: 47pF, Capacitor_SMD:C_0402_1005Metric, symbol Device:C
- removed C16, C3: 10uF/10V, Capacitor_SMD:C_0805_2012Metric, symbol Device:C
- removed FID1, FID2, FID3, FID4, FID5, FID6: Fiducial, Fiducial:Fiducial_1mm_Mask2mm, symbol Mechanical:Fiducial
- removed H1, H2, H3, H4: MountingHole, MountingHole:MountingHole_2.2mm_M2_DIN965, symbol Mechanical:MountingHole
- removed R60, R61: 50mR, Resistor_SMD:R_0805_2012Metric, symbol Device:R
- removed R7, R8: 20K/1%, Resistor_SMD:R_0402_1005Metric, symbol Device:R
- removed U3: SY8120, Package_TO_SOT_SMD:TSOT-23-6, symbol symbols:SY8120
- removed U5: XC6SLX16-FTG256, footprints:Xilinx_FTG256, symbol FPGA_Xilinx_Spartan6:XC6SLX16-FTG256
- added C100, C101, C64, C65: 100nF, Capacitor_SMD:C_0402_1005Metric, symbol Device:C
- added C102: 1uF/50V, Capacitor_SMD:C_0603_1608Metric, symbol Device:C
- added C140, C98, C99: 4.7uF/50V, Capacitor_SMD:C_0805_2012Metric, symbol Device:C
- added C157: 470nF, Capacitor_SMD:C_0402_1005Metric, symbol Device:C
- added C182, C183, C184, C191, C192, C193, C194, C195, C196, C197, C198, C27, C67, C94, C96: 10uF/10V, Capacitor_SMD:C_0603_1608Metric, symbol Device:C
- added C185: 100uF, Capacitor_SMD:C_0805_2012Metric, symbol Device:C
- added C186, C187, C188, C189: 47uF/4V, Capacitor_SMD:C_0603_1608Metric, symbol Device:C
- added C190, C97: 47uF/10V, Capacitor_SMD:C_0805_2012Metric, symbol Device:C
- added C66: 47pF, Capacitor_SMD:C_0402_1005Metric, symbol Device:C
- added C95: DNP, Capacitor_SMD:C_0402_1005Metric, symbol Device:C
- added F1: 3A, Fuse:Fuse_1206_3216Metric, symbol Device:Fuse
- added FB3: 120R, Inductor_SMD:L_0402_1005Metric, symbol Device:FerriteBead_Small
- added L13, L14: FTC201610SR24MBCA, Inductor_SMD:L_Murata_DFE201610P, symbol Device:L
- added L15: WPN4020H2R2MT, Inductor_SMD:L_Changjiang_FNR3012S, symbol Device:L
- added R123, R124, R58: 51K/1%, Resistor_SMD:R_0402_1005Metric, symbol Device:R
- added R125: 0.5R, Resistor_SMD:R_0805_2012Metric, symbol Device:R
- added R57: 160K/1%, Resistor_SMD:R_0402_1005Metric, symbol Device:R
- added U12, U29: SYR838, footprints:CSP-20_4x5_1.6x2.0mm, symbol symbols:SYR838
- added U13: JW3651QFNE, footprints:QFN15_3X4_JW3651, symbol symbols:JW3651QFNE
- added U28: SY8120, Package_TO_SOT_SMD:TSOT-23-6, symbol symbols:SY8120
- added U3: XC7Z010-CLG400, Package_BGA:Xilinx_CLG400, symbol symbols:XC7Z007S-CLG400
- C1, C14, C15, C151, C155, C17, C2: footprint Capacitor_SMD:C_0805_2012Metric -> Capacitor_SMD:C_0603_1608Metric
- C103: footprint Capacitor_SMD:C_1206_3216Metric -> Capacitor_SMD:C_0805_2012Metric
- C150, C21: Ref.Price 0.0036 -> (none)
- C18, C19: value 47uF/6.3V -> 470nF; footprint Capacitor_SMD:C_0603_1608Metric -> Capacitor_SMD:C_0402_1005Metric; Ref.Price 0.0036 -> (none)
- C20, C57, C59: value 4.7uF -> 470nF; Ref.Price 0.0036 -> (none)
- C22, C23: value 4.7uF -> 10uF/10V; footprint Capacitor_SMD:C_0402_1005Metric -> Capacitor_SMD:C_0603_1608Metric; Ref.Price 0.0036 -> (none)
- C24, C25: value 47uF/6.3V -> 100uF; footprint Capacitor_SMD:C_0603_1608Metric -> Capacitor_SMD:C_0805_2012Metric; Ref.Price 0.0036 -> (none)
- C58: value 470nF -> 47uF/4V; footprint Capacitor_SMD:C_0402_1005Metric -> Capacitor_SMD:C_0603_1608Metric; Ref.Price 0.0036 -> (none)
- L1, L2, L3, L8: value FTC201610S4R7MBCA -> WPN3012H4R7MT; footprint Inductor_SMD:L_Murata_DFE201610P -> Inductor_SMD:L_Changjiang_FNR3012S
- R10, R5: value 20K/1% -> 200K/1%
- R3: value 91K/1% -> 160K/1%
- R4: value 20K/1% -> 36K/1%
- R48: value 10K/1% -> 100K/1%
- R6: value 16K/1% -> 160K/1%
- R9: value 10K/1% -> 5.1K/1%
Connections:
- net +5V: now also C190.1, C191.1, C192.1, C193.1, C194.1, C27.2, C64.2, U12.A2 (EN), U12.D1 (VIN), U12.D2 (VIN), U12.E1 (VIN), U12.E2 (VIN), U28.4 (~{SHDN}), U28.5 (IN), U29.A2 (EN), U29.D1 (VIN), U29.D2 (VIN), U29.E1 (VIN), U29.E2 (VIN)
- net GND: now also C57.1, C58.1, C102.1, C140.1, C157.2, C182.2, C183.2, C184.2, C185.2, C186.2, C187.2, C188.2, C189.2, C190.2, C191.2, C192.2, C193.2, C194.2, C195.2, C196.2, C197.2, C198.2, C27.1, C64.1, C67.1, C94.1, C96.1, C97.1, C98.1, C99.1, R124.1, R58.1, U12.A1 (VSEL), U12.B2 (GND), U12.B3 (GND), U12.B4 (AGND), U12.C1 (GND), U12.C2 (GND), U12.C3 (GND), U12.C4 (GND), U13.1 (CSP), U13.12 (TEST), U13.14 (GND), U13.3 (PGND), U13.6 (OLIM), U28.2 (GND), U29.A1 (VSEL), U29.B2 (GND), U29.B3 (GND), U29.B4 (AGND), U29.C1 (GND), U29.C2 (GND), U29.C3 (GND), U29.C4 (GND), U3.A18 (GND[59]), U3.A8 (GND[59]), U3.B1 (GND[59]), U3.B11 (GND[59]), U3.C14 (GND[59]), U3.C4 (GND[59]), U3.C9 (GND[59]), U3.D17 (GND[59]), U3.E10 (GND[59]), U3.E20 (GND[59]), U3.F3 (GND[59]), U3.F7 (GND[59]), U3.G10 (GND[59]), U3.G12 (GND[59]), U3.G16 (GND[59]), U3.H11 (GND[59]), U3.H13 (GND[59]), U3.H19 (GND[59]), U3.H7 (GND[59]), U3.H9 (GND[59]), U3.J12 (GND[59]), U3.J2 (GND[59]), U3.J8 (GND[59]), U3.K11 (GND[59]), U3.K13 (GND[59]), U3.K15 (GND[59]), U3.K5 (GND[59]), U3.K7 (GND[59]), U3.L12 (GND[59]), U3.L18 (GND[59]), U3.L8 (GND[59]), U3.M1 (GND[59]), U3.M11 (GND[59]), U3.M13 (GND[59]), U3.M7 (GND[59]), U3.N10 (GND[59]), U3.N12 (GND[59]), U3.N14 (GND[59]), U3.N4 (GND[59]), U3.N8 (GND[59]), U3.P11 (GND[59]), U3.P13 (GND[59]), U3.P17 (GND[59]), U3.P7 (GND[59]), U3.P9 (GND[59]), U3.R12 (GND[59]), U3.R20 (GND[59]), U3.R8 (GND[59]), U3.T13 (GND[59]), U3.T3 (GND[59]), U3.T7 (GND[59]), U3.U16 (GND[59]), U3.U6 (GND[59]), U3.V19 (GND[59]), U3.V9 (GND[59]), U3.W12 (GND[59]), U3.W2 (GND[59]), U3.Y15 (GND[59]), U3.Y5 (GND[59]); no longer C57.2, C58.2
- net VBUS: now also F1.1; no longer U4.4 (EN), U4.5 (VIN)
- net at C153.1, U20.6 (SW): now also L1.1; no longer L8.1
- net at C8.1, U1.6 (SW): now also L2.1; no longer L1.1
- net at C9.1, U2.6 (SW): now also L8.1; no longer L2.1
- net at L3.1: now also C65.1, U28.6 (SW)
- net +1V2 renamed +1V0_PL
- net +1V0_PL: now also C24.1, C182.1, C185.1, U3.G11 (VCCBRAM[2]), U3.G13 (VCCINT[9]), U3.H10 (VCCBRAM[2]), U3.H12 (VCCINT[9]), U3.J13 (VCCINT[9]), U3.K12 (VCCINT[9]), U3.L13 (VCCINT[9]), U3.M12 (VCCINT[9]), U3.N13 (VCCINT[9]), U3.P12 (VCCINT[9]), U3.R13 (VCCINT[9]); no longer C19.1, C21.1, C23.1
- net +1V8 renamed +1V8_DCDC
- net +1V8_DCDC: now also L1.2; no longer L8.2
- removed net +3V3: C11.2, C14.2, C150.1, C24.1, C25.1, C57.1, C58.1, L1.2, R3.2
- net S5N renamed +1V35_DCDC
- net +1V35_DCDC: now also L8.2; no longer L2.2
- net S6N renamed +2V5
- net +2V5: now also C66.2, C67.2, R57.2
- new net: C65.2, U28.1 (BS)
- new net: C66.1, R57.1, R58.2, U28.3 (FB)
- new net: C100.2, L15.1, U13.10 (SW2)
- new net: C100.1, U13.11 (BST2)
- new net: C102.2, C98.2, C99.2, F1.2, R125.2, U13.2 (VIN)
- new net: C95.2, R123.2, R124.2, U13.5 (FB)
- new net: C101.1, U13.8 (BST1)
- new net: C101.2, L15.2, U13.9 (SW1)
- new net: C140.2, R125.1
- new net: L14.1, U29.D3 (LX), U29.D4 (LX), U29.E3 (LX), U29.E4 (LX)
- new net: L13.1, U12.D3 (LX), U12.D4 (LX), U12.E3 (LX), U12.E4 (LX)
- new net +1V0_PL_DCDC: C196.1, C198.1, L14.2, U29.A4 (VOUT)
- new net +1V0_PS: C19.1, C21.1, C23.1, C25.1, U3.G7 (VCCPINT[6]), U3.J7 (VCCPINT[6]), U3.L7 (VCCPINT[6]), U3.N7 (VCCPINT[6]), U3.P8 (VCCPINT[6]), U3.R7 (VCCPINT[6])
- new net +1V0_PS_DCDC: C195.1, C197.1, L13.2, U12.A4 (VOUT)
- new net +1V8_FPGA: C150.1, C157.1, C183.1, C184.1, C186.1, C187.1, C188.1, C189.1, FB3.2, U3.F8 (VCCPAUX[5]), U3.G9 (VCCPAUX[5]), U3.H8 (VCCPAUX[5]), U3.J11 (VCCAUX[6]), U3.K8 (VCCPAUX[5]), U3.L11 (VCCAUX[6]), U3.M8 (VCCPAUX[5]), U3.N11 (VCCAUX[6]), U3.N9 (VCCAUX[6]), U3.P10 (VCCAUX[6]), U3.R9 (VCCAUX[6])
- new net +3V3_DCDC: C11.2, C14.2, L2.2, R3.2
- new net +5V2: C95.1, C96.2, C97.2, R123.1, U13.4 (VO), U4.4 (EN), U4.5 (VIN)
- new net EVDD: C94.2, U13.13 (VCC), U13.15 (CSN), U13.7 (EN)
- new net I2C0_SCL: U29.B1 (SCL)
- new net I2C0_SDA: U29.A3 (SDA)
- new net I2C1_SCL: U12.B1 (SCL)
- new net I2C1_SDA: U12.A3 (SDA)
- new net VCCPLL: C57.2, C58.2, FB3.1, U3.G8 (VCCPLL)
Other:
- note added: "Ilim = 1.33A"
- note added: "VCCBRAM"
- note added: "VCCPAUX"
- note added: "VCCPINT"
- note removed: "Ilim = 0.68A"
- note removed: "Vout = 1.200V"
- moved on the sheet: C1, C103, C11, C12, C14, C15, C151, C152, C153, C154, C155, C17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

Commit message: PCB r0p10 wip
Parts:
- removed C150, C157: 470nF, Capacitor_SMD:C_0402_1005Metric, symbol Device:C
- removed C182, C183, C184, C191, C192, C193, C194, C195, C196, C197, C198: 10uF/10V, Capacitor_SMD:C_0603_1608Metric, symbol Device:C
- removed C185: 100uF, Capacitor_SMD:C_0805_2012Metric, symbol Device:C
- removed C186, C187, C188, C189: 47uF/4V, Capacitor_SMD:C_0603_1608Metric, symbol Device:C
- removed C190: 47uF/10V, Capacitor_SMD:C_0805_2012Metric, symbol Device:C
- removed FB3: 120R, Inductor_SMD:L_0402_1005Metric, symbol Device:FerriteBead_Small
- removed L13, L14: FTC201610SR24MBCA, Inductor_SMD:L_Murata_DFE201610P, symbol Device:L
- removed U12, U29: SYR838, footprints:CSP-20_4x5_1.6x2.0mm, symbol symbols:SYR838
- removed U3: XC7Z010-CLG400, Package_BGA:Xilinx_CLG400, symbol symbols:XC7Z007S-CLG400
- added C68: 470nF, Capacitor_SMD:C_0402_1005Metric, symbol Device:C
- added U29: XC6SLX-FTG256, symbol symbols:XC6SLX-FTG256
- C18, C19, C20, C21: value 470nF -> 47uF/6.3V; footprint Capacitor_SMD:C_0402_1005Metric -> Capacitor_SMD:C_0603_1608Metric; Ref.Price (none) -> 0.0036
- C22, C23: value 10uF/10V -> 4.7uF; footprint Capacitor_SMD:C_0603_1608Metric -> Capacitor_SMD:C_0402_1005Metric; Ref.Price (none) -> 0.0036
- C24: value 100uF -> 4.7uF; footprint Capacitor_SMD:C_0805_2012Metric -> Capacitor_SMD:C_0402_1005Metric; Ref.Price (none) -> 0.0036
- C25: value 100uF -> 470nF; footprint Capacitor_SMD:C_0805_2012Metric -> Capacitor_SMD:C_0402_1005Metric; Ref.Price (none) -> 0.0036
- C57, C59: value 470nF -> 4.7uF; Ref.Price (none) -> 0.0036
- C58: value 47uF/4V -> 470nF; footprint Capacitor_SMD:C_0603_1608Metric -> Capacitor_SMD:C_0402_1005Metric; Ref.Price (none) -> 0.0036
- R57: value 160K/1% -> TBD
- U1, U2, U20, U28: value SY8120 -> SY8113C
Connections:
- net VCCPLL is gone; now on net GND: C57.2, C58.2
- net GND: now also C68.2, U29.A1 (GND), U29.A16 (GND), U29.B11 (GND), U29.B7 (GND), U29.D13 (GND), U29.D4 (GND), U29.E9 (GND), U29.G15 (GND), U29.G2 (GND), U29.G8 (GND), U29.H12 (GND), U29.H7 (GND), U29.H9 (GND), U29.J5 (GND), U29.J8 (GND), U29.K7 (GND), U29.K9 (GND), U29.L15 (GND), U29.L2 (GND), U29.M8 (GND), U29.N13 (GND), U29.P3 (GND), U29.R10 (GND), U29.R6 (GND), U29.T1 (GND), U29.T16 (GND); no longer C57.1, C58.1
- net +1V0_PL renamed +1V2_FPGA
- net +1V2_FPGA: now also C57.1, C68.1, U29.G7 (VCCINT), U29.G9 (VCCINT), U29.H10 (VCCINT), U29.H8 (VCCINT), U29.J7 (VCCINT), U29.J9 (VCCINT), U29.K10 (VCCINT), U29.K8 (VCCINT)
- net +1V0_PS renamed +3V3
- net +3V3: now also C58.1, U29.E5 (VCCAUX), U29.F11 (VCCAUX), U29.F8 (VCCAUX), U29.G10 (VCCAUX), U29.H6 (VCCAUX), U29.J10 (VCCAUX), U29.L6 (VCCAUX), U29.L9 (VCCAUX)
- net +2V5 renamed +1V2_DCDC
- net VBUS renamed +VBUS
Other:
- note added: "Vout = ?"
- note removed: "VCCBRAM"
- note removed: "VCCPAUX"
- note removed: "VCCPINT"
- moved on the sheet: C1, C100, C101, C102, C103, C11, C12, C14, C140, C15, C151, C152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

Commit message: PCB r0p10
Parts:
- R10: value 200K/1% -> 240K/1%
- R3: value 160K/1% -> 680K/1%
- R4: value 36K/1% -> 150K/1%
- R48: value 100K/1% -> 120K/1%
- R5: value 200K/1% -> 150K/1%
- R57: value TBD -> 100K/1%
- R58: value 51K/1% -> 100K/1%
- R6: value 160K/1% -> 120K/1%
- U1: renamed from U29; footprint (none) -> footprints:Xilinx_FTG256
- renumbered U1 to U5
Other:
- note added: "Vout = 1.200V"
- note added: "Vout = 3.326V"
- note removed: "Vout = 3.330V"
- note removed: "Vout = ?"

Commit message: PCB r0p11
Parts:
- L15: footprint Inductor_SMD:L_Changjiang_FNR3012S -> Inductor_SMD:L_Changjiang_FNR4020S
- R123: value 51K/1% -> 100K/1%
- R124: value 51K/1% -> 22K/1%
Connections:
- net +5V2 renamed +5V_DCDC
Changed lines of the file:
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@@
 		(on_board yes)
 		(dnp no)
-		(fields_autoplaced yes)
 		(property "Reference" "#PWR0106"
 			(at 96.52 46.99 0)
@@
 			)
 		)
-		(property "Value" "+5V2"
-			(at 96.52 38.1 0)
+		(property "Value" "+5V_DCDC"
+			(at 91.44 38.1 0)
 			(effects
 				(font
 					(size 1.27 1.27)
 				)
+				(justify left)
 			)
 		)
@@
 		(on_board yes)
 		(dnp no)
-		(fields_autoplaced yes)
 		(property "Reference" "#PWR0107"
 			(at 106.68 46.99 0)
@@
 			)
 		)
-		(property "Value" "+5V2"
-			(at 106.68 38.1 0)
+		(property "Value" "+5V_DCDC"
+			(at 102.87 38.1 0)
 			(effects
 				(font
 					(size 1.27 1.27)
 				)
+				(justify left)
 			)
 		)
@@
 			)
 		)
-		(property "Footprint" "Inductor_SMD:L_Changjiang_FNR3012S"
+		(property "Footprint" "Inductor_SMD:L_Changjiang_FNR4020S"
 			(at 63.5 27.94 0)
 			(effects
@@
 			)
 		)
-		(property "Value" "51K/1%"
+		(property "Value" "100K/1%"
 			(at 95.25 48.26 90)
 			(effects
@@
 			)
 		)
-		(property "Value" "51K/1%"
+		(property "Value" "22K/1%"
 			(at 86.36 57.15 90)
 			(effects

Commit message: PCB r0p13
Parts:
- removed C17: 10uF/10V, Capacitor_SMD:C_0603_1608Metric, symbol Device:C
- removed R125: 0.5R, Resistor_SMD:R_0805_2012Metric, symbol Device:R
- C1, C151, C2, C27: value 10uF/10V -> 22uF/10V; footprint Capacitor_SMD:C_0603_1608Metric -> Capacitor_SMD:C_0805_2012Metric; Ref.Price (none) -> 0.0165
- C100, C101, C152, C153, C4, C5, C64, C65, C8, C9: value 100nF -> 100nF/50V
- C102: value 1uF/50V -> 100nF/50V; footprint Capacitor_SMD:C_0603_1608Metric -> Capacitor_SMD:C_0402_1005Metric
- C103, C97: value 47uF/10V -> 22uF/10V
- C11, C12, C154, C66: value 47pF -> 18pF/50V
- C14, C15, C155, C67: value 10uF/10V -> 22uF/6.3V; Ref.Price (none) -> 0.0036
- C18, C19, C20, C21: value 47uF/6.3V -> 22uF/6.3V
- C22, C23, C24, C57, C59: value 4.7uF -> 4.7uF/6.3V
- C25, C58, C68: value 470nF -> 470nF/25V
- C94, C96: value 10uF/10V -> 22uF/10V; footprint Capacitor_SMD:C_0603_1608Metric -> Capacitor_SMD:C_0805_2012Metric
- R123: value 100K/1% -> 470K/1%
- R124: value 22K/1% -> 100K/1%
- R3: value 680K/1% -> 100K/1%
- R4: value 150K/1% -> 22K/1%
Connections:
- net +1V2_DCDC: now also C67.1; no longer C67.2
- net +1V35_DCDC: now also C155.1; no longer C15.2
- net +1V8_DCDC: now also C14.1; no longer C155.2
- net +3V3_DCDC: now also C15.1; no longer C14.2
- net GND: now also C14.2, C15.2, C155.2, C67.2; no longer C14.1, C15.1, C155.1, C67.1
- net at C102.2, C98.2, C99.2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: now also C140.2
Other:
- company: Copyright 2024 Wenting Zhang -> Copyright 2025 Wenting Zhang
- moved on the sheet: C103

Commit message: PCB r1.1
Parts:
- C1, C103, C151, C2, C27, C94, C96, C97: LCSC (none) -> C29277
- C100, C101, C102, C152, C153, C4, C5, C64, C65, C8, C9: LCSC (none) -> C131394
- C11, C12, C154, C66: LCSC (none) -> C106202
- C14, C15, C155, C18, C19, C20, C21, C67: LCSC (none) -> C59461
- C140, C98, C99: LCSC (none) -> C6119903
- C22, C23, C24, C57, C59: LCSC (none) -> C307423
- C25, C58, C68: LCSC (none) -> C6119801
- C95: value DNP -> 1nF/50V; LCSC (none) -> C14442
- F1: LCSC (none) -> C14165
- L1, L2, L3, L8: LCSC (none) -> C98357
- L15: LCSC (none) -> C98361
- R10: LCSC (none) -> C64043
- R123: LCSC (none) -> C25790
- R124, R3, R57, R58: LCSC (none) -> C25741
- R4: LCSC (none) -> C25768
- R48, R6: LCSC (none) -> C25750
- R5: LCSC (none) -> C25755
- R9: LCSC (none) -> C25905
- U1: LCSC (none) -> C39313
- U13: LCSC (none) -> C5444670
- U2, U20, U28, U5: LCSC (none) -> C6338414
- U4: LCSC (none) -> C89855
Connections:
- net +1V2_DCDC: now also C66.1, R57.1; no longer C66.2, R57.2
- net +1V35_DCDC: now also C12.1, R5.1; no longer C12.2, R5.2
- net +1V8_DCDC: now also C154.1, R10.1; no longer C154.2, R10.2
- net +3V3_DCDC: now also C11.1, R3.1; no longer C11.2, R3.2
- net GND: now also R4.2, R48.2, R58.2, R6.2; no longer R4.1, R48.1, R58.1, R6.1
- new net: C66.2, R57.2, R58.1, U28.3 (FB)
- new net: C11.2, R3.2, R4.1, U5.3 (FB)
- new net: C154.2, R10.2, R48.1, U20.3 (FB)
- new net: C12.2, R5.2, R6.1, U2.3 (FB)
Other:
- company: Copyright 2025 Wenting Zhang -> Copyright 2025 Modos Tech Inc
- moved on the sheet: C1, C11, C12, C14, C15, C151, C154, C155, C2, C20, C21, C22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
