File: pcb/mainboard/pcb.kicad_sch (KiCad schematic)
At the start: 0 parts

Commit message: pcb: r0p4
Other:
- added sheet mcu (mcu.kicad_sch)
- note added: "Microcontroller"
- note added: "USB Type-C Input"
- note removed: "DisplayPort Input"
- company: Copyright 2021 Modos / Engineer: Wenting Zhang -> Copyright 2022 Modos / Engineer: Wenting Zhang

Commit message: r0p7 wip, check in before switch to kicad 8
Other:
- added sheet tmds_in (tmds_in.kicad_sch)
- note added: "I2C Addresses 0100010 FUSB302B 1100000 PTN3460BS 1001100 ADV7611"
- note added: "TMDS Input"
- company: Copyright 2022 Modos / Engineer: Wenting Zhang -> Copyright 2023 Modos / Engineer: Wenting Zhang
- title: Caster EPDC -> Glider Lite
Changed lines of the file:
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@@
   (paper "A4")
   (title_block
-    (title "Caster EPDC")
-    (date "2022-07-03")
-    (rev "R0.4")
-    (company "Copyright 2022 Modos / Engineer: Wenting Zhang")
+    (title "Glider Lite")
+    (date "2023-12-24")
+    (rev "R0.7")
+    (company "Copyright 2023 Modos / Engineer: Wenting Zhang")
   )
   (text "FPGA DDR Memory" (at 35.56 67.31 0)
@@
     (effects (font (size 2.54 2.54)) (justify left bottom))
   )
-  (text "Microcontroller" (at 35.56 90.17 0)
+  (text "USB Type-C Input" (at 35.56 78.74 0)
+    (effects (font (size 2.54 2.54)) (justify left bottom))
+  )
+  (text "Microcontroller" (at 35.56 101.6 0)
     (effects (font (size 2.54 2.54)) (justify left bottom))
   )
@@
     (effects (font (size 2.54 2.54)) (justify left bottom))
   )
+  (text "I2C Addresses\n0100010 FUSB302B\n1100000 PTN3460BS\n1001100 ADV7611"
+    (at 33.02 185.42 0)
+    (effects (font (size 1.27 1.27)) (justify left bottom))
+  )
   (text "FPGA Core" (at 35.56 44.45 0)
     (effects (font (size 2.54 2.54)) (justify left bottom))
   )
-  (text "USB Type-C Input" (at 35.56 78.74 0)
+  (text "TMDS Input" (at 35.56 90.17 0)
     (effects (font (size 2.54 2.54)) (justify left bottom))
   )
-  (sheet (at 33.02 27.94) (size 54.61 6.35) (fields_autoplaced)
+  (sheet (at 33.02 27.94) (size 53.34 6.35) (fields_autoplaced)
     (stroke (width 0.1524) (type solid))
     (fill (color 0 0 0 0.0000))
@@
     )
   )
-  (sheet (at 33.02 39.37) (size 54.61 6.35) (fields_autoplaced)
+  (sheet (at 33.02 85.09) (size 53.34 6.35) (fields_autoplaced)
+    (stroke (width 0.1524) (type solid))
+    (fill (color 0 0 0 0.0000))
+    (property "Sheetname" "tmds_in" (at 33.02 84.3784 0)
+      (effects (font (size 1.27 1.27)) (justify left bottom))
+    )
+    (property "Sheetfile" "tmds_in.kicad_sch" (at 33.02 92.0246 0)
+      (effects (font (size 1.27 1.27)) (justify left top))
+    )
+    (instances
+      (project "pcb"
+        (path "/4654897e-3e2f-4522-96c3-20b19803c088" (page "8"))
+      )
+    )
+  )
+  (sheet (at 33.02 39.37) (size 53.34 6.35) (fields_autoplaced)
     (stroke (width 0.1524) (type solid))
     (fill (color 0 0 0 0.0000))
@@
     )
   )
-  (sheet (at 33.02 73.66) (size 54.61 6.35) (fields_autoplaced)
+  (sheet (at 33.02 73.66) (size 53.34 6.35) (fields_autoplaced)
     (stroke (width 0.1524) (type solid))
     (fill (color 0 0 0 0.0000))
@@
     (instances
       (project "pcb"
-        (path "/4654897e-3e2f-4522-96c3-20b19803c088" (page "7"))
+        (path "/4654897e-3e2f-4522-96c3-20b19803c088" (page "5"))
       )
     )
   )
-  (sheet (at 33.02 62.23) (size 54.61 6.35) (fields_autoplaced)
+  (sheet (at 33.02 62.23) (size 53.34 6.35) (fields_autoplaced)
     (stroke (width 0.1524) (type solid))
     (fill (color 0 0 0 0.0000))
@@
     (instances
       (project "pcb"
-        (path "/4654897e-3e2f-4522-96c3-20b19803c088" (page "5"))
+        (path "/4654897e-3e2f-4522-96c3-20b19803c088" (page "4"))
       )
     )
   )
-  (sheet (at 33.02 50.8) (size 54.61 6.35) (fields_autoplaced)
+  (sheet (at 33.02 50.8) (size 53.34 6.35) (fields_autoplaced)
     (stroke (width 0.1524) (type solid))
     (fill (color 0 0 0 0.0000))
@@
     )
   )
-  (sheet (at 33.02 85.09) (size 54.61 6.35) (fields_autoplaced)
+  (sheet (at 33.02 96.52) (size 53.34 6.35) (fields_autoplaced)
     (stroke (width 0.1524) (type solid))
     (fill (color 0 0 0 0.0000))
-    (property "Sheetname" "mcu" (at 33.02 84.3784 0)
+    (property "Sheetname" "mcu" (at 33.02 95.8084 0)
       (effects (font (size 1.27 1.27)) (justify left bottom))
     )
-    (property "Sheetfile" "mcu.kicad_sch" (at 33.02 92.0246 0)
+    (property "Sheetfile" "mcu.kicad_sch" (at 33.02 103.4546 0)
       (effects (font (size 1.27 1.27)) (justify left top))
     )
     (instances
       (project "pcb"
-        (path "/4654897e-3e2f-4522-96c3-20b19803c088" (page "7"))
+        (path "/4654897e-3e2f-4522-96c3-20b19803c088" (page "6"))
       )
     )

Commit message: Bug fixes and changes for r0p8
Other:
- company: Copyright 2023 Modos / Engineer: Wenting Zhang -> Copyright 2024 Wenting Zhang
- title: Glider Lite -> Glider
Changed lines of the file:
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@@
 	(paper "A4")
 	(title_block
-		(title "Glider Lite")
-		(date "2023-12-24")
-		(rev "R0.7")
-		(company "Copyright 2023 Modos / Engineer: Wenting Zhang")
+		(title "Glider")
+		(date "2024-05-09")
+		(rev "R0.8")
+		(company "Copyright 2024 Wenting Zhang")
 	)
 	(text "FPGA DDR Memory"

Commit message: R0P9 PCB WIP
Other:
- removed sheet eink
- added sheet epd (epd.kicad_sch)
- added sheet epd_power (epd_power.kicad_sch)
- note added: "Display Power Supply"
- note added: "I2C Addresses 0100010 FUSB302B 1100000 PTN3460BS 1001100 ADV7611 1000000 INA3221 #0 1000001 INA3221 #1"
- note added: "Logic Power Supply"
- note removed: "I2C Addresses 0100010 FUSB302B 1100000 PTN3460BS 1001100 ADV7611"
- note removed: "Power Supply"
Changed lines of the file:
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@@
 	(text "FPGA DDR Memory"
 		(exclude_from_sim no)
+		(at 35.56 55.88 0)
+		(effects
+			(font
+				(size 2.54 2.54)
+			)
+			(justify left bottom)
+		)
+	)
+	(text "Logic Power Supply"
+		(exclude_from_sim no)
+		(at 35.56 33.02 0)
+		(effects
+			(font
+				(size 2.54 2.54)
+			)
+			(justify left bottom)
+		)
+	)
+	(text "USB Type-C Input"
+		(exclude_from_sim no)
 		(at 35.56 67.31 0)
 		(effects
@@
 		)
 	)
-	(text "Power Supply"
-		(exclude_from_sim no)
-		(at 35.56 33.02 0)
-		(effects
-			(font
-				(size 2.54 2.54)
-			)
-			(justify left bottom)
-		)
-	)
-	(text "USB Type-C Input"
+	(text "Microcontroller"
+		(exclude_from_sim no)
+		(at 35.56 90.17 0)
+		(effects
+			(font
+				(size 2.54 2.54)
+			)
+			(justify left bottom)
+		)
+	)
+	(text "Display Power Supply"
+		(exclude_from_sim no)
+		(at 35.56 113.03 0)
+		(effects
+			(font
+				(size 2.54 2.54)
+			)
+			(justify left bottom)
+		)
+	)
+	(text "Display"
+		(exclude_from_sim no)
+		(at 35.56 101.6 0)
+		(effects
+			(font
+				(size 2.54 2.54)
+			)
+			(justify left bottom)
+		)
+	)
+	(text "I2C Addresses\n0100010 FUSB302B\n1100000 PTN3460BS\n1001100 ADV7611\n1000000 INA3221 #0\n1000001 INA3221 #1"
+		(exclude_from_sim no)
+		(at 33.02 185.42 0)
+		(effects
+			(font
+				(size 1.27 1.27)
+			)
+			(justify left bottom)
+		)
+	)
+	(text "FPGA Core"
+		(exclude_from_sim no)
+		(at 35.56 44.45 0)
+		(effects
+			(font
+				(size 2.54 2.54)
+			)
+			(justify left bottom)
+		)
+	)
+	(text "TMDS Input"
 		(exclude_from_sim no)
 		(at 35.56 78.74 0)
@@
 		)
 	)
-	(text "Microcontroller"
-		(exclude_from_sim no)
-		(at 35.56 101.6 0)
-		(effects
-			(font
-				(size 2.54 2.54)
-			)
-			(justify left bottom)
-		)
-	)
-	(text "Display"
-		(exclude_from_sim no)
-		(at 35.56 55.88 0)
-		(effects
-			(font
-				(size 2.54 2.54)
-			)
-			(justify left bottom)
-		)
-	)
-	(text "I2C Addresses\n0100010 FUSB302B\n1100000 PTN3460BS\n1001100 ADV7611"
-		(exclude_from_sim no)
-		(at 33.02 185.42 0)
-		(effects
-			(font
-				(size 1.27 1.27)
-			)
-			(justify left bottom)
-		)
-	)
-	(text "FPGA Core"
-		(exclude_from_sim no)
-		(at 35.56 44.45 0)
-		(effects
-			(font
-				(size 2.54 2.54)
-			)
-			(justify left bottom)
-		)
-	)
-	(text "TMDS Input"
-		(exclude_from_sim no)
-		(at 35.56 90.17 0)
-		(effects
-			(font
-				(size 2.54 2.54)
-			)
-			(justify left bottom)
+	(sheet
+		(at 33.02 96.52)
+		(size 53.34 6.35)
+		(fields_autoplaced yes)
+		(stroke
+			(width 0.1524)
+			(type solid)
+		)
+		(fill
+			(color 0 0 0 0.0000)
+		)
+		(property "Sheetname" "epd"
+			(at 33.02 95.8084 0)
+			(effects
+				(font
+					(size 1.27 1.27)
+				)
+				(justify left bottom)
+			)
+		)
+		(property "Sheetfile" "epd.kicad_sch"
+			(at 33.02 103.4546 0)
+			(effects
+				(font
+					(size 1.27 1.27)
+				)
+				(justify left top)
+			)
+		)
+		(instances
+			(project "pcb"
+				(path "/4654897e-3e2f-4522-96c3-20b19803c088"
+					(page "7")
+				)
+			)
 		)
 	)
@@
 	)
 	(sheet
-		(at 33.02 85.09)
+		(at 33.02 73.66)
 		(size 53.34 6.35)
 		(fields_autoplaced yes)
@@
 		)
 		(property "Sheetname" "tmds_in"
-			(at 33.02 84.3784 0)
+			(at 33.02 72.9484 0)
 			(effects
 				(font
@@
 		)
 		(property "Sheetfile" "tmds_in.kicad_sch"
-			(at 33.02 92.0246 0)
-			(effects
-				(font
-					(size 1.27 1.27)
-				)
-				(justify left top)
-			)
-		)
-		(instances
-			(project "pcb"
-				(path "/4654897e-3e2f-4522-96c3-20b19803c088"
-					(page "8")
+			(at 33.02 80.5946 0)
+			(effects
+				(font
+					(size 1.27 1.27)
+				)
+				(justify left top)
+			)
+		)
+		(instances
+			(project "pcb"
+				(path "/4654897e-3e2f-4522-96c3-20b19803c088"
+					(page "6")
 				)
 			)
@@
 	)
 	(sheet
-		(at 33.02 73.66)
+		(at 33.02 62.23)
 		(size 53.34 6.35)
 		(fields_autoplaced yes)
@@
 		)
 		(property "Sheetname" "dp_in"
-			(at 33.02 72.9484 0)
+			(at 33.02 61.5184 0)
 			(effects
 				(font
@@
 		)
 		(property "Sheetfile" "dp_in.kicad_sch"
-			(at 33.02 80.5946 0)
+			(at 33.02 69.1646 0)
+			(effects
+				(font
+					(size 1.27 1.27)
+				)
+				(justify left top)
+			)
+		)
+		(instances
+			(project "pcb"
+				(path "/4654897e-3e2f-4522-96c3-20b19803c088"
+					(page "4")
+				)
+			)
+		)
+	)
+	(sheet
+		(at 33.02 50.8)
+		(size 53.34 6.35)
+		(fields_autoplaced yes)
+		(stroke
+			(width 0.1524)
+			(type solid)
+		)
+		(fill
+			(color 0 0 0 0.0000)
+		)
+		(property "Sheetname" "fpga_ddr"
+			(at 33.02 50.0884 0)
+			(effects
+				(font
+					(size 1.27 1.27)
+				)
+				(justify left bottom)
+			)
+		)
+		(property "Sheetfile" "fpga_ddr.kicad_sch"
+			(at 33.02 57.7346 0)
+			(effects
+				(font
+					(size 1.27 1.27)
+				)
+				(justify left top)
+			)
+		)
+		(instances
+			(project "pcb"
+				(path "/4654897e-3e2f-4522-96c3-20b19803c088"
+					(page "3")
+				)
+			)
+		)
+	)
+	(sheet
+		(at 33.02 85.09)
+		(size 53.34 6.35)
+		(fields_autoplaced yes)
+		(stroke
+			(width 0.1524)
+			(type solid)
+		)
+		(fill
+			(color 0 0 0 0.0000)
+		)
+		(property "Sheetname" "mcu"
+			(at 33.02 84.3784 0)
+			(effects
+				(font
+					(size 1.27 1.27)
+				)
+				(justify left bottom)
+			)
+		)
+		(property "Sheetfile" "mcu.kicad_sch"
+			(at 33.02 92.0246 0)
 			(effects
 				(font
@@
 	)
 	(sheet
-		(at 33.02 62.23)
-		(size 53.34 6.35)
-		(fields_autoplaced yes)
-		(stroke
-			(width 0.1524)
-			(type solid)
-		)
-		(fill
-			(color 0 0 0 0.0000)
-		)
-		(property "Sheetname" "fpga_ddr"
-			(at 33.02 61.5184 0)
-			(effects
-				(font
-					(size 1.27 1.27)
-				)
-				(justify left bottom)
-			)
-		)
-		(property "Sheetfile" "fpga_ddr.kicad_sch"
-			(at 33.02 69.1646 0)
-			(effects
-				(font
-					(size 1.27 1.27)
-				)
-				(justify left top)
-			)
-		)
-		(instances
-			(project "pcb"
-				(path "/4654897e-3e2f-4522-96c3-20b19803c088"
-					(page "4")
-				)
-			)
-		)
-	)
-	(sheet
-		(at 33.02 50.8)
-		(size 53.34 6.35)
-		(fields_autoplaced yes)
-		(stroke
-			(width 0.1524)
-			(type solid)
-		)
-		(fill
-			(color 0 0 0 0.0000)
-		)
-		(property "Sheetname" "eink"
-			(at 33.02 50.0884 0)
-			(effects
-				(font
-					(size 1.27 1.27)
-				)
-				(justify left bottom)
-			)
-		)
-		(property "Sheetfile" "eink.kicad_sch"
-			(at 33.02 57.7346 0)
-			(effects
-				(font
-					(size 1.27 1.27)
-				)
-				(justify left top)
-			)
-		)
-		(instances
-			(project "pcb"
-				(path "/4654897e-3e2f-4522-96c3-20b19803c088"
-					(page "3")
-				)
-			)
-		)
-	)
-	(sheet
-		(at 33.02 96.52)
-		(size 53.34 6.35)
-		(fields_autoplaced yes)
-		(stroke
-			(width 0.1524)
-			(type solid)
-		)
-		(fill
-			(color 0 0 0 0.0000)
-		)
-		(property "Sheetname" "mcu"
-			(at 33.02 95.8084 0)
-			(effects
-				(font
-					(size 1.27 1.27)
-				)
-				(justify left bottom)
-			)
-		)
-		(property "Sheetfile" "mcu.kicad_sch"
-			(at 33.02 103.4546 0)
-			(effects
-				(font
-					(size 1.27 1.27)
-				)
-				(justify left top)
-			)
-		)
-		(instances
-			(project "pcb"
-				(path "/4654897e-3e2f-4522-96c3-20b19803c088"
-					(page "6")
-				)
-			)
+		(at 33.02 107.95)
+		(size 53.34 6.35)
+		(fields_autoplaced yes)
+		(stroke
+			(width 0.1524)
+			(type solid)
+		)
+		(fill
+			(color 0 0 0 0.0000)
+		)
+		(property "Sheetname" "epd_power"
+			(at 33.02 107.2384 0)
+			(effects
+				(font
+					(size 1.27 1.27)
+				)
+				(justify left bottom)
+			)
+		)
+		(property "Sheetfile" "epd_power.kicad_sch"
+			(at 33.02 114.8846 0)
+			(effects
+				(font
+					(size 1.27 1.27)
+				)
+				(justify left top)
+			)
+		)
+		(instances
+			(project "pcb"
+				(path "/4654897e-3e2f-4522-96c3-20b19803c088"
+					(page "8")
+				)
+			)

Commit message: PCB r0p9
Parts:
- added FID1, FID2, FID3, FID4, FID5, FID6: Fiducial, Fiducial:Fiducial_1mm_Mask2mm, symbol Mechanical:Fiducial
- added H1, H2, H3, H4: MountingHole, MountingHole:MountingHole_2.2mm_M2_DIN965_Pad, symbol Mechanical:MountingHole_Pad
- added H10, H11, H12, H13, H14, H15, H16, H17, H18, H19, H20, H21, H22, H5, H6, H7, H8, H9: Shield, footprints:ICSRC6508-030SFR, symbol Mechanical:MountingHole_Pad
Connections:
- new net GND: H1.1, H10.1, H11.1, H12.1, H13.1, H14.1, H15.1, H16.1, H17.1, H18.1, H19.1, H2.1, H20.1, H21.1, H22.1, H3.1, H4.1, H5.1, H6.1, H7.1, H8.1, H9.1
Other:
- removed sheet fpga
- removed sheet mcu
- added sheet fpga_config (fpga_config.kicad_sch)
- added sheet fpga_io (fpga_io.kicad_sch)
- added sheet power_mon (power_mon.kicad_sch)
- note added: "FPGA Config"
- note added: "FPGA IO"
- note added: "I2C Addresses 0100010 FUSB302B 1100000 PTN3460BS 1001100 ADV7611 1010110 STM32 BL 1000000 INA3221 #0 1000001 INA3221 #1"
- note added: "Power Monitoring"
- note removed: "FPGA Core"
- note removed: "I2C Addresses 0100010 FUSB302B 1100000 PTN3460BS 1001100 ADV7611 1000000 INA3221 #0 1000001 INA3221 #1"
- note removed: "Microcontroller"
