File: pcb/mainboard/pcb.kicad_sch (KiCad schematic)
At the start: 28 parts

Commit message: PCB r0p10 wip
Other:
- added sheet mcu (mcu.kicad_sch)
- note added: "Microcontroller"
Changed lines of the file:
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@@
 	(text "FPGA DDR Memory"
 		(exclude_from_sim no)
-		(at 35.56 67.31 0)
+		(at 35.56 63.5 0)
 		(effects
 			(font
@@
 	(text "Power Monitoring"
 		(exclude_from_sim no)
-		(at 35.56 124.46 0)
+		(at 35.56 114.3 0)
 		(effects
 			(font
@@
 	(text "USB Type-C Input"
 		(exclude_from_sim no)
-		(at 35.56 78.74 0)
+		(at 35.56 73.66 0)
 		(effects
 			(font
@@
 	(text "FPGA Config"
 		(exclude_from_sim no)
-		(at 35.56 44.45 0)
+		(at 35.56 43.18 0)
 		(effects
 			(font
@@
 	(text "Display Power Supply"
 		(exclude_from_sim no)
-		(at 35.56 113.03 0)
+		(at 35.56 104.14 0)
 		(effects
 			(font
@@
 	(text "Display"
 		(exclude_from_sim no)
-		(at 35.56 101.6 0)
+		(at 35.56 93.98 0)
 		(effects
 			(font
@@
 	(text "FPGA IO"
 		(exclude_from_sim no)
-		(at 35.56 55.88 0)
+		(at 35.56 53.34 0)
+		(effects
+			(font
+				(size 2.54 2.54)
+			)
+			(justify left bottom)
+		)
+	)
+	(text "Microcontroller"
+		(exclude_from_sim no)
+		(at 35.56 124.46 0)
 		(effects
 			(font
@@
 	(text "TMDS Input"
 		(exclude_from_sim no)
-		(at 35.56 90.17 0)
+		(at 35.56 83.82 0)
 		(effects
 			(font
@@
 	)
 	(sheet
-		(at 33.02 96.52)
-		(size 53.34 6.35)
+		(at 33.02 88.9)
+		(size 53.34 5.08)
 		(fields_autoplaced yes)
 		(stroke
@@
 		)
 		(property "Sheetname" "epd"
-			(at 33.02 95.8084 0)
+			(at 33.02 88.1884 0)
 			(effects
 				(font
@@
 		)
 		(property "Sheetfile" "epd.kicad_sch"
-			(at 33.02 103.4546 0)
+			(at 33.02 94.5646 0)
 			(effects
 				(font
@@
 	(sheet
 		(at 33.02 27.94)
-		(size 53.34 6.35)
+		(size 53.34 5.08)
 		(fields_autoplaced yes)
 		(stroke
@@
 		)
 		(property "Sheetfile" "power.kicad_sch"
-			(at 33.02 34.8746 0)
+			(at 33.02 33.6046 0)
 			(effects
 				(font
@@
 	)
 	(sheet
-		(at 33.02 119.38)
-		(size 53.34 6.35)
+		(at 33.02 109.22)
+		(size 53.34 5.08)
 		(fields_autoplaced yes)
 		(stroke
@@
 		)
 		(property "Sheetname" "power_mon"
-			(at 33.02 118.6684 0)
+			(at 33.02 108.5084 0)
 			(effects
 				(font
@@
 		)
 		(property "Sheetfile" "power_mon.kicad_sch"
-			(at 33.02 126.3146 0)
+			(at 33.02 114.8846 0)
 			(effects
 				(font
@@
 	)
 	(sheet
-		(at 33.02 85.09)
-		(size 53.34 6.35)
+		(at 33.02 78.74)
+		(size 53.34 5.08)
 		(fields_autoplaced yes)
 		(stroke
@@
 		)
 		(property "Sheetname" "tmds_in"
-			(at 33.02 84.3784 0)
+			(at 33.02 78.0284 0)
 			(effects
 				(font
@@
 		)
 		(property "Sheetfile" "tmds_in.kicad_sch"
-			(at 33.02 92.0246 0)
+			(at 33.02 84.4046 0)
 			(effects
 				(font
@@
 	)
 	(sheet
-		(at 33.02 39.37)
-		(size 53.34 6.35)
+		(at 33.02 119.38)
+		(size 53.34 5.08)
+		(fields_autoplaced yes)
+		(stroke
+			(width 0.1524)
+			(type solid)
+		)
+		(fill
+			(color 0 0 0 0.0000)
+		)
+		(property "Sheetname" "mcu"
+			(at 33.02 118.6684 0)
+			(effects
+				(font
+					(size 1.27 1.27)
+				)
+				(justify left bottom)
+			)
+		)
+		(property "Sheetfile" "mcu.kicad_sch"
+			(at 33.02 125.0446 0)
+			(effects
+				(font
+					(size 1.27 1.27)
+				)
+				(justify left top)
+			)
+		)
+		(instances
+			(project "pcb"
+				(path "/4654897e-3e2f-4522-96c3-20b19803c088"
+					(page "10")
+				)
+			)
+		)
+	)
+	(sheet
+		(at 33.02 38.1)
+		(size 53.34 5.08)
 		(fields_autoplaced yes)
 		(stroke
@@
 		)
 		(property "Sheetname" "fpga_config"
-			(at 33.02 38.6584 0)
+			(at 33.02 37.3884 0)
 			(effects
 				(font
@@
 		)
 		(property "Sheetfile" "fpga_config.kicad_sch"
-			(at 33.02 46.3046 0)
+			(at 33.02 43.7646 0)
 			(effects
 				(font
@@
 	)
 	(sheet
-		(at 33.02 73.66)
-		(size 53.34 6.35)
+		(at 33.02 68.58)
+		(size 53.34 5.08)
 		(fields_autoplaced yes)
 		(stroke
@@
 		)
 		(property "Sheetname" "dp_in"
-			(at 33.02 72.9484 0)
+			(at 33.02 67.8684 0)
 			(effects
 				(font
@@
 		)
 		(property "Sheetfile" "dp_in.kicad_sch"
-			(at 33.02 80.5946 0)
+			(at 33.02 74.2446 0)
 			(effects
 				(font
@@
 	)
 	(sheet
-		(at 33.02 62.23)
-		(size 53.34 6.35)
+		(at 33.02 58.42)
+		(size 53.34 5.08)
 		(fields_autoplaced yes)
 		(stroke
@@
 		)
 		(property "Sheetname" "fpga_ddr"
-			(at 33.02 61.5184 0)
+			(at 33.02 57.7084 0)
 			(effects
 				(font
@@
 		)
 		(property "Sheetfile" "fpga_ddr.kicad_sch"
-			(at 33.02 69.1646 0)
+			(at 33.02 64.0846 0)
 			(effects
 				(font
@@
 	)
 	(sheet
-		(at 33.02 50.8)
-		(size 53.34 6.35)
+		(at 33.02 48.26)
+		(size 53.34 5.08)
 		(fields_autoplaced yes)
 		(stroke
@@
 		)
 		(property "Sheetname" "fpga_io"
-			(at 33.02 50.0884 0)
+			(at 33.02 47.5484 0)
 			(effects
 				(font
@@
 		)
 		(property "Sheetfile" "fpga_io.kicad_sch"
-			(at 33.02 57.7346 0)
+			(at 33.02 53.9246 0)
 			(effects
 				(font
@@
 	)
 	(sheet
-		(at 33.02 107.95)
-		(size 53.34 6.35)
+		(at 33.02 99.06)
+		(size 53.34 5.08)
 		(fields_autoplaced yes)
 		(stroke
@@
 		)
 		(property "Sheetname" "epd_power"
-			(at 33.02 107.2384 0)
+			(at 33.02 98.3484 0)
 			(effects
 				(font
@@
 		)
 		(property "Sheetfile" "epd_power.kicad_sch"
-			(at 33.02 114.8846 0)
+			(at 33.02 104.7246 0)
 			(effects
 				(font

Commit message: PCB r0p10
Parts:
- added H23, H24, H25, H26: ICSRC6508-030SFR, footprints:ICSRC6508-030SFR, symbol Mechanical:MountingHole_Pad
- H10, H11, H12, H13, H14, H15, H16, H17, H18, H19, H20, H21, H22, H5, H6, H7, H8, H9: value Shield -> ICSRC6508-030SFR
Connections:
- net GND: now also H23.1, H24.1, H25.1, H26.1

Commit message: PCB r0p13
Parts:
- removed H10, H11, H24: ICSRC6508-030SFR, footprints:ICSRC6508-030SFR, symbol Mechanical:MountingHole_Pad
- removed H2: MountingHole, MountingHole:MountingHole_2.2mm_M2_DIN965_Pad, symbol Mechanical:MountingHole_Pad
Other:
- added sheet user_ext (user_extension.kicad_sch)
- note added: "I2C Addresses 0100010 FUSB302B 1100000 PTN3460BS 1001100 ADV7611 1000000 INA3221 #0 1000001 INA3221 #1"
- note added: "User Extension"
- note removed: "I2C Addresses 0100010 FUSB302B 1100000 PTN3460BS 1001100 ADV7611 1010110 STM32 BL 1000000 INA3221 #0 1000001 INA3221 #1"
- company: Copyright 2024 Wenting Zhang -> Copyright 2025 Wenting Zhang
- moved on the sheet: FID1, FID2, FID3, FID4, FID5, FID6, H1, H12, H13, H14, H15, H16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

Commit message: PCB r1.1
Parts:
- removed FID1, FID2, FID3, FID4, FID5, FID6: Fiducial, Fiducial:Fiducial_1mm_Mask2mm, symbol Mechanical:Fiducial
- H1, H3, H4: LCSC (none) -> DNP
- H12, H13, H14, H15, H16, H17, H18, H19, H20, H21, H22, H23, H25, H26, H5, H6, H7, H8, H9: LCSC (none) -> C2836609
Other:
- note added: "I2C Addresses 0100010 FUSB302B 1100000 PTN3460BS 1001100 ADV7611 1000000 INA3221 #0 1000001 INA3221 #1 1000010 INA3221 #2"
- note removed: "I2C Addresses 0100010 FUSB302B 1100000 PTN3460BS 1001100 ADV7611 1000000 INA3221 #0 1000001 INA3221 #1"
- company: Copyright 2025 Wenting Zhang -> Copyright 2025 Modos Tech Inc
