File: pcb/mainboard/dp_in.kicad_sch (KiCad schematic)
At the start: 33 parts, among them J1 XUNPU TYPEC-324G-ACP24, U16 USBLC6-2P6, U17 FUSB302BMPX, U18 CBTL02043A, U19 PTN3460

Commit message: PCB r0p8
Parts:
- J1: footprint footprints:AMPHENOL_10137065-00021LF -> footprints:XUNPU_TypeC-324G-ACP24
Other:
- note added: "Use XUNPU TYPEC-324G-ACP24"
- note removed: "Use AMPHENOL_10137065-00021LF XUNPU TYPEC-324G-ACP24"
Changed lines of the file:
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@@
 		)
 	)
-	(text "Use\nAMPHENOL_10137065-00021LF\nXUNPU TYPEC-324G-ACP24"
+	(text "Use\nXUNPU TYPEC-324G-ACP24"
 		(exclude_from_sim no)
 		(at 22.86 63.5 0)
@@
 			)
 		)
-		(property "Footprint" "footprints:AMPHENOL_10137065-00021LF"
+		(property "Footprint" "footprints:XUNPU_TypeC-324G-ACP24"
 			(at 44.45 93.98 0)
 			(effects
@@
 					(reference "J1")
 					(unit 1)
+				)
+				(path "/4654897e-3e2f-4522-96c3-20b19803c088/1afc3cb7-9ace-435f-9131-835660c51142"
+					(reference "J1")
+					(unit 1)

Commit message: BOM adjustments
Parts:
- FB1, FB2: value 120 -> 120R
- R1, R2: value 4.7K -> 5.1K
Changed lines of the file:
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@@
 			)
 		)
-		(property "Value" "4.7K"
+		(property "Value" "5.1K"
 			(at 213.36 80.01 90)
 			(effects
@@
 					(unit 1)
 				)
-				(path "/4654897e-3e2f-4522-96c3-20b19803c088/1afc3cb7-9ace-435f-9131-835660c51142"
-					(reference "J1")
-					(unit 1)
-				)
 			)
 		)
@@
 			)
 		)
-		(property "Value" "120"
+		(property "Value" "120R"
 			(at 171.45 137.16 90)
 			(effects
@@
 			)
 		)
-		(property "Value" "4.7K"
+		(property "Value" "5.1K"
 			(at 210.82 69.85 90)
 			(effects
@@
 			)
 		)
-		(property "Value" "120"
+		(property "Value" "120R"
 			(at 171.45 116.84 90)
 			(effects

Commit message: PCB r0p9
Parts:
- added C13, C16: 18pF, Capacitor_SMD:C_0402_1005Metric, symbol Device:C
- added C208, C212: 4.7uF, Capacitor_SMD:C_0603_1608Metric, symbol Device:C
- added C209, C210, C211, C26, C92, C93: 100nF, Capacitor_SMD:C_0402_1005Metric, symbol Device:C
- added FL1: Choke_Coilcraft_0603USB-251, Inductor_SMD:L_CommonModeChoke_Coilcraft_0603USB, symbol Filter:Choke_Coilcraft_0603USB-251
- added R120, R121, R122, R55, R76, R77, R81: 120R, Resistor_SMD:R_0402_1005Metric, symbol Device:R
- added R41: 27R, Resistor_SMD:R_0402_1005Metric, symbol Device:R
- added R43: 12K/1%, Resistor_SMD:R_0402_1005Metric, symbol Device:R
- added U31: USB3300, Package_DFN_QFN:QFN-32-1EP_5x5mm_P0.5mm_EP3.3x3.3mm, symbol Interface_USB:USB3300-EZK
- added Y1: 24MHz, Crystal:Crystal_SMD_3225-4Pin_3.2x2.5mm, symbol Device:Crystal_GND24
Connections:
- net +3V3: now also C26.2, C92.2, C93.2, U31.16 (VDD3.3), U31.25 (VDD3.3), U31.30 (VDD3.3), U31.31 (REG_EN), U31.6 (VDD3.3); no longer FB1.1, FB2.1
- net GND: now also C13.2, C16.2, C208.2, C209.1, C210.1, C211.1, C212.2, C26.1, C92.1, C93.1, R43.1, U31.1 (GND), U31.2 (GND), U31.33 (GND), U31.5 (ID), U31.9 (RESET), Y1.2, Y1.4
- net LVDS_EVEN_AN: now also R121.2
- net LVDS_EVEN_AP: now also R121.1
- net LVDS_EVEN_BN: now also R120.2
- net LVDS_EVEN_BP: now also R120.1
- net LVDS_EVEN_CN: now also R122.2
- net LVDS_EVEN_CP: now also R122.1
- net LVDS_ODD_AN: now also R55.2
- net LVDS_ODD_AP: now also R55.1
- net LVDS_ODD_BN: now also R76.2
- net LVDS_ODD_BP: now also R76.1
- net LVDS_ODD_CN: now also R77.2
- net LVDS_ODD_CP: now also R77.1
- net USB_DN: now also FL1.3; no longer J1.A7 (D-), J1.B7 (D-), U16.3 (I/O2)
- net USB_DP: now also FL1.2; no longer J1.A6 (D+), J1.B6 (D+), U16.1 (I/O1)
- net LVDS_EVEN_CKP: now reaches U19.34 (LVSCKE_P)
- net LVDS_EVEN_CKP: now also R81.1
- net LVDS_EVEN_CKN: now reaches U19.35 (LVSCKE_N)
- net LVDS_EVEN_CKN: now also R81.2
- net +1V8 renamed +1V8_VID
- net DP_VALID: no longer names the net of U19.26 (BKLTEN)
- net I2C_SCL renamed I2C1_SCL
- net I2C_SDA renamed I2C1_SDA
- net LVDS_ODD_CKN: no longer names the net of U19.47 (LVSCKO_N)
- net LVDS_ODD_CKP: no longer names the net of U19.46 (LVSCKO_P)
- new net: C211.2, C212.1, U31.29 (VDDA1.8)
- new net: R41.1, U31.14 (CLKOUT)
- new net: C208.1, C209.2, C210.2, U31.15 (VDD1.8), U31.26 (VDD1.8)
- new net: C13.1, U31.27 (XO), Y1.1
- new net: C16.1, U31.28 (XI), Y1.3
- new net: R43.2, U31.32 (RBIAS)
- new net: FL1.1, U31.7 (DP)
- new net: FL1.4, U31.8 (DM)
- new net: J1.A6 (D+), J1.B6 (D+), U16.1 (I/O1)
- new net: J1.A7 (D-), J1.B7 (D-), U16.3 (I/O2)
- new net +3V3_VID: FB1.1, FB2.1
- new net +5V: U31.4 (VBUS)
- new net CPEN: U31.3 (CPEN)
- new net EXTVBUS: U31.10 (EXTVBUS)
- new net USB0_CLKOUT: R41.2
- new net USB0_DATA0: U31.24 (DATA0)
- new net USB0_DATA1: U31.23 (DATA1)
- new net USB0_DATA2: U31.22 (DATA2)
- new net USB0_DATA3: U31.21 (DATA3)
- new net USB0_DATA4: U31.20 (DATA4)
- new net USB0_DATA5: U31.19 (DATA5)
- new net USB0_DATA6: U31.18 (DATA6)
- new net USB0_DATA7: U31.17 (DATA7)
- new net USB0_DIR: U31.12 (DIR)
- new net USB0_NXT: U31.11 (NXT)
- new net USB0_STP: U31.13 (STP)
- no-connect marks 16 -> 17
Other:
- moved on the sheet: C105, C106, C107, C108, C109, C110, C111, C112, C114, C115, C116, C117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

Commit message: PCB r0p10 wip
Parts:
- removed C13, C16: 18pF, Capacitor_SMD:C_0402_1005Metric, symbol Device:C
- removed C208, C212: 4.7uF, Capacitor_SMD:C_0603_1608Metric, symbol Device:C
- removed C209, C210, C211, C26, C92, C93: 100nF, Capacitor_SMD:C_0402_1005Metric, symbol Device:C
- removed FL1: Choke_Coilcraft_0603USB-251, Inductor_SMD:L_CommonModeChoke_Coilcraft_0603USB, symbol Filter:Choke_Coilcraft_0603USB-251
- removed R120, R121, R122, R55, R76, R77, R81: 120R, Resistor_SMD:R_0402_1005Metric, symbol Device:R
- removed R41: 27R, Resistor_SMD:R_0402_1005Metric, symbol Device:R
- removed R43: 12K/1%, Resistor_SMD:R_0402_1005Metric, symbol Device:R
- removed U31: USB3300, Package_DFN_QFN:QFN-32-1EP_5x5mm_P0.5mm_EP3.3x3.3mm, symbol Interface_USB:USB3300-EZK
- removed Y1: 24MHz, Crystal:Crystal_SMD_3225-4Pin_3.2x2.5mm, symbol Device:Crystal_GND24
Connections:
- net VBUS renamed +VBUS
Other:
- moved on the sheet: C105, C106, C107, C108, C109, C110, C111, C112, C114, C115, C116, C117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

Commit message: PCB r0p10
Connections:
- net SBU1: now also C112.1; no longer C111.1
- net SBU2: now also C111.1; no longer C112.1
- net LVDS_ODD_CKP: now reaches U19.46 (LVSCKO_P)
- net LVDS_ODD_CKN: now reaches U19.47 (LVSCKO_N)
- net LVDS_EVEN_CKN: no longer names the net of U19.35 (LVSCKE_N)
- net LVDS_EVEN_CKP: no longer names the net of U19.34 (LVSCKE_P)
Other:
- moved on the sheet: C111, C112

Commit message: PCB r0p13
Parts:
- C105, C106, C107, C108, C109, C110, C111, C112, C114, C115, C119, C120, C121, C122, C123, C124, C55, C7: value 100nF -> 100nF/50V
- C116, C117, C118: value 1uF -> 4.7uF/6.3V
- FB1, FB2: value 120R -> 120R@100M
- J1: value XUNPU TYPEC-324G-ACP24 -> GT-USB-7007A; footprint footprints:XUNPU_TypeC-324G-ACP24 -> footprints:USB_C_Receptacle_GT-USB-7007A
- R1, R2: value 5.1K -> 5.1K/1%
Connections:
- net CC2: now also D13.5 (IO4), D13.6 (NC1); no longer D13.1 (IO1), D13.10 (NC4)
- net SBU1: now also D13.2 (IO2), D13.9 (NC3); no longer D13.5 (IO4), D13.6 (NC1)
- net SBU2: now also D13.1 (IO1), D13.10 (NC4); no longer D13.2 (IO2), D13.9 (NC3)
Other:
- note removed: "Use XUNPU TYPEC-324G-ACP24"
- company: Copyright 2024 Wenting Zhang -> Copyright 2025 Wenting Zhang
Changed lines of the file:
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@@
 	(title_block
 		(title "Glider")
-		(date "2024-05-09")
-		(rev "R0.8")
-		(company "Copyright 2024 Wenting Zhang")
+		(date "2025-04-18")
+		(rev "R0.13")
+		(company "Copyright 2025 Wenting Zhang")
 	)
 	(junction
@@
 		)
 	)
-	(text "Use\nXUNPU TYPEC-324G-ACP24"
-		(exclude_from_sim no)
-		(at 22.86 76.2 0)
-		(effects
-			(font
-				(size 1.27 1.27)
-			)
-			(justify left bottom)
-		)
-	)
 	(text "SBU reverse is handled by PTN3460"
 		(exclude_from_sim no)
@@
 	)
 	(label "SBU1"
-		(at 27.94 50.8 0)
+		(at 27.94 58.42 0)
 		(fields_autoplaced yes)
 		(effects
@@
 	)
 	(label "SBU2"
-		(at 27.94 58.42 0)
+		(at 27.94 60.96 0)
 		(fields_autoplaced yes)
 		(effects
@@
 	)
 	(label "CC2"
-		(at 27.94 60.96 0)
+		(at 27.94 50.8 0)
 		(fields_autoplaced yes)
 		(effects
@@
 			)
 		)
-		(property "Value" "100nF"
+		(property "Value" "100nF/50V"
 			(at 208.661 111.633 0)
 			(effects
@@
 			)
 		)
-		(property "Value" "100nF"
+		(property "Value" "100nF/50V"
 			(at 95.123 112.649 90)
 			(effects
@@
 			)
 		)
-		(property "Value" "100nF"
+		(property "Value" "100nF/50V"
 			(at 208.661 152.273 0)
 			(effects
@@
 			)
 		)
-		(property "Value" "100nF"
+		(property "Value" "100nF/50V"
 			(at 120.65 96.52 0)
 			(effects
@@
 			)
 		)
-		(property "Value" "100nF"
+		(property "Value" "100nF/50V"
 			(at 93.091 60.833 0)
 			(effects
@@
 			)
 		)
-		(property "Value" "100nF"
+		(property "Value" "100nF/50V"
 			(at 95.123 120.269 90)
 			(effects
@@
 			)
 		)
-		(property "Value" "100nF"
+		(property "Value" "100nF/50V"
 			(at 95.123 115.189 90)
 			(effects
@@
 			)
 		)
-		(property "Value" "100nF"
+		(property "Value" "100nF/50V"
 			(at 208.661 131.953 0)
 			(effects
@@
 			)
 		)
-		(property "Value" "100nF"
+		(property "Value" "100nF/50V"
 			(at 197.231 152.273 0)
 			(effects
@@
 			)
 		)
-		(property "Value" "100nF"
+		(property "Value" "100nF/50V"
 			(at 95.123 127.889 90)
 			(effects
@@
 			)
 		)
-		(property "Value" "100nF"
+		(property "Value" "100nF/50V"
 			(at 95.123 122.809 90)
 			(effects
@@
 			)
 		)
-		(property "Value" "5.1K"
+		(property "Value" "5.1K/1%"
 			(at 218.44 82.55 90)
 			(effects
@@
 			)
 		)
-		(property "Value" "100nF"
+		(property "Value" "100nF/50V"
 			(at 95.123 138.049 90)
 			(effects
@@
 			)
 		)
-		(property "Value" "XUNPU TYPEC-324G-ACP24"
+		(property "Value" "GT-USB-7007A"
 			(at 27.94 116.84 90)
 			(effects
@@
 			)
 		)
-		(property "Footprint" "footprints:XUNPU_TypeC-324G-ACP24"
+		(property "Footprint" "footprints:USB_C_Receptacle_GT-USB-7007A"
 			(at 44.45 106.68 0)
 			(effects
@@
 			)
 		)
-		(property "Value" "120R"
+		(property "Value" "120R@100M"
 			(at 176.53 149.86 90)
 			(effects
@@
 			)
 		)
-		(property "Value" "100nF"
+		(property "Value" "100nF/50V"
 			(at 197.231 111.633 0)
 			(effects
@@
 			)
 		)
-		(property "Value" "1uF"
+		(property "Value" "4.7uF/6.3V"
 			(at 185.801 111.633 0)
 			(effects
@@
 			)
 		)
-		(property "Value" "100nF"
+		(property "Value" "100nF/50V"
 			(at 95.123 107.569 90)
 			(effects
@@
 			)
 		)
-		(property "Value" "100nF"
+		(property "Value" "100nF/50V"
 			(at 95.123 130.429 90)
 			(effects
@@
 			)
 		)
-		(property "Value" "1uF"
+		(property "Value" "4.7uF/6.3V"
 			(at 185.801 152.273 0)
 			(effects
@@
 			)
 		)
-		(property "Value" "5.1K"
+		(property "Value" "5.1K/1%"
 			(at 215.9 72.39 90)
 			(effects
@@
 			)
 		)
-		(property "Value" "100nF"
+		(property "Value" "100nF/50V"
 			(at 95.123 105.029 90)
 			(effects
@@
 			)
 		)
-		(property "Value" "100nF"
+		(property "Value" "100nF/50V"
 			(at 95.123 135.509 90)
 			(effects
@@
 			)
 		)
-		(property "Value" "100nF"
+		(property "Value" "100nF/50V"
 			(at 197.231 131.953 0)
 			(effects
@@
 			)
 		)
-		(property "Value" "1uF"
+		(property "Value" "4.7uF/6.3V"
 			(at 185.801 131.953 0)
 			(effects
@@
 			)
 		)
-		(property "Value" "120R"
+		(property "Value" "120R@100M"
 			(at 176.53 129.54 90)
 			(effects

Commit message: PCB r1.1
Parts:
- C105, C106, C107, C108, C109, C110, C111, C112, C114, C115, C119, C120, C121, C122, C123, C124, C55, C7: LCSC (none) -> C131394
- C116, C117, C118: LCSC (none) -> C307423
- D11, D12, D13: LCSC (none) -> C907837
- FB1, FB2: LCSC (none) -> C14709
- J1: LCSC (none) -> C5299422
- R1, R2: LCSC (none) -> C25905
- U16: footprint Package_TO_SOT_SMD:SOT-666 -> footprints:SOT-666-Alt; LCSC (none) -> C15999
- U17: LCSC (none) -> C132291
- U18: LCSC (none) -> C2652457
- U19: LCSC (none) -> C5190369
Other:
- company: Copyright 2025 Wenting Zhang -> Copyright 2025 Modos Tech Inc
