File: pcb/mainboard/epd.kicad_sch (KiCad schematic)
At the start: 8 parts, among them J4 FH12-50S-0.5SH, J5 Conn_01x08_MountingPin

Commit message: PCB r0p9
Parts:
- added C178, C179, C180, C181: 220nF, Capacitor_SMD:C_0402_1005Metric, symbol Device:C
- added J3: FH12-16S-0.5SH, Connector_FFC-FPC:Hirose_FH12-16S-0.5SH_1x16-1MP_P0.50mm_Horizontal, symbol Connector_Generic_MountingPin:Conn_01x16_MountingPin
- J5: value Conn_01x08_MountingPin -> FH12-8S-0.5SH
Connections:
- net EPDC_GDCLK: now also J3.11 (Pin_11); no longer J4.10 (Pin_10)
- net EPDC_GDOE: now also J3.9 (Pin_9); no longer J4.8 (Pin_8)
- net EPDC_GDSP: now also J3.10 (Pin_10); no longer J4.11 (Pin_11)
- net EPDC_SDCE0: now also J3.8 (Pin_8); no longer J4.40 (Pin_40)
- net EPDC_SDLE: now also J3.7 (Pin_7); no longer J4.41 (Pin_41)
- net EPDC_SDOE: now also J3.6 (Pin_6); no longer J4.43 (Pin_43)
- net GND: now also C178.2, C179.2, C180.2, C181.2, J3.12 (Pin_12), J3.5 (Pin_5), J3.MP (MountPin)
- net EPDC_CLKP: now reaches J4.26 (Pin_26)
- net EPDC_D0P: now reaches J4.44 (Pin_44)
- net EPDC_D11N: now reaches J4.7 (Pin_7)
- net EPDC_D0 renamed EPDC_D9N
- net EPDC_D1 renamed EPDC_D9P
- net EPDC_D10 renamed EPDC_D4N
- net EPDC_D11 renamed EPDC_D4P
- net EPDC_D12 renamed EPDC_D3N
- net EPDC_D13 renamed EPDC_D3P
- net EPDC_D14 renamed EPDC_D2N
- net EPDC_D15 renamed EPDC_D2P
- net EPDC_D2 renamed EPDC_D8N
- net EPDC_D3 renamed EPDC_D8P
- net EPDC_D4 renamed EPDC_D7N
- net EPDC_D5 renamed EPDC_D7P
- net EPDC_D6 renamed EPDC_D6N
- net EPDC_D7 renamed EPDC_D6P
- net EPDC_D8 renamed EPDC_D5N
- net EPDC_D9 renamed EPDC_D5P
- net EPDC_SDCLK renamed EPDC_CLKN
- net VBUS renamed +5V2
- net VNEG renamed VN3
- net VPOS renamed VP3
- new net EPDC_D0N: J4.43 (Pin_43)
- new net EPDC_D10N: J4.10 (Pin_10)
- new net EPDC_D10P: J4.11 (Pin_11)
- new net EPDC_D11P: J4.8 (Pin_8)
- new net EPDC_D1N: J4.40 (Pin_40)
- new net EPDC_D1P: J4.41 (Pin_41)
- new net VN1: C179.1, J3.13 (Pin_13)
- new net VN2: C178.1, J3.15 (Pin_15)
- new net VP1: C180.1, J3.3 (Pin_3)
- new net VP2: C181.1, J3.1 (Pin_1)
Other:
- moved on the sheet: J5

Commit message: PCB r0p10 wip
Connections:
- net +5V2 renamed +5V2_FL
- net VCOM renamed -VCOM
- net VGH renamed +VGH
- net VGL renamed -VGL
- net VN1 renamed -VN1
- net VN2 renamed -VN2
- net VN3 renamed -VN3
- net VP1 renamed +VP1
- net VP2 renamed +VP2
- net VP3 renamed +VP3

Commit message: PCB r0p10
Parts:
- removed C178, C179, C181: 220nF, Capacitor_SMD:C_0402_1005Metric, symbol Device:C
- removed J3: FH12-16S-0.5SH, Connector_FFC-FPC:Hirose_FH12-16S-0.5SH_1x16-1MP_P0.50mm_Horizontal, symbol Connector_Generic_MountingPin:Conn_01x16_MountingPin
- removed J4: FH12-50S-0.5SH, Connector_FFC-FPC:Hirose_FH12-50S-0.5SH_1x50-1MP_P0.50mm_Horizontal, symbol Connector_Generic_MountingPin:Conn_01x50_MountingPin
- removed J5: FH12-8S-0.5SH, Connector_FFC-FPC:Hirose_FH12-8S-0.5SH_1x08-1MP_P0.50mm_Horizontal, symbol Connector_Generic_MountingPin:Conn_01x08_MountingPin
- added C147: 220nF, Capacitor_SMD:C_0402_1005Metric, symbol Device:C
- added J3: FH12-36S-0.5SH, Connector_FFC-FPC:Hirose_FH12-36S-0.5SH_1x36-1MP_P0.50mm_Horizontal, symbol Connector_Generic_MountingPin:Conn_01x36_MountingPin
- added J4: FH12-30S-0.5SH, Connector_FFC-FPC:Hirose_FH12-30S-0.5SH_1x30-1MP_P0.50mm_Horizontal, symbol Connector_Generic_MountingPin:Conn_01x30_MountingPin
Connections:
- net +VP1 is gone; now on net +5V2_FL: C180.1
- net +3V3: now also J3.31 (Pin_31), J3.6 (Pin_6)
- net +5V2_FL: now also C147.1, J3.30 (Pin_30), J3.7 (Pin_7), J4.28 (Pin_28)
- net +VGH: now also J3.3 (Pin_3)
- net -VCOM: now also J3.5 (Pin_5)
- net -VGL: now also J3.1 (Pin_1)
- net EPDC_CLKN: now also J4.19 (Pin_19)
- net EPDC_CLKP: now also J4.20 (Pin_20)
- net EPDC_D0N: now also J3.26 (Pin_26)
- net EPDC_D0P: now also J3.27 (Pin_27)
- net EPDC_D10N: now also J4.4 (Pin_4)
- net EPDC_D10P: now also J4.5 (Pin_5)
- net EPDC_D11N: now also J4.1 (Pin_1)
- net EPDC_D11P: now also J4.2 (Pin_2)
- net EPDC_D1N: now also J3.23 (Pin_23)
- net EPDC_D1P: now also J3.24 (Pin_24)
- net EPDC_D2N: now also J3.20 (Pin_20)
- net EPDC_D2P: now also J3.21 (Pin_21)
- net EPDC_D3N: now also J3.17 (Pin_17)
- net EPDC_D3P: now also J3.18 (Pin_18)
- net EPDC_D4N: now also J4.25 (Pin_25)
- net EPDC_D4P: now also J4.26 (Pin_26)
- net EPDC_D5N: now also J4.22 (Pin_22)
- net EPDC_D5P: now also J4.23 (Pin_23)
- net EPDC_D6N: now also J4.16 (Pin_16)
- net EPDC_D6P: now also J4.17 (Pin_17)
- net EPDC_D7N: now also J4.13 (Pin_13)
- net EPDC_D7P: now also J4.14 (Pin_14)
- net EPDC_D8N: now also J4.10 (Pin_10)
- net EPDC_D8P: now also J4.11 (Pin_11)
- net EPDC_D9N: now also J4.7 (Pin_7)
- net EPDC_D9P: now also J4.8 (Pin_8)
- net EPDC_GDCLK: now also J3.13 (Pin_13)
- net EPDC_GDOE: now also J3.11 (Pin_11)
- net EPDC_GDSP: now also J3.12 (Pin_12)
- net EPDC_SDCE0: now also J3.10 (Pin_10)
- net EPDC_SDLE: now also J3.9 (Pin_9)
- net EPDC_SDOE: now also J3.8 (Pin_8)
- net FL_PWM1: now also J3.29 (Pin_29)
- net FL_PWM2: now also J4.29 (Pin_29)
- net GND: now also C147.2, J3.14 (Pin_14), J3.16 (Pin_16), J3.19 (Pin_19), J3.22 (Pin_22), J3.25 (Pin_25), J3.28 (Pin_28), J3.MP (MountPin), J4.12 (Pin_12), J4.15 (Pin_15), J4.18 (Pin_18), J4.21 (Pin_21), J4.24 (Pin_24), J4.27 (Pin_27), J4.3 (Pin_3), J4.6 (Pin_6), J4.9 (Pin_9), J4.MP (MountPin)
- net +VP3 renamed +VP
- net +VP: now also J3.35 (Pin_35)
- net -VN3 renamed -VN
- net -VN: now also J3.33 (Pin_33)
- new net EPDC_SE_CLK: J3.15 (Pin_15)
- new net FL_EN: J4.30 (Pin_30)
- no-connect marks 8 -> 5
Other:
- note added: "SE_D0"
- note added: "SE_D1"
- note added: "SE_D10"
- note added: "SE_D11"
- note added: "SE_D12"
- note added: "SE_D13"
- note added: "SE_D14"
- note added: "SE_D15"
- note added: "SE_D2"
- note added: "SE_D3"
- note added: "SE_D4"
- note added: "SE_D5"
- note added: "SE_D6"
- note added: "SE_D7"
- note added: "SE_D8"
- note added: "SE_D9"
- moved on the sheet: C158, C159, C180, C60, C61, C62, C63

Commit message: PCB r0p11
Parts:
- removed C180: 220nF, Capacitor_SMD:C_0402_1005Metric, symbol Device:C
- removed J3: FH12-36S-0.5SH, Connector_FFC-FPC:Hirose_FH12-36S-0.5SH_1x36-1MP_P0.50mm_Horizontal, symbol Connector_Generic_MountingPin:Conn_01x36_MountingPin
- removed J4: FH12-30S-0.5SH, Connector_FFC-FPC:Hirose_FH12-30S-0.5SH_1x30-1MP_P0.50mm_Horizontal, symbol Connector_Generic_MountingPin:Conn_01x30_MountingPin
- added J3: FH12-16S-0.5SH, Connector_FFC-FPC:Hirose_FH12-16S-0.5SH_1x16-1MP_P0.50mm_Horizontal, symbol Connector_Generic_MountingPin:Conn_01x16_MountingPin
- added J6: FH12-50S-0.5SH, Connector_FFC-FPC:Hirose_FH12-50S-0.5SH_1x50-1MP_P0.50mm_Horizontal, symbol Connector_Generic_MountingPin:Conn_01x50_MountingPin
Connections:
- net +3V3: now also J6.45 (Pin_45), J6.6 (Pin_6)
- net +5V2_FL: now also J6.44 (Pin_44), J6.7 (Pin_7)
- net +VGH: now also J6.3 (Pin_3)
- net +VP: now also J6.49 (Pin_49)
- net -VCOM: now also J6.5 (Pin_5)
- net -VGL: now also J6.1 (Pin_1)
- net -VN: now also J6.47 (Pin_47)
- net EPDC_CLKN: now also J3.2 (Pin_2)
- net EPDC_CLKP: now also J3.3 (Pin_3)
- net EPDC_D0N: now also J6.38 (Pin_38)
- net EPDC_D0P: now also J6.39 (Pin_39)
- net EPDC_D10N: now also J3.8 (Pin_8)
- net EPDC_D10P: now also J3.9 (Pin_9)
- net EPDC_D11N: now also J3.5 (Pin_5)
- net EPDC_D11P: now also J3.6 (Pin_6)
- net EPDC_D1N: now also J6.35 (Pin_35)
- net EPDC_D1P: now also J6.36 (Pin_36)
- net EPDC_D2N: now also J6.32 (Pin_32)
- net EPDC_D2P: now also J6.33 (Pin_33)
- net EPDC_D3N: now also J6.29 (Pin_29)
- net EPDC_D3P: now also J6.30 (Pin_30)
- net EPDC_D4N: now also J6.26 (Pin_26)
- net EPDC_D4P: now also J6.27 (Pin_27)
- net EPDC_D5N: now also J6.23 (Pin_23)
- net EPDC_D5P: now also J6.24 (Pin_24)
- net EPDC_D6N: now also J6.20 (Pin_20)
- net EPDC_D6P: now also J6.21 (Pin_21)
- net EPDC_D7N: now also J6.17 (Pin_17)
- net EPDC_D7P: now also J6.18 (Pin_18)
- net EPDC_D8N: now also J3.14 (Pin_14)
- net EPDC_D8P: now also J3.15 (Pin_15)
- net EPDC_D9N: now also J3.11 (Pin_11)
- net EPDC_D9P: now also J3.12 (Pin_12)
- net EPDC_GDCLK: now also J6.13 (Pin_13)
- net EPDC_GDOE: now also J6.11 (Pin_11)
- net EPDC_GDSP: now also J6.12 (Pin_12)
- net EPDC_SDCE0: now also J6.10 (Pin_10)
- net EPDC_SDLE: now also J6.9 (Pin_9)
- net EPDC_SDOE: now also J6.8 (Pin_8)
- net EPDC_SE_CLK: now also J6.15 (Pin_15)
- net FL_EN: now also J6.43 (Pin_43)
- net FL_PWM1: now also J6.41 (Pin_41)
- net FL_PWM2: now also J6.42 (Pin_42)
- net GND: now also J3.1 (Pin_1), J3.10 (Pin_10), J3.13 (Pin_13), J3.16 (Pin_16), J3.4 (Pin_4), J3.7 (Pin_7), J3.MP (MountPin), J6.14 (Pin_14), J6.16 (Pin_16), J6.19 (Pin_19), J6.22 (Pin_22), J6.25 (Pin_25), J6.28 (Pin_28), J6.31 (Pin_31), J6.34 (Pin_34), J6.37 (Pin_37), J6.40 (Pin_40), J6.MP (MountPin)
Other:
- moved on the sheet: C147, C158, C159, C60, C61, C62, C63

Commit message: PCB r0p13
Parts:
- C147, C158, C159, C60, C61, C62, C63: value 220nF -> 100nF/50V
- J3: footprint Connector_FFC-FPC:Hirose_FH12-16S-0.5SH_1x16-1MP_P0.50mm_Horizontal -> footprints:Xunpu_FPC-05F-16PH20_1x16-1MP_P0.50mm_Horizontal
- J6: footprint Connector_FFC-FPC:Hirose_FH12-50S-0.5SH_1x50-1MP_P0.50mm_Horizontal -> footprints:Xunpu_FPC-05F-50PH20_1x50-1MP_P0.50mm_Horizontal
Other:
- company: (none) -> Copyright 2025 Wenting Zhang
- title: (none) -> Glider
Changed lines of the file:
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@@
 	(generator_version "8.0")
 	(paper "A4")
+	(title_block
+		(title "Glider")
+		(date "2025-04-18")
+		(rev "R0.13")
+		(company "Copyright 2025 Wenting Zhang")
+	)
 	(junction
 		(at 129.54 165.1)
@@
 			)
 		)
-		(property "Value" "220nF"
+		(property "Value" "100nF/50V"
 			(at 111.76 156.21 90)
 			(effects
@@
 			)
 		)
-		(property "Value" "220nF"
+		(property "Value" "100nF/50V"
 			(at 111.76 151.13 90)
 			(effects
@@
 			)
 		)
-		(property "Value" "220nF"
+		(property "Value" "100nF/50V"
 			(at 111.76 44.45 90)
 			(effects
@@
 			)
 		)
-		(property "Footprint" "Connector_FFC-FPC:Hirose_FH12-16S-0.5SH_1x16-1MP_P0.50mm_Horizontal"
+		(property "Footprint" "footprints:Xunpu_FPC-05F-16PH20_1x16-1MP_P0.50mm_Horizontal"
 			(at 208.28 81.28 0)
 			(effects
@@
 			)
 		)
-		(property "Footprint" "Connector_FFC-FPC:Hirose_FH12-50S-0.5SH_1x50-1MP_P0.50mm_Horizontal"
+		(property "Footprint" "footprints:Xunpu_FPC-05F-50PH20_1x50-1MP_P0.50mm_Horizontal"
 			(at 139.7 104.14 0)
 			(effects
@@
 			)
 		)
-		(property "Value" "220nF"
+		(property "Value" "100nF/50V"
 			(at 111.76 153.67 90)
 			(effects
@@
 			)
 		)
-		(property "Value" "220nF"
+		(property "Value" "100nF/50V"
 			(at 111.76 39.37 90)
 			(effects
@@
 			)
 		)
-		(property "Value" "220nF"
+		(property "Value" "100nF/50V"
 			(at 111.76 49.53 90)
 			(effects
@@
 			)
 		)
-		(property "Value" "220nF"
+		(property "Value" "100nF/50V"
 			(at 111.76 161.29 90)
 			(effects

Commit message: PCB r1.1
Parts:
- C147, C158, C159, C60, C61, C62, C63: LCSC (none) -> C131394
- J3: value FH12-16S-0.5SH -> FPC-05F-16PH20; LCSC (none) -> C2856801
- J6: value FH12-50S-0.5SH -> FPC-05F-50PH20; LCSC (none) -> C2856813
Other:
- company: Copyright 2025 Wenting Zhang -> Copyright 2025 Modos Tech Inc
Changed lines of the file:
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@@
 	(title_block
 		(title "Glider")
-		(date "2025-04-18")
-		(rev "R0.13")
-		(company "Copyright 2025 Wenting Zhang")
+		(date "2025-06-26")
+		(rev "R1.1")
+		(company "Copyright 2025 Modos Tech Inc")
 	)
 	(junction
@@
 			)
 		)
+		(property "LCSC" "C131394"
+			(at 110.49 157.48 0)
+			(effects
+				(font
+					(size 1.27 1.27)
+				)
+				(hide yes)
+			)
+		)
 		(pin "1"
 		)
@@
 			)
 		)
+		(property "LCSC" "C131394"
+			(at 110.49 152.4 0)
+			(effects
+				(font
+					(size 1.27 1.27)
+				)
+				(hide yes)
+			)
+		)
 		(pin "1"
 		)
@@
 			)
 		)
+		(property "LCSC" "C131394"
+			(at 110.49 45.72 0)
+			(effects
+				(font
+					(size 1.27 1.27)
+				)
+				(hide yes)
+			)
+		)
 		(pin "1"
 		)
@@
 			)
 		)
-		(property "Value" "FH12-16S-0.5SH"
+		(property "Value" "FPC-05F-16PH20"
 			(at 210.82 84.1755 0)
 			(effects
@@
 			)
 		)
+		(property "LCSC" "C2856801"
+			(at 208.28 81.28 0)
+			(effects
+				(font
+					(size 1.27 1.27)
+				)
+				(hide yes)
+			)
+		)
 		(pin "10"
 		)
@@
 			)
 		)
-		(property "Value" "FH12-50S-0.5SH"
+		(property "Value" "FPC-05F-50PH20"
 			(at 142.24 107.0355 0)
 			(effects
@@
 			)
 		)
+		(property "LCSC" "C2856813"
+			(at 139.7 104.14 0)
+			(effects
+				(font
+					(size 1.27 1.27)
+				)
+				(hide yes)
+			)
+		)
 		(pin "1"
 		)
@@
 			)
 		)
+		(property "LCSC" "C131394"
+			(at 110.49 154.94 0)
+			(effects
+				(font
+					(size 1.27 1.27)
+				)
+				(hide yes)
+			)
+		)
 		(pin "1"
 		)
@@
 			)
 		)
+		(property "LCSC" "C131394"
+			(at 110.49 40.64 0)
+			(effects
+				(font
+					(size 1.27 1.27)
+				)
+				(hide yes)
+			)
+		)
 		(pin "1"
 		)
@@
 			)
 		)
+		(property "LCSC" "C131394"
+			(at 110.49 50.8 0)
+			(effects
+				(font
+					(size 1.27 1.27)
+				)
+				(hide yes)
+			)
+		)
 		(pin "1"
 		)
@@
 			(at 110.49 162.56 0)
 			(effects
+				(font
+					(size 1.27 1.27)
+				)
+				(hide yes)
+			)
+		)
+		(property "LCSC" "C131394"
+			(at 110.49 162.56 0)
+			(effects
