File: pcb/mainboard/power_mon.kicad_sch (KiCad schematic)
At the start: 41 parts, among them U14 STM32G030K6Tx, U21 INA3221, U22 INA3221, U27 INA3221

Commit message: PCB r0p10 wip
Parts:
- removed C89: 1uF, Capacitor_SMD:C_0402_1005Metric, symbol Device:C
- removed C90: 100nF, Capacitor_SMD:C_0402_1005Metric, symbol Device:C
- removed D20: LED GREEN, LED_SMD:LED_0603_1608Metric, symbol Device:LED
- removed D21: LED RED, LED_SMD:LED_0603_1608Metric, symbol Device:LED
- removed R119, R42: 1K, Resistor_SMD:R_0402_1005Metric, symbol Device:R
- removed U14: STM32G030K6Tx, Package_QFP:LQFP-32_7x7mm_P0.8mm, symbol MCU_ST_STM32G0:STM32G030K6Tx
Connections:
- net +1V8_FPGA is gone; now on net +1V8_VID: R7.1, U22.11 (IN-1)
- net MCU_I2C_SCL is gone; now on net I2C1_SCL: U21.6 (SCL), U22.6 (SCL), U27.6 (SCL)
- net MCU_I2C_SDA is gone; now on net I2C1_SDA: U21.7 (SDA), U22.7 (SDA), U27.5 (A0), U27.7 (SDA)
- net +1V8_DCDC: no longer R8.2, U22.15 (IN+2)
- net +1V8_VID: no longer R8.1, U22.14 (IN-2)
- net +3V3: no longer C141.1, C142.1, U22.16 (VPU), U22.4 (VS), U27.16 (VPU), U27.4 (VS)
- net +3V3_DCDC: now also C141.1, C142.1, R8.2, U22.15 (IN+2), U22.16 (VPU), U22.4 (VS), U27.16 (VPU), U27.2 (IN+3), U27.4 (VS); no longer U22.2 (IN+3)
- net +3V3_VID: now also R8.1, U22.14 (IN-2); no longer R15.1, U22.1 (IN-3)
- net +1V0_PL renamed +3V3_FPGA
- net +3V3_FPGA: now also R15.1; no longer R72.1
- net +1V0_PL_DCDC renamed +5V2
- net +5V2: now also U22.2 (IN+3); no longer U27.2 (IN+3)
- net +1V0_PS renamed +1V2
- net +1V0_PS_DCDC renamed +1V2_DCDC
- net EPD_SHDN renamed EPD_PWR_EN
- net VBUS renamed +VBUS
- net VGH renamed +VGH
- net VGL renamed -VGL
- net VN1 renamed -VN1
- net VN2 renamed -VN2
- net VN3 renamed -VN3
- net VP1 renamed +VP1
- net VP2 renamed +VP2
- net VP3 renamed +VP3
- new net +5V2_FL: R72.1, U22.1 (IN-3)
Other:
- moved on the sheet: C141, C142, C143, C91, R111, R112, R113, R114, R115, R116, R117, R118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

Commit message: PCB r0p10
Parts:
- removed R111, R113, R59, R69: 100K, Resistor_SMD:R_0402_1005Metric, symbol Device:R
- removed R112, R67: 10K, Resistor_SMD:R_0402_1005Metric, symbol Device:R
- removed R114, R68: 20K, Resistor_SMD:R_0402_1005Metric, symbol Device:R
- removed R15: 50mR, Resistor_SMD:R_0805_2012Metric, symbol Device:R
- R115, R117, R96, R98: value 100K -> 1M
- R116, R87: value 10K -> 100K
- R118, R97: value 7.5K -> 100K
- R50: value 2M -> 1M
- R51: value 200K/1% -> 100K
Connections:
- net +3V3_FPGA is gone; now on net GND: U27.1 (IN-3)
- net +3V3_DCDC: no longer U27.2 (IN+3)
- net GND: now also U27.2 (IN+3)
- net +1V2 renamed +1V2_FPGA
- net +VP3 renamed +VP
- net -VN3 renamed -VN
- net VN3_MEA renamed VN_MEA
- net VP3_MEA renamed VP_MEA
Other:
- moved on the sheet: R87, R96, R97, R98

Commit message: PCB r0p11
Connections:
- net +5V2 renamed +5V_DCDC
Changed lines of the file:
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@@
 			)
 		)
-		(property "Value" "+5V2"
-			(at 85.09 109.22 0)
+		(property "Value" "+5V_DCDC"
+			(at 87.63 109.22 0)
 			(effects
 				(font

Commit message: PCB r0p13
Parts:
- C141, C142, C143, C91: value 100nF -> 100nF/50V
- R115, R117, R50, R96, R98: value 1M -> 1M/1%
- R116, R118, R51, R87, R97: value 100K -> 100K/1%
- R53, R54, R56, R60, R61, R7, R72, R8: value 50mR -> 20mR
Other:
- company: (none) -> Copyright 2025 Wenting Zhang
- title: (none) -> Glider
Changed lines of the file:
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@@
 	(generator_version "8.0")
 	(paper "A4")
+	(title_block
+		(title "Glider")
+		(date "2025-04-18")
+		(rev "R0.13")
+		(company "Copyright 2025 Wenting Zhang")
+	)
 	(junction
 		(at 63.5 96.52)
@@
 			)
 		)
-		(property "Value" "100K"
+		(property "Value" "100K/1%"
 			(at 233.68 93.98 90)
 			(effects
@@
 			)
 		)
-		(property "Value" "1M"
+		(property "Value" "1M/1%"
 			(at 233.68 73.66 90)
 			(effects
@@
 			)
 		)
-		(property "Value" "100K"
+		(property "Value" "100K/1%"
 			(at 220.98 73.66 90)
 			(effects
@@
 			)
 		)
-		(property "Value" "50mR"
+		(property "Value" "20mR"
 			(at 74.93 147.32 90)
 			(effects
@@
 			)
 		)
-		(property "Value" "100nF"
+		(property "Value" "100nF/50V"
 			(at 132.461 91.313 0)
 			(effects
@@
 			)
 		)
-		(property "Value" "50mR"
+		(property "Value" "20mR"
 			(at 74.93 101.6 90)
 			(effects
@@
 			)
 		)
-		(property "Value" "100nF"
+		(property "Value" "100nF/50V"
 			(at 132.461 144.653 0)
 			(effects
@@
 			)
 		)
-		(property "Value" "100K"
+		(property "Value" "100K/1%"
 			(at 233.68 104.14 90)
 			(effects
@@
 			)
 		)
-		(property "Value" "1M"
+		(property "Value" "1M/1%"
 			(at 215.9 132.08 0)
 			(effects
@@
 			)
 		)
-		(property "Value" "100K"
+		(property "Value" "100K/1%"
 			(at 215.9 144.78 0)
 			(effects
@@
 			)
 		)
-		(property "Value" "50mR"
+		(property "Value" "20mR"
 			(at 74.93 109.22 90)
 			(effects
@@
 			)
 		)
-		(property "Value" "50mR"
+		(property "Value" "20mR"
 			(at 74.93 154.94 90)
 			(effects
@@
 			)
 		)
-		(property "Value" "1M"
+		(property "Value" "1M/1%"
 			(at 220.98 93.98 90)
 			(effects
@@
 			)
 		)
-		(property "Value" "1M"
+		(property "Value" "1M/1%"
 			(at 233.68 83.82 90)
 			(effects
@@
 			)
 		)
-		(property "Value" "50mR"
+		(property "Value" "20mR"
 			(at 74.93 48.26 90)
 			(effects
@@
 			)
 		)
-		(property "Value" "100nF"
+		(property "Value" "100nF/50V"
 			(at 226.441 144.653 0)
 			(effects
@@
 			)
 		)
-		(property "Value" "50mR"
+		(property "Value" "20mR"
 			(at 74.93 40.64 90)
 			(effects
@@
 			)
 		)
-		(property "Value" "50mR"
+		(property "Value" "20mR"
 			(at 74.93 93.98 90)
 			(effects
@@
 			)
 		)
-		(property "Value" "100K"
+		(property "Value" "100K/1%"
 			(at 220.98 83.82 90)
 			(effects
@@
 			)
 		)
-		(property "Value" "50mR"
+		(property "Value" "20mR"
 			(at 74.93 55.88 90)
 			(effects
@@
 			)
 		)
-		(property "Value" "100nF"
+		(property "Value" "100nF/50V"
 			(at 132.461 37.973 0)
 			(effects
@@
 			)
 		)
-		(property "Value" "1M"
+		(property "Value" "1M/1%"
 			(at 220.98 104.14 90)
 			(effects

Commit message: PCB r1.1
Parts:
- added C163, C164, C168, C169: 470nF/25V, Capacitor_SMD:C_0402_1005Metric, symbol Device:C
- C141, C142, C143, C91: LCSC (none) -> C131394
- R115, R117, R50, R96, R98: LCSC (none) -> C26083
- R116, R118, R51, R87, R97: LCSC (none) -> C25741
- R53, R54, R56, R60, R61, R7, R72, R8: LCSC (none) -> C7467301
- U21, U22, U27: LCSC (none) -> C181255
Connections:
- net +3V3_DCDC: now also R116.2, R118.2
- net GND: now also C163.1, C164.1, C168.1, C169.1; no longer R116.2, R118.2
- net VGH_MEA: now also C164.2
- net VGL_MEA: now also C169.2
- net VN_MEA: now also C168.2
- net VP_MEA: now also C163.2
Other:
- company: Copyright 2025 Wenting Zhang -> Copyright 2025 Modos Tech Inc
- moved on the sheet: C91, R115, R116, R117, R118, R50, R51, R87, R96, R97, R98
