File: pcb/mainboard/tmds_in.kicad_sch (KiCad schematic)
At the start: 33 parts, among them J2 XUNPU HDMI-101S, U15 ADV7611, Y3 28.63636MHz

Commit message: PCB r0p10 wip
Connections:
- net HDMI_5V: no longer J2.19 (+5V), R16.2, R49.2
- net DPI_B0: no longer names the net of RN13.8 (R1.2)
- net DPI_B1: no longer names the net of RN13.7 (R2.2)
- net DPI_G0: no longer names the net of RN8.8 (R1.2)
- net DPI_G1: no longer names the net of RN8.7 (R2.2)
- net DPI_R0: no longer names the net of RN11.8 (R1.2)
- net DPI_R1: no longer names the net of RN11.7 (R2.2)
- new net +5V_HDMI: J2.19 (+5V), R16.2, R49.2
- no-connect marks 8 -> 14

Commit message: PCB r0p10
Parts:
- Y3: value 28.63636MHz -> 24MHz

Commit message: PCB r0p13
Parts:
- removed J2: XUNPU HDMI-101S, footprints:HDMI_Micro-D_Molex_46765-1x01_MOD, symbol Connector:HDMI_D_1.4
- added C161, C162: 22uF/6.3V, Capacitor_SMD:C_0603_1608Metric, symbol Device:C
- added J4: HDMI_C_1.3, footprints:HDMI_C_GT-HD006A-CGNGX, symbol Connector:HDMI_C_1.3
- C113, C125: value 18pF -> 18pF/50V
- C126, C132: value 1uF -> 4.7uF/6.3V
- C127, C128, C129, C130, C131, C133, C134, C135, C136, C137, C138, C139: value 100nF -> 100nF/50V
- R16, R47, R49: value 10K -> 10K/1%
- R45: value 1M -> 1M/1%
- R46: value 27R -> 33R/1%
Connections:
- net HDMI_5V is gone; now on net +5V_HDMI: U15.64 (RXA_5V)
- net +1V8_VID: now also C161.1
- net +3V3_VID: now also C162.1
- net +5V_HDMI: now also J4.18 (+5V)
- net GND: now also C161.2, C162.2, J4.1 (D2S), J4.10 (CKS), J4.13 (GND), J4.4 (D1S), J4.7 (D0S), J4.SH
- net HDMI_HPD: now also J4.19 (HPD)
- net HDMI_SCL: now also J4.15 (SCL)
- net HDMI_SDA: now also J4.16 (SDA)
- net TMDS_CKN: now also J4.12 (CK-)
- net TMDS_CKP: now also J4.11 (CK+)
- net TMDS_D0N: now also J4.9 (D0-)
- net TMDS_D0P: now also J4.8 (D0+)
- net TMDS_D1N: now also J4.6 (D1-)
- net TMDS_D1P: now also J4.5 (D1+)
- net TMDS_D2N: now also J4.3 (D2-)
- net TMDS_D2P: now also J4.2 (D2+)
Other:
- company: Copyright 2024 Wenting Zhang -> Copyright 2025 Wenting Zhang

Commit message: PCB r1.1
Parts:
- added C170: 1nF/50V, Capacitor_SMD:C_0402_1005Metric, symbol Device:C
- added R15: 100R/1%, Resistor_SMD:R_0402_1005Metric, symbol Device:R
- C113, C125: LCSC (none) -> C106202
- C126, C132: LCSC (none) -> C307423
- C127, C128, C129, C130, C131, C133, C134, C135, C136, C137, C138, C139: LCSC (none) -> C131394
- C161, C162: LCSC (none) -> C59461
- D10, D9: LCSC (none) -> C907837
- J4: LCSC (none) -> C27636755
- R16, R47, R49: LCSC (none) -> C25744
- R45: LCSC (none) -> C26083
- R46: LCSC (none) -> C25105
- RN10, RN11, RN12, RN13, RN7, RN8, RN9: LCSC (none) -> C425299
- U15: LCSC (none) -> C146553
- Y3: LCSC (none) -> C70590
Connections:
- net GND: now also C170.2
- net HDMI_HPD: now also C170.1, R15.2; no longer U15.1 (HPA_A/INT2)
- new net: R15.1, U15.1 (HPA_A/INT2)
Other:
- company: Copyright 2025 Wenting Zhang -> Copyright 2025 Modos Tech Inc
- moved on the sheet: C161, C162
