File: pcb/mainboard/user_extension.kicad_sch (KiCad schematic)
At the start: 1 part, among them J2 Conn_01x08_MountingPin

Commit message: PCB r1.1
Parts:
- J2: LCSC (none) -> DNP
Other:
- company: Copyright 2025 Wenting Zhang -> Copyright 2025 Modos Tech Inc
Changed lines of the file:
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@@
 	(title_block
 		(title "Glider")
-		(date "2025-04-18")
-		(rev "R0.13")
-		(company "Copyright 2025 Wenting Zhang")
+		(date "2025-06-26")
+		(rev "R1.1")
+		(company "Copyright 2025 Modos Tech Inc")
 	)
 	(wire
@@
 			(at 154.94 99.06 0)
 			(effects
+				(font
+					(size 1.27 1.27)
+				)
+				(hide yes)
+			)
+		)
+		(property "LCSC" "DNP"
+			(at 154.94 99.06 0)
+			(effects
