File: pcb/33p-adapter-a/adapter.kicad_pcb (KiCad board)
At the start: 2 copper layers, 30 x 21 mm, 9 parts, among them J1 FH12-40S-0.5SH, J2 FH34S-34S-0.5SH(50)

Commit message: Update adapters
Parts:
- removed C10, C11, C12, C13, C14, C8, C9: 220nF, Capacitor_SMD:C_0402_1005Metric
- removed J2: FH34S-34S-0.5SH(50), Connector_FFC-FPC:Hirose_FH12-34S-0.5SH_1x34-1MP_P0.50mm_Horizontal
- added J3: Conn_01x33_MountingPin, Connector_FFC-FPC:Hirose_FH12-33S-0.5SH_1x33-1MP_P0.50mm_Horizontal, F.Cu at (165.7, 89.0)
- added R1: 0, Resistor_SMD:R_0402_1005Metric, F.Cu at (159.8, 84.8)
- added R2: 0, Resistor_SMD:R_0402_1005Metric, F.Cu at (172.2, 84.9)
Connections:
- J1 pad 40: VCOM -> /BORDER
Routing:
- net VPOS: track 7.79 -> 29.2 mm, vias 0 -> 2
- net VGL: track 8.18 -> 26.4 mm, vias 0 -> 2
- net VCOM: track 30.9 -> 15.8 mm, vias 3 -> 2
- net +3V3: track 14.0 -> 28.1 mm, vias 0 -> 2
- net GND: track 16.0 -> 4.94 mm, vias 24 -> 14
- net VGH: track 30.0 -> 20.5 mm
- net /BORDER: track 0.00 -> 7.95 mm
- net /RL: track 0.00 -> 7.51 mm, vias 0 -> 2
- net /GDOE: track 20.8 -> 24.3 mm
- net /GDCLK: track 20.3 -> 22.1 mm
- net /UD: track 0.00 -> 1.74 mm
- net VNEG: track 30.8 -> 31.6 mm
- net /GDSP: track 19.9 -> 20.7 mm
Other:
- board text added: "097OC/TC"
- board text added: "Glider 33P-A"
- board text removed: "060S/X/K"
- board text removed: "Glider 34P-A"
