File: pcb/34p-adapter-b/adapter.kicad_sch (KiCad schematic)
At the start: 2 parts, among them J1 FH12-40S-0.5SH, J2 AXT334124

Commit message: Update adapters
Parts:
- J2: footprint Connector_FFC-FPC:Hirose_FH12-34S-0.5SH_1x34-1MP_P0.50mm_Horizontal -> footprints:AXT334124
Changed lines of the file:
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@@
 			)
 		)
-		(property "Footprint" "Connector_FFC-FPC:Hirose_FH12-34S-0.5SH_1x34-1MP_P0.50mm_Horizontal"
+		(property "Footprint" "footprints:AXT334124"
 			(at 198.12 96.52 0)
 			(effects
